Commit message: added dependency

File: src/moveit_pro_kinova_configs/kinova_gen3_mujoco_config/description/picknik_kinova_gen3.xacro (robot description, xacro)
@@ -48,14 +48,14 @@
         <origin rpy="0 0 0" xyz="0 0 0"/>
         <geometry>
-          <mesh filename="package://kortex_description/arms/gen3/7dof/meshes/base_link.dae"/>
-        </geometry>
-        <material name="">
-          <color rgba="0.75294 0.75294 0.75294 1"/>
-        </material>
-      </visual>
-      <collision>
-        <origin rpy="0 0 0" xyz="0 0 0"/>
-        <geometry>
-          <mesh filename="package://kortex_description/arms/gen3/7dof/meshes/base_link.dae"/>
+          <mesh filename="package://kortex_description/arms/gen3/7dof/meshes/base_link.STL"/>
+        </geometry>
+        <material name="">
+          <color rgba="0.75294 0.75294 0.75294 1"/>
+        </material>
+      </visual>
+      <collision>
+        <origin rpy="0 0 0" xyz="0 0 0"/>
+        <geometry>
+          <mesh filename="package://kortex_description/arms/gen3/7dof/meshes/base_link.STL"/>
         </geometry>
       </collision>
@@ -70,14 +70,14 @@
         <origin rpy="0 0 0" xyz="0 0 0"/>
         <geometry>
-          <mesh filename="package://kortex_description/arms/gen3/7dof/meshes/shoulder_link.dae"/>
-        </geometry>
-        <material name="">
-          <color rgba="0.75294 0.75294 0.75294 1"/>
-        </material>
-      </visual>
-      <collision>
-        <origin rpy="0 0 0" xyz="0 0 0"/>
-        <geometry>
-          <mesh filename="package://kortex_description/arms/gen3/7dof/meshes/shoulder_link.dae"/>
+          <mesh filename="package://kortex_description/arms/gen3/7dof/meshes/shoulder_link.STL"/>
+        </geometry>
+        <material name="">
+          <color rgba="0.75294 0.75294 0.75294 1"/>
+        </material>
+      </visual>
+      <collision>
+        <origin rpy="0 0 0" xyz="0 0 0"/>
+        <geometry>
+          <mesh filename="package://kortex_description/arms/gen3/7dof/meshes/shoulder_link.STL"/>
         </geometry>
       </collision>
@@ -99,14 +99,14 @@
         <origin rpy="0 0 0" xyz="0 0 0"/>
         <geometry>
-          <mesh filename="package://kortex_description/arms/gen3/7dof/meshes/half_arm_1_link.dae"/>
-        </geometry>
-        <material name="">
-          <color rgba="0.75294 0.75294 0.75294 1"/>
-        </material>
-      </visual>
-      <collision>
-        <origin rpy="0 0 0" xyz="0 0 0"/>
-        <geometry>
-          <mesh filename="package://kortex_description/arms/gen3/7dof/meshes/half_arm_1_link.dae"/>
+          <mesh filename="package://kortex_description/arms/gen3/7dof/meshes/half_arm_1_link.STL"/>
+        </geometry>
+        <material name="">
+          <color rgba="0.75294 0.75294 0.75294 1"/>
+        </material>
+      </visual>
+      <collision>
+        <origin rpy="0 0 0" xyz="0 0 0"/>
+        <geometry>
+          <mesh filename="package://kortex_description/arms/gen3/7dof/meshes/half_arm_1_link.STL"/>
         </geometry>
       </collision>
@@ -128,14 +128,14 @@
         <origin rpy="0 0 0" xyz="0 0 0"/>
         <geometry>
-          <mesh filename="package://kortex_description/arms/gen3/7dof/meshes/half_arm_2_link.dae"/>
-        </geometry>
-        <material name="">
-          <color rgba="0.75294 0.75294 0.75294 1"/>
-        </material>
-      </visual>
-      <collision>
-        <origin rpy="0 0 0" xyz="0 0 0"/>
-        <geometry>
-          <mesh filename="package://kortex_description/arms/gen3/7dof/meshes/half_arm_2_link.dae"/>
+          <mesh filename="package://kortex_description/arms/gen3/7dof/meshes/half_arm_2_link.STL"/>
+        </geometry>
+        <material name="">
+          <color rgba="0.75294 0.75294 0.75294 1"/>
+        </material>
+      </visual>
+      <collision>
+        <origin rpy="0 0 0" xyz="0 0 0"/>
+        <geometry>
+          <mesh filename="package://kortex_description/arms/gen3/7dof/meshes/half_arm_2_link.STL"/>
         </geometry>
       </collision>
@@ -157,14 +157,14 @@
         <origin rpy="0 0 0" xyz="0 0 0"/>
         <geometry>
-          <mesh filename="package://kortex_description/arms/gen3/7dof/meshes/forearm_link.dae"/>
-        </geometry>
-        <material name="">
-          <color rgba="0.75294 0.75294 0.75294 1"/>
-        </material>
-      </visual>
-      <collision>
-        <origin rpy="0 0 0" xyz="0 0 0"/>
-        <geometry>
-          <mesh filename="package://kortex_description/arms/gen3/7dof/meshes/forearm_link.dae"/>
+          <mesh filename="package://kortex_description/arms/gen3/7dof/meshes/forearm_link.STL"/>
+        </geometry>
+        <material name="">
+          <color rgba="0.75294 0.75294 0.75294 1"/>
+        </material>
+      </visual>
+      <collision>
+        <origin rpy="0 0 0" xyz="0 0 0"/>
+        <geometry>
+          <mesh filename="package://kortex_description/arms/gen3/7dof/meshes/forearm_link.STL"/>
         </geometry>
       </collision>
@@ -186,14 +186,14 @@
         <origin rpy="0 0 0" xyz="0 0 0"/>
         <geometry>
-          <mesh filename="package://kortex_description/arms/gen3/7dof/meshes/spherical_wrist_1_link.dae"/>
-        </geometry>
-        <material name="">
-          <color rgba="0.75294 0.75294 0.75294 1"/>
-        </material>
-      </visual>
-      <collision>
-        <origin rpy="0 0 0" xyz="0 0 0"/>
-        <geometry>
-          <mesh filename="package://kortex_description/arms/gen3/7dof/meshes/spherical_wrist_1_link.dae"/>
+          <mesh filename="package://kortex_description/arms/gen3/7dof/meshes/spherical_wrist_1_link.STL"/>
+        </geometry>
+        <material name="">
+          <color rgba="0.75294 0.75294 0.75294 1"/>
+        </material>
+      </visual>
+      <collision>
+        <origin rpy="0 0 0" xyz="0 0 0"/>
+        <geometry>
+          <mesh filename="package://kortex_description/arms/gen3/7dof/meshes/spherical_wrist_1_link.STL"/>
         </geometry>
       </collision>
@@ -215,14 +215,14 @@
         <origin rpy="0 0 0" xyz="0 0 0"/>
         <geometry>
-          <mesh filename="package://kortex_description/arms/gen3/7dof/meshes/spherical_wrist_2_link.dae"/>
-        </geometry>
-        <material name="">
-          <color rgba="0.75294 0.75294 0.75294 1"/>
-        </material>
-      </visual>
-      <collision>
-        <origin rpy="0 0 0" xyz="0 0 0"/>
-        <geometry>
-          <mesh filename="package://kortex_description/arms/gen3/7dof/meshes/spherical_wrist_2_link.dae"/>
+          <mesh filename="package://kortex_description/arms/gen3/7dof/meshes/spherical_wrist_2_link.STL"/>
+        </geometry>
+        <material name="">
+          <color rgba="0.75294 0.75294 0.75294 1"/>
+        </material>
+      </visual>
+      <collision>
+        <origin rpy="0 0 0" xyz="0 0 0"/>
+        <geometry>
+          <mesh filename="package://kortex_description/arms/gen3/7dof/meshes/spherical_wrist_2_link.STL"/>
         </geometry>
       </collision>
@@ -244,14 +244,14 @@
         <origin rpy="0 0 0" xyz="0 0 0"/>
         <geometry>
-          <mesh filename="package://kortex_description/arms/gen3/7dof/meshes/bracelet_with_vision_link.dae"/>
-        </geometry>
-        <material name="">
-          <color rgba="0.75294 0.75294 0.75294 1"/>
-        </material>
-      </visual>
-      <collision>
-        <origin rpy="0 0 0" xyz="0 0 0"/>
-        <geometry>
-          <mesh filename="package://kortex_description/arms/gen3/7dof/meshes/bracelet_with_vision_link.dae"/>
+          <mesh filename="package://kortex_description/arms/gen3/7dof/meshes/bracelet_with_vision_link.STL"/>
+        </geometry>
+        <material name="">
+          <color rgba="0.75294 0.75294 0.75294 1"/>
+        </material>
+      </visual>
+      <collision>
+        <origin rpy="0 0 0" xyz="0 0 0"/>
+        <geometry>
+          <mesh filename="package://kortex_description/arms/gen3/7dof/meshes/bracelet_with_vision_link.STL"/>
         </geometry>
       </collision>
