Commit message: Setup the fanuc_sim config with a tool-changing example
Former-commit-id: c84e5e276c6220e2775d151950947e94bafff380

File: src/fanuc_sim/description/fanuc_lrmate200id.ros2_control.xacro (robot description, xacro)
@@ -6,4 +6,5 @@
   >
     <xacro:arg name="mujoco_model" default="description/scene.xml" />
+    <xacro:arg name="mujoco_viewer" default="false" />
     <xacro:arg name="hardware_interface" default="mock" />
     <xacro:property
@@ -26,4 +27,5 @@
           <param name="mujoco_model">$(arg mujoco_model)</param>
           <param name="mujoco_model_package">fanuc_sim</param>
+          <param name="mujoco_viewer">$(arg mujoco_viewer)</param>
           <param name="render_publish_rate">10</param>
           <param name="tf_publish_rate">60</param>

File: src/fanuc_sim/description/picknik_fanuc.xacro (robot description, xacro)
@@ -13,9 +13,56 @@
     filename="$(find fanuc_sim)/description/fanuc_lrmate200id.ros2_control.xacro"
   />
-  <link name="world" />
-  <joint name="world_joint" type="fixed">
+  <link name="world"/>
+  <link name="arm_pedestal">
+    <visual>
+      <origin rpy="0 0 0" xyz="0 0 0" />
+      <geometry>
+        <box size="0.4 0.4 0.3" />
+      </geometry>
+    </visual>
+    <visual>
+      <origin rpy="0 0 0" xyz="0.23 0.03 0.1" />
+      <geometry>
+        <box size="0.12 0.02 0.02" />
+      </geometry>
+    </visual>
+    <visual>
+      <origin rpy="0 0 0" xyz="0.23 -0.03 0.1" />
+      <geometry>
+        <box size="0.12 0.02 0.02" />
+      </geometry>
+    </visual>
+  </link>
+  <joint name="scene_joint" type="fixed">
     <parent link="world" />
+    <child link="arm_pedestal" />
+    <origin rpy="0 0 0" xyz="0 0.3 0.15" />
+  </joint>
+  <joint name="base_joint" type="fixed">
+    <parent link="arm_pedestal" />
     <child link="base_link" />
-    <origin rpy="0 0 0" xyz="0 0 0" />
+    <origin rpy="0 0 0" xyz="0 0 0.15" />
+  </joint>
+  <link name="table">
+    <visual>
+      <origin rpy="0 0 0" xyz="0 0 0" />
+      <geometry>
+        <box size="1 1 0.05" />
+      </geometry>
+      <material name="brown">
+        <color rgba="0.3 0.15 0.05 1" />
+      </material>
+    </visual>
+    <collision>
+      <origin rpy="0 0 0" xyz="0 0 0" />
+      <geometry>
+        <box size="1 1 0.05" />
+      </geometry>
+    </collision>
+  </link>
+  <joint name="table_joint" type="fixed">
+    <parent link="world" />
+    <child link="table" />
+    <origin rpy="0 0 0" xyz="0 1 0.45" />
   </joint>
   <xacro:fanuc_lrmate200id prefix="" />
