Commit message: Vacuum gripping working!

File: src/fanuc_sim/description/picknik_fanuc.xacro (robot description, xacro)
@@ -44,26 +44,4 @@
     <origin rpy="0 0 0" xyz="0 0 0.15" />
   </joint>
-  <link name="table">
-    <visual>
-      <origin rpy="0 0 0" xyz="0 0 0" />
-      <geometry>
-        <box size="1 1 0.05" />
-      </geometry>
-      <material name="brown">
-        <color rgba="0.3 0.15 0.05 1" />
-      </material>
-    </visual>
-    <collision>
-      <origin rpy="0 0 0" xyz="0 0 0" />
-      <geometry>
-        <box size="1 1 0.05" />
-      </geometry>
-    </collision>
-  </link>
-  <joint name="table_joint" type="fixed">
-    <parent link="world" />
-    <child link="table" />
-    <origin rpy="0 0 0" xyz="0 1 0.45" />
-  </joint>
   <xacro:fanuc_lrmate200id prefix="" />
   <xacro:fanuc_lrmate200id_ros2_control

Commit message: Add assembly and rasterize workcells to world

File: src/fanuc_sim/description/picknik_fanuc.xacro (robot description, xacro)
@@ -37,5 +37,5 @@
     <parent link="world" />
     <child link="arm_pedestal" />
-    <origin rpy="0 0 0" xyz="0 0.3 0.15" />
+    <origin rpy="0 0 0" xyz="0 0 0.15" />
   </joint>
   <joint name="base_joint" type="fixed">

Commit message: Start of cleaning example - need to invert hemisphere stl normals for mesh used by mesh normals behavior  or add flipped a tool link, and then turn of 'pose_only' in planning behavior

File: src/fanuc_sim/description/picknik_fanuc.xacro (robot description, xacro)
@@ -44,4 +44,28 @@
     <origin rpy="0 0 0" xyz="0 0 0.15" />
   </joint>
+  <!-- Need these entries in URDF due to limitations in GetMeshNormalPoses behavior -->
+  <link name="convex_hemisphere">
+    <visual>
+      <origin rpy="0 0 0" xyz="0 0 0" />
+      <geometry>
+        <mesh
+          filename="package://picknik_accessories/mujoco_assets/assets/convex_hemisphere.stl"
+        />
+      </geometry>
+      <xacro:material_fanuc_gray28 />
+    </visual>
+    <!-- <collision>
+      <geometry>
+        <mesh
+          filename="package://picknik_accessories/mujoco_assets/assets/convex_hemisphere.stl"
+        />
+      </geometry>
+    </collision> -->
+  </link>
+  <joint name="convex_hemisphere_joint" type="fixed">
+    <parent link="world" />
+    <child link="convex_hemisphere" />
+      <origin xyz="0.75 0 0.6" rpy="0 0 1.5708" />
+  </joint>
   <xacro:fanuc_lrmate200id prefix="" />
   <xacro:fanuc_lrmate200id_ros2_control
