Commit message: Remove april_tag_hardware_interface

File: src/moveit_pro_ur_configs/ur5e_ridgeback_mujoco_config/description/picknik_ur.xacro (robot description, xacro)
@@ -20,5 +20,4 @@
   <xacro:arg name="spawn_airfoil" default="true"/>
   <xacro:arg name="mujoco_model" default="description/scene.xml"/>
-  <xacro:arg name="run_apriltag_hardware_interface" default="true"/>
   <!-- Import UR and environment macros -->
   <xacro:include filename="$(find picknik_ur_base_config)/description/picknik_ur_macro.xacro"/>
@@ -123,4 +122,4 @@
   </xacro:picknik_ur>
   <!-- MuJoCo Hardware interface -->
-  <xacro:picknik_ur_mujoco_ros2_control mujoco_model="$(arg mujoco_model)" run_apriltag_hardware_interface="$(arg mujoco_model)"/>
+  <xacro:picknik_ur_mujoco_ros2_control mujoco_model="$(arg mujoco_model)"/>
 </robot>

File: src/moveit_pro_ur_configs/ur5e_ridgeback_mujoco_config/description/picknik_ur_mujoco_ros2_control.xacro (robot description, xacro)
@@ -1,5 +1,5 @@
 <?xml version="1.0" encoding="utf-8"?>
 <robot xmlns:xacro="http://ros.org/wiki/xacro">
-  <xacro:macro name="picknik_ur_mujoco_ros2_control" params="mujoco_model run_apriltag_hardware_interface">
+  <xacro:macro name="picknik_ur_mujoco_ros2_control" params="mujoco_model">
     <ros2_control name="ur_mujoco_control" type="system">
       <joint name="shoulder_pan_joint">
@@ -94,11 +94,4 @@
       </hardware>
     </ros2_control>
-    <xacro:if value="$(arg run_apriltag_hardware_interface)">
-      <ros2_control name="apriltag_hardware_interface" type="system">
-          <hardware>
-              <plugin>apriltag_hardware_interface/AprilTagHardwareInterface</plugin>
-          </hardware>
-      </ros2_control>
-    </xacro:if>
   </xacro:macro>
 </robot>
