Commit message: update config to integrate bar world

File: src/moveit_pro_ur_configs/bring_it_sim/description/ur5e_ridgeback.xacro (robot description, xacro)
@@ -18,9 +18,9 @@
   <xacro:arg name="tool_device_name" default="/dev/ttyUSB0"/>
   <xacro:arg name="initial_positions_file" default="$(find picknik_ur_base_config)/config/initial_positions.yaml"/>
-  <xacro:arg name="mujoco_model" default="description/scene.xml"/>
+  <xacro:arg name="mujoco_model" default="description/bar_scene.xml"/>
   <!-- Import UR and environment macros -->
   <xacro:include filename="$(find picknik_ur_base_config)/description/picknik_ur_macro.xacro"/>
-  <xacro:include filename="$(find ur5e_ridgeback_mujoco_config)/description/picknik_ur_attachments_macro.xacro"/>
-  <xacro:include filename="$(find ur5e_ridgeback_mujoco_config)/description/picknik_ur_mujoco_ros2_control.xacro"/>
+  <xacro:include filename="$(find bring_it_sim)/description/picknik_ur_attachments_macro.xacro"/>
+  <xacro:include filename="$(find bring_it_sim)/description/picknik_ur_mujoco_ros2_control.xacro"/>
   <xacro:include filename="$(find ridgeback_description)/urdf/ridgeback.urdf.xacro"/>
   <link name="world"/>
@@ -37,5 +37,5 @@
     <visual>
       <geometry>
-        <mesh filename="package://ur5e_ridgeback_mujoco_config/description/assets/HAM_Assem.stl"/>
+        <mesh filename="package://bring_it_sim/description/assets/HAM_Assem.stl"/>
       </geometry>
       <material name="grey">
@@ -45,5 +45,5 @@
     <collision>
       <geometry>
-        <mesh filename="package://ur5e_ridgeback_mujoco_config/description/assets/HAM_Assem.stl"/>
+        <mesh filename="package://bring_it_sim/description/assets/HAM_Assem.stl"/>
       </geometry>
     </collision>

Commit message: Adds bar map to navigation and increases the max position limits for the base linear joints

File: src/moveit_pro_ur_configs/bring_it_sim/description/ur5e_ridgeback.xacro (robot description, xacro)
@@ -61,5 +61,5 @@
     <child link="virual_rail_link_1" />
     <origin xyz="0 0 0" rpy="0 0 0" />
-    <limit effort="1000.0" lower="-5.0" upper="5.0" velocity="0.175" acceleration="10.0"/>
+    <limit effort="1000.0" lower="-20.0" upper="20.0" velocity="0.175" acceleration="10.0"/>
     <dynamics damping="20.0" friction="500.0" />
   </joint>
@@ -70,5 +70,5 @@
     <child link="virual_rail_link_2" />
     <origin xyz="0 0 0" rpy="0 0 0" />
-    <limit effort="1000.0" lower="-5.0" upper="5.0" velocity="0.175" acceleration="10.0"/>
+    <limit effort="1000.0" lower="-20.0" upper="20.0" velocity="0.175" acceleration="10.0"/>
     <dynamics damping="20.0" friction="500.0" />
   </joint>

Commit message: Fix typo

File: src/moveit_pro_ur_configs/bring_it_sim/description/ur5e_ridgeback.xacro (robot description, xacro)
@@ -55,18 +55,18 @@
     <child link="ur_mount_point" />
   </joint>
-  <link name="virual_rail_link_1"/>
+  <link name="virtual_rail_link_1"/>
   <joint name="linear_x_joint" type="prismatic">
     <axis xyz="1 0 0"/>
     <parent link="world" />
-    <child link="virual_rail_link_1" />
+    <child link="virtual_rail_link_1" />
     <origin xyz="0 0 0" rpy="0 0 0" />
     <limit effort="1000.0" lower="-20.0" upper="20.0" velocity="0.175" acceleration="10.0"/>
     <dynamics damping="20.0" friction="500.0" />
   </joint>
-  <link name="virual_rail_link_2"/>
+  <link name="virtual_rail_link_2"/>
   <joint name="linear_y_joint" type="prismatic">
     <axis xyz="0 1 0"/>
-    <parent link="virual_rail_link_1" />
-    <child link="virual_rail_link_2" />
+    <parent link="virtual_rail_link_1" />
+    <child link="virtual_rail_link_2" />
     <origin xyz="0 0 0" rpy="0 0 0" />
     <limit effort="1000.0" lower="-20.0" upper="20.0" velocity="0.175" acceleration="10.0"/>
@@ -75,5 +75,5 @@
   <joint name="rotational_yaw_joint" type="revolute">
     <axis xyz="0 0 1"/>
-    <parent link="virual_rail_link_2"/>
+    <parent link="virtual_rail_link_2"/>
     <child link="ridgeback_base_link"/>
     <origin rpy="0 0 0" xyz="0 0 0"/>
