Commit message: Remove unused MuJoCo scenes, split xacro into assets/and body for easier include, adjust scene and xacro for horizontal mounting, fix scene camera orientation
Former-commit-id: 7efb4fc6bd364e1a8c5d135623cc19254dfb49c6

File: src/moveit_pro_kinova_configs/picknik_kinova_satellite_sim/description/picknik_kinova_gen3.xacro (robot description, xacro)
@@ -25,8 +25,8 @@
     <!-- Import macros for main hardware components -->
     <xacro:include filename="$(find kortex_description)/arms/$(arg arm)/$(arg dof)dof/urdf/$(arg arm)_macro.xacro" />
-    <xacro:include filename="$(find kortex_description)/grippers/$(arg gripper)/urdf/$(arg gripper)_macro.xacro" />
+    <!-- <xacro:include filename="$(find kortex_description)/grippers/$(arg gripper)/urdf/$(arg gripper)_macro.xacro" /> -->
     <xacro:include filename="$(find picknik_accessories)/descriptions/sensors/realsense_d415.urdf.xacro"/>
     <!-- Import environment macros -->
-    <xacro:include filename="$(find picknik_accessories)/descriptions/geometry/cube.urdf.xacro"/>
+    <!-- <xacro:include filename="$(find picknik_accessories)/descriptions/geometry/cube.urdf.xacro"/> -->
     <!-- World is centered under base_link of the robot, on the ground -->
     <link name="world"/>
@@ -36,5 +36,5 @@
     <!-- Load the arm -->
     <joint name="base_joint" type="fixed">
-      <origin rpy="0 0 0" xyz="0 0 0.02"/>
+      <origin rpy="1.5708 0 1.5708" xyz="0 0 0.5"/>
       <parent link="world"/>
       <child link="base_link"/>
@@ -530,7 +530,7 @@
     </joint>
     <!-- Environment -->
-    <xacro:cube link_name="table" connected_to="world" length="2.00" width="2.00" height="0.25" alpha="0.3">
+    <!-- <xacro:cube link_name="table" connected_to="world" length="2.00" width="2.00" height="0.25" alpha="0.3">
       <origin xyz="0 0 -0.145" rpy="0 0 0"/>
-    </xacro:cube>
+    </xacro:cube> -->
     <!-- Visual aids for grasping -->
     <link name="finger_tip_closed_point">
@@ -561,5 +561,5 @@
       <parent link="world" />
       <child link="external_camera_link" />
-      <origin xyz="-0.3 0.3 1.0" rpy="0.0 0.4 0" />
+      <origin xyz="-0.3 0.3 1.0" rpy="0 0.5236 0" />
     </joint>
     <xacro:realsense_d415 parent="external_camera_link" name="scene_camera">
