Commit message: fixed collsion on the vacuum. Planning is still very strange
Signed-off-by: Paul Gesel <paul.gesel@picknik.ai>

File: src/moveit_pro_mobile_manipulation/bring_it_sim/description/picknik_ur_mujoco_ros2_control.xacro (robot description, xacro)
@@ -82,4 +82,5 @@
           <param name="odom_zero_z">true</param>
           <param name="mujoco_viewer">true</param>
+          <param name="mujoco_keyframe">default</param>
       </hardware>
     </ros2_control>

File: src/moveit_pro_mobile_manipulation/bring_it_sim/description/vacuum_urdf.xacro (robot description, xacro)
@@ -15,36 +15,18 @@
         </geometry>
       </visual>
+    </link>
+    <link name="collision_vacuum_base">
       <collision>
         <origin rpy="0.0 0.0 0.0" xyz="0.0 0.0 0.0"/>
         <geometry>
-          <mesh filename="package://bring_it_sim/description/assets/vacuum_base.obj" scale="1.0 1.0 1.0"/>
-        </geometry>
-      </collision>
-    </link>
-    <link name="collision_vacuum_base">
-      <visual>
-        <origin rpy="0.0 -0.0 0.0" xyz="2.925628969631447e-17 0.09096898138523102 0.0491398349404335"/>
-        <geometry>
-          <mesh filename="package://bring_it_sim/description/assets/collision_vacuum_base.obj" scale="0.09352162480354309 0.13757896423339844 0.02057690918445587"/>
-        </geometry>
-      </visual>
-      <collision>
-        <origin rpy="0.0 -0.0 0.0" xyz="2.925628969631447e-17 0.09096898138523102 0.0491398349404335"/>
-        <geometry>
-          <mesh filename="package://bring_it_sim/description/assets/collision_vacuum_base.obj" scale="0.09352162480354309 0.13757896423339844 0.02057690918445587"/>
+          <mesh filename="package://bring_it_sim/description/assets/collision_vacuum_base.obj" scale="1.0 1.0 1.0"/>
         </geometry>
       </collision>
     </link>
     <link name="collision_vacuum_suction_cups">
-      <visual>
-        <origin rpy="0.0 -0.0 0.0" xyz="2.925628969631447e-17 0.09096898138523102 0.13839076459407806"/>
+      <collision>
+        <origin rpy="0.0 0.0 0.0" xyz="0.0 0.0 0.0"/>
         <geometry>
-          <mesh filename="package://bring_it_sim/description/assets/collision_vacuum_suction_cups.obj" scale="0.08370228856801987 0.13757896423339844 0.02057690918445587"/>
-        </geometry>
-      </visual>
-      <collision>
-        <origin rpy="0.0 -0.0 0.0" xyz="2.925628969631447e-17 0.09096898138523102 0.13839076459407806"/>
-        <geometry>
-          <mesh filename="package://bring_it_sim/description/assets/collision_vacuum_suction_cups.obj" scale="0.08370228856801987 0.13757896423339844 0.02057690918445587"/>
+          <mesh filename="package://bring_it_sim/description/assets/collision_vacuum_suction_cups.obj" scale="1.0 1.0 1.0"/>
         </geometry>
       </collision>
@@ -57,10 +39,4 @@
         </geometry>
       </visual>
-      <collision>
-        <origin rpy="0.0 0.0 0.0" xyz="0.0 0.0 0.0"/>
-        <geometry>
-          <mesh filename="package://bring_it_sim/description/assets/vacuum_base_top.obj" scale="1.0 1.0 1.0"/>
-        </geometry>
-      </collision>
     </link>
     <link name="vacuum_suction_cups">
@@ -71,10 +47,4 @@
         </geometry>
       </visual>
-      <collision>
-        <origin rpy="0.0 0.0 0.0" xyz="0.0 0.0 0.0"/>
-        <geometry>
-          <mesh filename="package://bring_it_sim/description/assets/vacuum_suction_cups.obj" scale="1.0 1.0 1.0"/>
-        </geometry>
-      </collision>
     </link>
     <joint name="vacuum_base_collision_vacuum_base_joint" type="fixed">
@@ -98,4 +68,10 @@
       <origin rpy="0.0 0.0 0.0" xyz="0.0 0.0 0.0"/>
     </joint>
+    <link name="grasp_link"/>
+    <joint name="vacuum_suction_cups_grasp_link_joint" type="fixed">
+      <parent link="vacuum_suction_cups"/>
+      <child link="grasp_link"/>
+      <origin rpy="0.0 0.0 0.0" xyz="0.0 0.0 0.1"/>
+    </joint>
   </xacro:macro>
 </robot>

Commit message: velocity control almost working
Signed-off-by: Paul Gesel <paul.gesel@picknik.ai>

File: src/moveit_pro_mobile_manipulation/bring_it_sim/description/picknik_ur_mujoco_ros2_control.xacro (robot description, xacro)
@@ -3,71 +3,71 @@
   <xacro:macro name="picknik_ur_mujoco_ros2_control" params="mujoco_model">
     <ros2_control name="ur_mujoco_control" type="system">
-      <joint name="shoulder_pan_joint">
-          <command_interface name="position">
-          <param name="min">${-2*pi}</param>
-          <param name="max">${2*pi}</param>
-          </command_interface>
-          <state_interface name="position">
-          <param name="initial_value">0.0</param>
-          </state_interface>
-          <state_interface name="velocity"/>
-          <state_interface name="effort"/>
-      </joint>
-      <joint name="shoulder_lift_joint">
-          <command_interface name="position">
-          <param name="min">-2.41</param>
-          <param name="max">2.41</param>
-          <param name="initial_value">-1.57</param>
-          </command_interface>
-          <state_interface name="position">
-          <param name="initial_value">-1.57</param>
-          </state_interface>
-          <state_interface name="velocity"/>
-          <state_interface name="effort"/>
-      </joint>
-      <joint name="elbow_joint">
-          <command_interface name="position">
-          <param name="min">${-2*pi}</param>
-          <param name="max">${2*pi}</param>
-          </command_interface>
-          <state_interface name="position">
-          <param name="initial_value">-3.14</param>
-          </state_interface>
-          <state_interface name="velocity"/>
-          <state_interface name="effort"/>
-      </joint>
-      <joint name="wrist_1_joint">
-          <command_interface name="position">
-          <param name="min">-2.66</param>
-          <param name="max">2.66</param>
-          </command_interface>
-          <state_interface name="position">
-          <param name="initial_value">-2.51</param>
-          </state_interface>
-          <state_interface name="velocity"/>
-          <state_interface name="effort"/>
-      </joint>
-      <joint name="wrist_2_joint">
-          <command_interface name="position">
-          <param name="min">${-2*pi}</param>
-          <param name="max">${2*pi}</param>
-          </command_interface>
-          <state_interface name="position">
-          <param name="initial_value">0.0</param>
-          </state_interface>
-          <state_interface name="velocity"/>
-          <state_interface name="effort"/>
-      </joint>
-      <joint name="wrist_3_joint">
-          <command_interface name="position">
-          <param name="min">-2.23</param>
-          <param name="max">2.23</param>
-          </command_interface>
-          <state_interface name="position">
-          <param name="initial_value">0.96</param>
-          </state_interface>
-          <state_interface name="velocity"/>
-          <state_interface name="effort"/>
-      </joint>
+<!--      <joint name="shoulder_pan_joint">-->
+<!--          <command_interface name="position">-->
+<!--          <param name="min">${-2*pi}</param>-->
+<!--          <param name="max">${2*pi}</param>-->
+<!--          </command_interface>-->
+<!--          <state_interface name="position">-->
+<!--          <param name="initial_value">0.0</param>-->
+<!--          </state_interface>-->
+<!--          <state_interface name="velocity"/>-->
+<!--          <state_interface name="effort"/>-->
+<!--      </joint>-->
+<!--      <joint name="shoulder_lift_joint">-->
+<!--          <command_interface name="position">-->
+<!--          <param name="min">-2.41</param>-->
+<!--          <param name="max">2.41</param>-->
+<!--          <param name="initial_value">-1.57</param>-->
+<!--          </command_interface>-->
+<!--          <state_interface name="position">-->
+<!--          <param name="initial_value">-1.57</param>-->
+<!--          </state_interface>-->
+<!--          <state_interface name="velocity"/>-->
+<!--          <state_interface name="effort"/>-->
+<!--      </joint>-->
+<!--      <joint name="elbow_joint">-->
+<!--          <command_interface name="position">-->
+<!--          <param name="min">${-2*pi}</param>-->
+<!--          <param name="max">${2*pi}</param>-->
+<!--          </command_interface>-->
+<!--          <state_interface name="position">-->
+<!--          <param name="initial_value">-3.14</param>-->
+<!--          </state_interface>-->
+<!--          <state_interface name="velocity"/>-->
+<!--          <state_interface name="effort"/>-->
+<!--      </joint>-->
+<!--      <joint name="wrist_1_joint">-->
+<!--          <command_interface name="position">-->
+<!--          <param name="min">-2.66</param>-->
+<!--          <param name="max">2.66</param>-->
+<!--          </command_interface>-->
+<!--          <state_interface name="position">-->
+<!--          <param name="initial_value">-2.51</param>-->
+<!--          </state_interface>-->
+<!--          <state_interface name="velocity"/>-->
+<!--          <state_interface name="effort"/>-->
+<!--      </joint>-->
+<!--      <joint name="wrist_2_joint">-->
+<!--          <command_interface name="position">-->
+<!--          <param name="min">${-2*pi}</param>-->
+<!--          <param name="max">${2*pi}</param>-->
+<!--          </command_interface>-->
+<!--          <state_interface name="position">-->
+<!--          <param name="initial_value">0.0</param>-->
+<!--          </state_interface>-->
+<!--          <state_interface name="velocity"/>-->
+<!--          <state_interface name="effort"/>-->
+<!--      </joint>-->
+<!--      <joint name="wrist_3_joint">-->
+<!--          <command_interface name="position">-->
+<!--          <param name="min">-2.23</param>-->
+<!--          <param name="max">2.23</param>-->
+<!--          </command_interface>-->
+<!--          <state_interface name="position">-->
+<!--          <param name="initial_value">0.96</param>-->
+<!--          </state_interface>-->
+<!--          <state_interface name="velocity"/>-->
+<!--          <state_interface name="effort"/>-->
+<!--      </joint>-->
       <hardware>
           <plugin>picknik_mujoco_ros/MujocoSystem</plugin>
@@ -77,5 +77,5 @@
           <param name="tf_publish_rate">60</param>
           <param name="lidar_publish_rate">10</param>
-          <param name="ignore_joint_validation">linear_x_joint linear_y_joint rotational_yaw_joint</param>
+<!--          <param name="ignore_joint_validation">linear_x_joint linear_y_joint rotational_yaw_joint</param>-->
           <param name="publish_odom">true</param>
           <param name="odom_child_frame">ridgeback_base_link</param>
