Commit message: URDF working in UI!
Signed-off-by: Paul Gesel <paul.gesel@picknik.ai>

File: src/moveit_pro_mobile_manipulation/bring_it_sim/description/hangar_urdf.xacro (robot description, xacro)
@@ -23,925 +23,529 @@
     </joint>
     <link name="collision_SM_Floor_376">
-      <visual>
-        <origin rpy="0.0 -0.0 0.0" xyz="0.0 25.808658599853516 -0.5"/>
+      <collision>
+        <origin rpy="0.0 0.0 0.0" xyz="0.0 25.80866050720215 -0.5"/>
         <geometry>
           <mesh filename="package://bring_it_sim/description/assets/hangar_mesh/collision_SM_Floor_376.obj" scale="1.0 1.0 1.0"/>
         </geometry>
-      </visual>
-      <collision>
-        <origin rpy="0.0 -0.0 0.0" xyz="0.0 25.808658599853516 -0.5"/>
-        <geometry>
-          <mesh filename="package://bring_it_sim/description/assets/hangar_mesh/collision_SM_Floor_376.obj" scale="1.0 1.0 1.0"/>
-        </geometry>
       </collision>
     </link>
     <link name="collision_Cube">
-      <visual>
-        <origin rpy="0.0 -0.0 0.0" xyz="7.231803894042969 -12.968038558959961 1.2229089736938477"/>
+      <collision>
+        <origin rpy="0.0 0.0 0.0" xyz="7.231803894042969 -12.968037605285645 1.2229089736938477"/>
         <geometry>
           <mesh filename="package://bring_it_sim/description/assets/hangar_mesh/collision_Cube.obj" scale="1.0 1.0 1.0"/>
         </geometry>
-      </visual>
-      <collision>
-        <origin rpy="0.0 -0.0 0.0" xyz="7.231803894042969 -12.968038558959961 1.2229089736938477"/>
-        <geometry>
-          <mesh filename="package://bring_it_sim/description/assets/hangar_mesh/collision_Cube.obj" scale="1.0 1.0 1.0"/>
-        </geometry>
       </collision>
     </link>
     <link name="collision_Cube_001">
-      <visual>
-        <origin rpy="0.0 -0.0 0.0" xyz="11.559599876403809 -16.500215530395508 1.300389289855957"/>
+      <collision>
+        <origin rpy="0.0 0.0 0.0" xyz="11.559602737426758 -16.50021743774414 1.300389289855957"/>
         <geometry>
           <mesh filename="package://bring_it_sim/description/assets/hangar_mesh/collision_Cube_001.obj" scale="1.0 1.0 1.0"/>
         </geometry>
-      </visual>
-      <collision>
-        <origin rpy="0.0 -0.0 0.0" xyz="11.559599876403809 -16.500215530395508 1.300389289855957"/>
-        <geometry>
-          <mesh filename="package://bring_it_sim/description/assets/hangar_mesh/collision_Cube_001.obj" scale="1.0 1.0 1.0"/>
-        </geometry>
       </collision>
     </link>
     <link name="collision_Cube_002">
-      <visual>
-        <origin rpy="0.0 -0.0 0.0" xyz="-19.290809631347656 -9.404718399047852 1.300389289855957"/>
+      <collision>
+        <origin rpy="0.0 0.0 0.0" xyz="-19.29080581665039 -9.404716491699219 1.300389289855957"/>
         <geometry>
           <mesh filename="package://bring_it_sim/description/assets/hangar_mesh/collision_Cube_002.obj" scale="1.0 1.0 1.0"/>
         </geometry>
-      </visual>
-      <collision>
-        <origin rpy="0.0 -0.0 0.0" xyz="-19.290809631347656 -9.404718399047852 1.300389289855957"/>
-        <geometry>
-          <mesh filename="package://bring_it_sim/description/assets/hangar_mesh/collision_Cube_002.obj" scale="1.0 1.0 1.0"/>
-        </geometry>
       </collision>
     </link>
     <link name="collision_Cube_004">
-      <visual>
-        <origin rpy="0.0 -0.0 0.0" xyz="-22.695959091186523 -17.61707305908203 1.300389289855957"/>
+      <collision>
+        <origin rpy="0.0 0.0 0.0" xyz="-22.69596290588379 -17.617074966430664 1.300389289855957"/>
         <geometry>
           <mesh filename="package://bring_it_sim/description/assets/hangar_mesh/collision_Cube_004.obj" scale="1.0 1.0 1.0"/>
         </geometry>
-      </visual>
-      <collision>
-        <origin rpy="0.0 -0.0 0.0" xyz="-22.695959091186523 -17.61707305908203 1.300389289855957"/>
-        <geometry>
-          <mesh filename="package://bring_it_sim/description/assets/hangar_mesh/collision_Cube_004.obj" scale="1.0 1.0 1.0"/>
-        </geometry>
       </collision>
     </link>
     <link name="collision_Cube_005">
-      <visual>
-        <origin rpy="0.0 -0.0 0.0" xyz="-23.86355972290039 -14.983378410339355 1.4106760025024414"/>
+      <collision>
+        <origin rpy="0.0 0.0 0.0" xyz="-23.86355972290039 -14.983379364013672 1.4106760025024414"/>
         <geometry>
           <mesh filename="package://bring_it_sim/description/assets/hangar_mesh/collision_Cube_005.obj" scale="1.0 1.0 1.0"/>
         </geometry>
-      </visual>
-      <collision>
-        <origin rpy="0.0 -0.0 0.0" xyz="-23.86355972290039 -14.983378410339355 1.4106760025024414"/>
-        <geometry>
-          <mesh filename="package://bring_it_sim/description/assets/hangar_mesh/collision_Cube_005.obj" scale="1.0 1.0 1.0"/>
-        </geometry>
       </collision>
     </link>
     <link name="collision_Cube_006">
-      <visual>
-        <origin rpy="0.0 -0.0 0.0" xyz="-24.01235008239746 -9.977728843688965 1.5179870128631592"/>
+      <collision>
+        <origin rpy="0.0 0.0 0.0" xyz="-24.01235008239746 -9.977728843688965 1.5179872512817383"/>
         <geometry>
           <mesh filename="package://bring_it_sim/description/assets/hangar_mesh/collision_Cube_006.obj" scale="1.0 1.0 1.0"/>
         </geometry>
-      </visual>
-      <collision>
-        <origin rpy="0.0 -0.0 0.0" xyz="-24.01235008239746 -9.977728843688965 1.5179870128631592"/>
-        <geometry>
-          <mesh filename="package://bring_it_sim/description/assets/hangar_mesh/collision_Cube_006.obj" scale="1.0 1.0 1.0"/>
-        </geometry>
       </collision>
     </link>
     <link name="collision_Cube_007">
-      <visual>
-        <origin rpy="0.0 -0.0 0.0" xyz="24.00054931640625 -17.49724006652832 1.5179870128631592"/>
+      <collision>
+        <origin rpy="0.0 0.0 0.0" xyz="24.00054931640625 -17.497241973876953 1.5179872512817383"/>
         <geometry>
           <mesh filename="package://bring_it_sim/description/assets/hangar_mesh/collision_Cube_007.obj" scale="1.0 1.0 1.0"/>
         </geometry>
-      </visual>
-      <collision>
-        <origin rpy="0.0 -0.0 0.0" xyz="24.00054931640625 -17.49724006652832 1.5179870128631592"/>
-        <geometry>
-          <mesh filename="package://bring_it_sim/description/assets/hangar_mesh/collision_Cube_007.obj" scale="1.0 1.0 1.0"/>
-        </geometry>
       </collision>
     </link>
     <link name="collision_Cube_008">
-      <visual>
-        <origin rpy="0.0 -0.0 0.0" xyz="24.14933967590332 -14.472249031066895 1.5179870128631592"/>
+      <collision>
+        <origin rpy="0.0 0.0 0.0" xyz="24.14933967590332 -14.472247123718262 1.5179872512817383"/>
         <geometry>
           <mesh filename="package://bring_it_sim/description/assets/hangar_mesh/collision_Cube_008.obj" scale="1.0 1.0 1.0"/>
         </geometry>
-      </visual>
-      <collision>
-        <origin rpy="0.0 -0.0 0.0" xyz="24.14933967590332 -14.472249031066895 1.5179870128631592"/>
-        <geometry>
-          <mesh filename="package://bring_it_sim/description/assets/hangar_mesh/collision_Cube_008.obj" scale="1.0 1.0 1.0"/>
-        </geometry>
       </collision>
     </link>
     <link name="collision_Cube_009">
-      <visual>
-        <origin rpy="0.0 -0.0 0.0" xyz="24.14933967590332 -9.992018699645996 1.5179870128631592"/>
+      <collision>
+        <origin rpy="0.0 0.0 0.0" xyz="24.14933967590332 -9.992019653320312 1.5179872512817383"/>
         <geometry>
           <mesh filename="package://bring_it_sim/description/assets/hangar_mesh/collision_Cube_009.obj" scale="1.0 1.0 1.0"/>
         </geometry>
-      </visual>
-      <collision>
-        <origin rpy="0.0 -0.0 0.0" xyz="24.14933967590332 -9.992018699645996 1.5179870128631592"/>
-        <geometry>
-          <mesh filename="package://bring_it_sim/description/assets/hangar_mesh/collision_Cube_009.obj" scale="1.0 1.0 1.0"/>
-        </geometry>
       </collision>
     </link>
     <link name="collision_Cube_010">
-      <visual>
-        <origin rpy="0.0 -0.0 0.0" xyz="-23.473468780517578 5.198320388793945 1.300389289855957"/>
+      <collision>
+        <origin rpy="0.0 0.0 0.0" xyz="-23.473466873168945 5.19831657409668 1.300389289855957"/>
         <geometry>
           <mesh filename="package://bring_it_sim/description/assets/hangar_mesh/collision_Cube_010.obj" scale="1.0 1.0 1.0"/>
         </geometry>
-      </visual>
-      <collision>
-        <origin rpy="0.0 -0.0 0.0" xyz="-23.473468780517578 5.198320388793945 1.300389289855957"/>
-        <geometry>
-          <mesh filename="package://bring_it_sim/description/assets/hangar_mesh/collision_Cube_010.obj" scale="1.0 1.0 1.0"/>
-        </geometry>
       </collision>
     </link>
     <link name="collision_Cube_011">
-      <visual>
-        <origin rpy="0.0 -0.0 0.0" xyz="-23.901168823242188 6.610160827636719 1.300389289855957"/>
+      <collision>
+        <origin rpy="0.0 0.0 0.0" xyz="-23.901172637939453 6.610162734985352 1.300389289855957"/>
         <geometry>
           <mesh filename="package://bring_it_sim/description/assets/hangar_mesh/collision_Cube_011.obj" scale="1.0 1.0 1.0"/>
         </geometry>
-      </visual>
-      <collision>
-        <origin rpy="0.0 -0.0 0.0" xyz="-23.901168823242188 6.610160827636719 1.300389289855957"/>
-        <geometry>
-          <mesh filename="package://bring_it_sim/description/assets/hangar_mesh/collision_Cube_011.obj" scale="1.0 1.0 1.0"/>
-        </geometry>
       </collision>
     </link>
     <link name="collision_Cube_012">
-      <visual>
-        <origin rpy="0.0 -0.0 0.0" xyz="-24.305639266967773 1.2454605102539062 0.9974985122680664"/>
+      <collision>
+        <origin rpy="0.0 0.0 0.0" xyz="-24.305641174316406 1.2454547882080078 0.9974985122680664"/>
         <geometry>
           <mesh filename="package://bring_it_sim/description/assets/hangar_mesh/collision_Cube_012.obj" scale="0.9999999403953552 0.9999999403953552 1.0"/>
         </geometry>
-      </visual>
-      <collision>
-        <origin rpy="0.0 -0.0 0.0" xyz="-24.305639266967773 1.2454605102539062 0.9974985122680664"/>
-        <geometry>
-          <mesh filename="package://bring_it_sim/description/assets/hangar_mesh/collision_Cube_012.obj" scale="0.9999999403953552 0.9999999403953552 1.0"/>
-        </geometry>
       </collision>
     </link>
     <link name="collision_Cube_013">
-      <visual>
-        <origin rpy="0.0 -0.0 0.0" xyz="24.258668899536133 3.9001903533935547 0.9974985122680664"/>
+      <collision>
+        <origin rpy="0.0 0.0 0.0" xyz="24.2586669921875 3.900186538696289 0.9974985122680664"/>
         <geometry>
           <mesh filename="package://bring_it_sim/description/assets/hangar_mesh/collision_Cube_013.obj" scale="0.9999999403953552 0.9999999403953552 1.0"/>
         </geometry>
-      </visual>
-      <collision>
-        <origin rpy="0.0 -0.0 0.0" xyz="24.258668899536133 3.9001903533935547 0.9974985122680664"/>
-        <geometry>
-          <mesh filename="package://bring_it_sim/description/assets/hangar_mesh/collision_Cube_013.obj" scale="0.9999999403953552 0.9999999403953552 1.0"/>
-        </geometry>
       </collision>
     </link>
     <link name="collision_Cube_014">
-      <visual>
-        <origin rpy="0.0 -0.0 0.0" xyz="24.258668899536133 4.701450347900391 0.9974985122680664"/>
+      <collision>
+        <origin rpy="0.0 0.0 0.0" xyz="24.2586669921875 4.701450347900391 0.9974985122680664"/>
         <geometry>
           <mesh filename="package://bring_it_sim/description/assets/hangar_mesh/collision_Cube_014.obj" scale="0.9999999403953552 0.9999999403953552 1.0"/>
         </geometry>
-      </visual>
-      <collision>
-        <origin rpy="0.0 -0.0 0.0" xyz="24.258668899536133 4.701450347900391 0.9974985122680664"/>
-        <geometry>
-          <mesh filename="package://bring_it_sim/description/assets/hangar_mesh/collision_Cube_014.obj" scale="0.9999999403953552 0.9999999403953552 1.0"/>
-        </geometry>
       </collision>
     </link>
     <link name="collision_Cube_015">
-      <visual>
-        <origin rpy="0.0 -0.0 0.0" xyz="7.401406764984131 28.7860107421875 1.2229089736938477"/>
-        <geometry>
-          <mesh filename="package://bring_it_sim/description/assets/hangar_mesh/collision_Cube_015.obj" scale="1.0 1.0 1.0"/>
-        </geometry>
-      </visual>
-      <collision>
-        <origin rpy="0.0 -0.0 0.0" xyz="7.401406764984131 28.7860107421875 1.2229089736938477"/>
-        <geometry>
-          <mesh filename="package://bring_it_sim/description/assets/hangar_mesh/collision_Cube_015.obj" scale="1.0 1.0 1.0"/>
+      <collision>
+        <origin rpy="0.0 0.0 0.0" xyz="7.401407241821289 28.786008834838867 1.2229089736938477"/>
+        <geometry>
+          <mesh filename="package://bring_it_sim/description/assets/hangar_mesh/collision_Cube_015.obj" scale="1.0000001192092896 1.0000001192092896 1.0"/>
         </geometry>
       </collision>
     </link>
     <link name="collision_Plane">
-      <visual>
-        <origin rpy="0.0 -0.0 0.0" xyz="0.0 0.0 0.5"/>
+      <collision>
+        <origin rpy="0.0 0.0 0.0" xyz="0.0 0.0 0.5"/>
         <geometry>
           <mesh filename="package://bring_it_sim/description/assets/hangar_mesh/collision_Plane.obj" scale="1.0 1.0 1.0"/>
         </geometry>
-      </visual>
-      <collision>
-        <origin rpy="0.0 -0.0 0.0" xyz="0.0 0.0 0.5"/>
-        <geometry>
-          <mesh filename="package://bring_it_sim/description/assets/hangar_mesh/collision_Plane.obj" scale="1.0 1.0 1.0"/>
-        </geometry>
       </collision>
     </link>
     <link name="collision_Plane_001">
-      <visual>
-        <origin rpy="0.0 -0.0 0.0" xyz="0.0 0.0 0.5"/>
+      <collision>
+        <origin rpy="0.0 0.0 0.0" xyz="0.0 0.0 0.5"/>
         <geometry>
           <mesh filename="package://bring_it_sim/description/assets/hangar_mesh/collision_Plane_001.obj" scale="1.0 1.0 1.0"/>
         </geometry>
-      </visual>
-      <collision>
-        <origin rpy="0.0 -0.0 0.0" xyz="0.0 0.0 0.5"/>
-        <geometry>
-          <mesh filename="package://bring_it_sim/description/assets/hangar_mesh/collision_Plane_001.obj" scale="1.0 1.0 1.0"/>
-        </geometry>
       </collision>
     </link>
     <link name="collision_Plane_002">
-      <visual>
-        <origin rpy="0.0 -0.0 0.0" xyz="-2.118288993835449 2.8453807830810547 0.5"/>
+      <collision>
+        <origin rpy="0.0 0.0 0.0" xyz="-2.11828875541687 2.8453807830810547 0.5"/>
         <geometry>
           <mesh filename="package://bring_it_sim/description/assets/hangar_mesh/collision_Plane_002.obj" scale="1.0 1.0 1.0"/>
         </geometry>
-      </visual>
-      <collision>
-        <origin rpy="0.0 -0.0 0.0" xyz="-2.118288993835449 2.8453807830810547 0.5"/>
-        <geometry>
-          <mesh filename="package://bring_it_sim/description/assets/hangar_mesh/collision_Plane_002.obj" scale="1.0 1.0 1.0"/>
-        </geometry>
       </collision>
     </link>
     <link name="collision_Plane_003">
-      <visual>
-        <origin rpy="0.0 -0.0 0.0" xyz="0.02430248074233532 0.0 0.5"/>
+      <collision>
+        <origin rpy="0.0 0.0 0.0" xyz="0.02430248260498047 0.0 0.5"/>
         <geometry>
           <mesh filename="package://bring_it_sim/description/assets/hangar_mesh/collision_Plane_003.obj" scale="1.0 1.0 1.0"/>
         </geometry>
-      </visual>
-      <collision>
-        <origin rpy="0.0 -0.0 0.0" xyz="0.02430248074233532 0.0 0.5"/>
-        <geometry>
-          <mesh filename="package://bring_it_sim/description/assets/hangar_mesh/collision_Plane_003.obj" scale="1.0 1.0 1.0"/>
-        </geometry>
       </collision>
     </link>
     <link name="collision_Plane_004">
-      <visual>
-        <origin rpy="0.0 -0.0 0.0" xyz="2.1425909996032715 2.8453807830810547 0.5"/>
+      <collision>
+        <origin rpy="0.0 0.0 0.0" xyz="2.1425912380218506 2.8453807830810547 0.5"/>
         <geometry>
           <mesh filename="package://bring_it_sim/description/assets/hangar_mesh/collision_Plane_004.obj" scale="1.0 1.0 1.0"/>
         </geometry>
-      </visual>
-      <collision>
-        <origin rpy="0.0 -0.0 0.0" xyz="2.1425909996032715 2.8453807830810547 0.5"/>
-        <geometry>
-          <mesh filename="package://bring_it_sim/description/assets/hangar_mesh/collision_Plane_004.obj" scale="1.0 1.0 1.0"/>
-        </geometry>
       </collision>
     </link>
     <link name="collision_Plane_005">
-      <visual>
-        <origin rpy="0.0 -0.0 0.0" xyz="0.021426009014248848 7.306232452392578 0.5"/>
+      <collision>
+        <origin rpy="0.0 0.0 0.0" xyz="0.021426012739539146 7.306234359741211 0.5"/>
         <geometry>
           <mesh filename="package://bring_it_sim/description/assets/hangar_mesh/collision_Plane_005.obj" scale="1.0 1.0 1.0"/>
         </geometry>
-      </visual>
-      <collision>
-        <origin rpy="0.0 -0.0 0.0" xyz="0.021426009014248848 7.306232452392578 0.5"/>
-        <geometry>
-          <mesh filename="package://bring_it_sim/description/assets/hangar_mesh/collision_Plane_005.obj" scale="1.0 1.0 1.0"/>
-        </geometry>
       </collision>
     </link>
     <link name="collision_Plane_006">
-      <visual>
-        <origin rpy="0.0 -0.0 0.0" xyz="0.021426009014248848 3.1153297424316406 0.5"/>
+      <collision>
+        <origin rpy="0.0 0.0 0.0" xyz="0.021426014602184296 3.115325927734375 0.5"/>
         <geometry>
           <mesh filename="package://bring_it_sim/description/assets/hangar_mesh/collision_Plane_006.obj" scale="1.0 1.0 1.0"/>
         </geometry>
-      </visual>
-      <collision>
-        <origin rpy="0.0 -0.0 0.0" xyz="0.021426009014248848 3.1153297424316406 0.5"/>
-        <geometry>
-          <mesh filename="package://bring_it_sim/description/assets/hangar_mesh/collision_Plane_006.obj" scale="1.0 1.0 1.0"/>
-        </geometry>
       </collision>
     </link>
     <link name="collision_Plane_007">
-      <visual>
-        <origin rpy="0.0 -0.0 0.0" xyz="7.323379039764404 3.269590377807617 0.5"/>
+      <collision>
+        <origin rpy="0.0 0.0 0.0" xyz="7.323379039764404 3.26959228515625 0.5"/>
         <geometry>
           <mesh filename="package://bring_it_sim/description/assets/hangar_mesh/collision_Plane_007.obj" scale="1.0 1.0 1.0"/>
         </geometry>
-      </visual>
-      <collision>
-        <origin rpy="0.0 -0.0 0.0" xyz="7.323379039764404 3.269590377807617 0.5"/>
-        <geometry>
-          <mesh filename="package://bring_it_sim/description/assets/hangar_mesh/collision_Plane_007.obj" scale="1.0 1.0 1.0"/>
-        </geometry>
       </collision>
     </link>
     <link name="collision_Plane_008">
-      <visual>
-        <origin rpy="0.0 -0.0 0.0" xyz="-7.353374004364014 3.269590377807617 0.5"/>
+      <collision>
+        <origin rpy="0.0 0.0 0.0" xyz="-7.353374481201172 3.26959228515625 0.5"/>
         <geometry>
           <mesh filename="package://bring_it_sim/description/assets/hangar_mesh/collision_Plane_008.obj" scale="1.0 1.0 1.0"/>
         </geometry>
-      </visual>
-      <collision>
-        <origin rpy="0.0 -0.0 0.0" xyz="-7.353374004364014 3.269590377807617 0.5"/>
-        <geometry>
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
Commit message: replace robotiq with vacuum
Signed-off-by: Paul Gesel <paul.gesel@picknik.ai>

File: src/moveit_pro_mobile_manipulation/bring_it_sim/description/hangar_urdf.xacro (robot description, xacro)
@@ -2,5 +2,5 @@
 <robot xmlns:xacro="http://ros.org/wiki/xacro">
   <xacro:macro name="hangar_urdf" params="parent">
-    <!-- connect collisions to parent frmae, e.g. world frame -->
+    <!-- connect collisions to parent frame, e.g. world frame -->
     <joint name="parent_collision_SM_Floor_376_joint" type="fixed">
       <parent link="${parent}"/>

File: src/moveit_pro_mobile_manipulation/bring_it_sim/description/picknik_ur_mujoco_ros2_control.xacro (robot description, xacro)
@@ -70,15 +70,4 @@
           <state_interface name="effort"/>
       </joint>
-      <joint name="robotiq_85_left_knuckle_joint">
-          <command_interface name="position"/>
-          <state_interface name="position">
-          <param name="initial_value">0.7929</param>
-          </state_interface>
-          <state_interface name="velocity"/>
-      </joint>
-      <joint name="robotiq_85_right_knuckle_joint">
-          <state_interface name="position"/>
-          <state_interface name="velocity"/>
-      </joint>
       <hardware>
           <plugin>picknik_mujoco_ros/MujocoSystem</plugin>

File: src/moveit_pro_mobile_manipulation/bring_it_sim/description/ur5e_ridgeback.xacro (robot description, xacro)
@@ -25,9 +25,10 @@
   <xacro:include filename="$(find ridgeback_description)/urdf/ridgeback.urdf.xacro"/>
   <xacro:include filename="$(find bring_it_sim)/description/hangar_urdf.xacro"/>
+  <xacro:include filename="$(find bring_it_sim)/description/vacuum_urdf.xacro"/>
   <link name="world"/>
   <!-- Hangar  -->
   <xacro:hangar_urdf parent="world"/>
   <!-- Gripper and UR adapter and realsense camera -->
-  <xacro:picknik_ur_attachments parent="tool0" child="grasp_link" has_tool_changer="$(arg has_tool_changer)"/>
+<!--  <xacro:picknik_ur_attachments parent="tool0" child="grasp_link" has_tool_changer="$(arg has_tool_changer)"/>-->
   <!-- Ridgeback -->
   <xacro:ridgeback parent="ridgeback_base_link"/>
@@ -89,4 +90,5 @@
     <origin xyz="0 0.0 0.0" rpy="0 0 0" />
   </xacro:picknik_ur>
+  <xacro:vacuum_urdf parent="tool0"/>
   <!-- MuJoCo Hardware interface -->
   <xacro:picknik_ur_mujoco_ros2_control mujoco_model="$(arg mujoco_model)"/>

Commit message: add ICP behavior
Signed-off-by: Paul Gesel <paul.gesel@picknik.ai>

File: src/moveit_pro_mobile_manipulation/bring_it_sim/description/hangar_urdf.xacro (robot description, xacro)
@@ -25,7 +25,7 @@
       <collision>
         <origin rpy="0.0 0.0 0.0" xyz="0.0 25.80866050720215 -0.5"/>
-        <geometry>
-          <mesh filename="package://bring_it_sim/description/assets/hangar_mesh/collision_SM_Floor_376.obj" scale="1.0 1.0 1.0"/>
-        </geometry>
+<!--        <geometry>-->
+<!--          <mesh filename="package://bring_it_sim/description/assets/hangar_mesh/collision_SM_Floor_376.obj" scale="1.0 1.0 1.0"/>-->
+<!--        </geometry>-->
       </collision>
     </link>
