Commit message: rename to factory sim

File: src/factory_sim/description/fanuc_lrmate200id.ros2_control.xacro (robot description, xacro)
@@ -26,5 +26,5 @@
           <plugin>picknik_mujoco_ros/MujocoSystem</plugin>
           <param name="mujoco_model">$(arg mujoco_model)</param>
-          <param name="mujoco_model_package">fanuc_sim</param>
+          <param name="mujoco_model_package">factory_sim</param>
           <param name="mujoco_viewer">$(arg mujoco_viewer)</param>
           <param name="render_publish_rate">10</param>

File: src/factory_sim/description/fanuc_materials.xacro (robot description, xacro)
@@ -2,5 +2,5 @@
 <robot xmlns:xacro="http://wiki.ros.org/xacro">
   <xacro:include
-    filename="$(find fanuc_sim)/description/fanuc_colours.xacro"
+    filename="$(find factory_sim)/description/fanuc_colours.xacro"
   />
   <xacro:macro name="material_fanuc_yellow">

File: src/factory_sim/description/lrmate200id_macro.xacro (robot description, xacro)
@@ -2,5 +2,5 @@
 <robot xmlns:xacro="http://wiki.ros.org/xacro">
   <xacro:include
-    filename="$(find fanuc_sim)/description/fanuc_materials.xacro"
+    filename="$(find factory_sim)/description/fanuc_materials.xacro"
   />
   <xacro:macro name="fanuc_lrmate200id" params="prefix">

File: src/factory_sim/description/picknik_fanuc.xacro (robot description, xacro)
@@ -3,13 +3,14 @@
   <xacro:arg
     name="initial_positions_file"
-    default="$(find fanuc_sim)/config/initial_positions.yaml"
+    default="$(find factory_sim)/config/initial_positions.yaml"
   />
   <xacro:arg name="hardware_interface" default="mock" />
   <xacro:arg name="mujoco_model" default="description/scene.xml" />
+  <!-- <param name="mujoco_viewer">true</param> -->
   <xacro:include
-    filename="$(find fanuc_sim)/description/lrmate200id_macro.xacro"
+    filename="$(find factory_sim)/description/lrmate200id_macro.xacro"
   />
   <xacro:include
-    filename="$(find fanuc_sim)/description/fanuc_lrmate200id.ros2_control.xacro"
+    filename="$(find factory_sim)/description/fanuc_lrmate200id.ros2_control.xacro"
   />
   <link name="world"/>
@@ -37,5 +38,5 @@
     <parent link="world" />
     <child link="arm_pedestal" />
-    <origin rpy="0 0 0" xyz="0 0.3 0.15" />
+    <origin rpy="0 0 0" xyz="0 0 0.15" />
   </joint>
   <joint name="base_joint" type="fixed">
@@ -44,5 +45,5 @@
     <origin rpy="0 0 0" xyz="0 0 0.15" />
   </joint>
-  <link name="table">
+  <!-- <link name="table">
     <visual>
       <origin rpy="0 0 0" xyz="0 0 0" />
@@ -65,4 +66,32 @@
     <child link="table" />
     <origin rpy="0 0 0" xyz="0 1 0.45" />
+  </joint> -->
+  <link name="convex_bowl">
+    <visual>
+      <origin rpy="0 0 0" xyz="0 0 0" />
+      <geometry>
+            <!-- <mesh filename="package://picknik_accessories/mujoco_assets/assets/bowl.stl"/> -->
+            <mesh filename="package://picknik_accessories/mujoco_assets/assets/bowl_concave_hemisphere.stl"/>
+      </geometry>
+    </visual>
+  </link>
+  <joint name="convex_bowl_joint" type="fixed">
+    <parent link="world" />
+    <child link="convex_bowl" />
+    <origin rpy="0 1.5707 0" xyz="0.65 0.2 0.9" />
+  </joint>
+  <link name="concave_bowl">
+    <visual>
+      <origin rpy="0 0 0" xyz="0 0 0" />
+      <geometry>
+            <!-- <mesh filename="package://picknik_accessories/mujoco_assets/assets/bowl.stl"/> -->
+            <mesh filename="package://picknik_accessories/mujoco_assets/assets/bowl_convex_hemisphere.stl"/>
+      </geometry>
+    </visual>
+  </link>
+  <joint name="concave_bowl_joint" type="fixed">
+    <parent link="world" />
+    <child link="concave_bowl" />
+    <origin rpy="0 -1.5707 0" xyz="0.75 -0.2 0.9" />
   </joint>
   <xacro:fanuc_lrmate200id prefix="" />
