Commit message: Add new tool changing Objectives
Former-commit-id: ac93095229137ecd784adc8e7b8e58c561f8edfb

File: src/factory_sim/description/inspection_tool.urdf (robot description, URDF)
Before this commit: robot fanuc_tool, 2 links, 1 joints
Links:
- removed link gripper_base
- removed link suction_cylinder
- added link inspection_cylinder; collision box size=0.01 0.01 0.03; visual box size=0.01 0.01 0.03
- added link inspection_tool_base; collision box size=0.06 0.06 0.04; visual box size=0.06 0.06 0.04
Joints:
- joint base_joint: child suction_cylinder -> inspection_cylinder; parent gripper_base -> inspection_tool_base

File: src/factory_sim/description/picknik_fanuc.xacro (robot description, xacro)
@@ -23,5 +23,5 @@
     </visual>
     <visual>
-      <origin rpy="0 0 0" xyz="0.23 0.03 0.1" />
+      <origin rpy="0 0 0" xyz="0.23 0.05 0.1" />
       <geometry>
         <box size="0.12 0.02 0.02" />
@@ -29,5 +29,17 @@
     </visual>
     <visual>
-      <origin rpy="0 0 0" xyz="0.23 -0.03 0.1" />
+      <origin rpy="0 0 0" xyz="0.23 0.11 0.1" />
+      <geometry>
+        <box size="0.12 0.02 0.02" />
+      </geometry>
+    </visual>
+    <visual>
+      <origin rpy="0 0 0" xyz="0.23 -0.05 0.1" />
+      <geometry>
+        <box size="0.12 0.02 0.02" />
+      </geometry>
+    </visual>
+    <visual>
+      <origin rpy="0 0 0" xyz="0.23 -0.11 0.1" />
       <geometry>
         <box size="0.12 0.02 0.02" />
