Commit message: Update configs to inherit "Request Teleoperation" core objective
Except for hangar_sim which requires link_padding to be 0.0 since the
shoulder of the arm is near the base.


Former-commit-id: 0e0f097ea131fbe126a3fd8289de08de197eb802

File: src/factory_sim/description/picknik_fanuc.xacro (robot description, xacro)
@@ -97,3 +97,10 @@
     mujoco_viewer="$(arg mujoco_viewer)"
   />
+  <!-- Create a grasp link at the tool so we can inherit default teleop objectives -->
+  <link name="grasp_link"/>
+  <joint name="grasp_link_joint" type="fixed">
+    <origin rpy="0 0 0" xyz="0.0 0.0 0.0"/>
+    <parent link="tool0"/>
+    <child link="grasp_link"/>
+  </joint>
 </robot>

File: src/grinding_sim/description/ur20.urdf (robot description, URDF)
Before this commit: robot ur20, 18 links, 17 joints
Links:
- removed link tool_tip
- added link grasp_link
Joints:
- removed joint tool_tip_joint
- added joint grasp_link_joint: type fixed, parent tool0, child grasp_link, origin xyz=0.0 0.0 0.0 rpy=0 0 0

Commit message: feat(factory_sim): improve sim and 3D viewer visuals
MuJoCo scene: remove gradient skybox, switch floor to a blue checker tile, add anti-aliasing/shadow render-quality settings, and color the arm pedestal with a dark-metal material. URDF: give the pedestal the matching material so the web 3D viewer renders it consistently.

File: src/factory_sim/description/picknik_fanuc.xacro (robot description, xacro)
@@ -14,4 +14,7 @@
     filename="$(find factory_sim)/description/fanuc_lrmate200id.ros2_control.xacro"
   />
+  <material name="pedestal_metal">
+    <color rgba="0.30 0.32 0.35 1.0" />
+  </material>
   <link name="world"/>
   <link name="arm_pedestal">
@@ -21,4 +24,5 @@
         <box size="0.4 0.4 0.3" />
       </geometry>
+      <material name="pedestal_metal" />
     </visual>
     <visual>
@@ -27,4 +31,5 @@
         <box size="0.12 0.02 0.02" />
       </geometry>
+      <material name="pedestal_metal" />
     </visual>
     <visual>
@@ -33,4 +38,5 @@
         <box size="0.12 0.02 0.02" />
       </geometry>
+      <material name="pedestal_metal" />
     </visual>
     <visual>
@@ -39,4 +45,5 @@
         <box size="0.12 0.02 0.02" />
       </geometry>
+      <material name="pedestal_metal" />
     </visual>
     <visual>
@@ -45,4 +52,5 @@
         <box size="0.12 0.02 0.02" />
       </geometry>
+      <material name="pedestal_metal" />
     </visual>
   </link>
