Commit message: Updated folder names
Former-commit-id: 749164096dfefa6f4e2c7f1427553c0121c7b51b

File: src/grinding_sim/description/ur20.urdf (robot description, URDF)
Before this commit: robot ur20, 18 links, 17 joints
Links:
- link base_link_inertia: geometry collision mesh filename=package://ur_description/meshes/ur20/collision/base.stl; visual mesh filename=package://picknik_accessories/mujoco_assets/grinding_sim_as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
- link forearm_link: geometry collision mesh filename=package://ur_description/meshes/ur20/collision/forearm.stl; visual mesh filename=package://picknik_accessories/mujoco_assets/grinding_sim_as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
- link shoulder_link: geometry collision mesh filename=package://ur_description/meshes/ur20/collision/shoulder.stl; visual mesh filename=package://picknik_accessories/mujoco_assets/grinding_sim_as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
- link tool0_tool: geometry collision mesh filename=package://picknik_accessories/mujoco_assets/grinding_sim_as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; visual mesh filename=package://picknik_accessories/mujoco_assets/grinding_sim_as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
- link tool_base: geometry collision mesh filename=package://picknik_accessories/mujoco_assets/grinding_sim_as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; visual mesh filename=package://picknik_accessories/mujoco_assets/grinding_sim_as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
- link upper_arm_link: geometry collision mesh filename=package://ur_description/meshes/ur20/collision/upperarm.stl; visual mesh filename=package://picknik_accessories/mujoco_assets/grinding_sim_as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
- link workcell: geometry collision mesh filename=package://picknik_accessories/mujoco_assets/grinding_sim_as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; visual mesh filename=package://picknik_accessories/mujoco_assets/grinding_sim_as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
- link wrist_1_link: geometry collision mesh filename=package://ur_description/meshes/ur20/collision/wrist1.stl; visual mesh filename=package://picknik_accessories/mujoco_assets/grinding_sim_as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
- link wrist_2_link: geometry collision mesh filename=package://ur_description/meshes/ur20/collision/wrist2.stl; visual mesh filename=package://picknik_accessories/mujoco_assets/grinding_sim_as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
- link wrist_3_link: geometry collision mesh filename=package://ur_description/meshes/ur20/collision/wrist3.stl; visual mesh filename=package://picknik_accessories/mujoco_assets/grinding_sim_as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
