Commit message: hangar_sim: rotate grasp link 180 deg
Former-commit-id: e99088738a9f51958680524d516b4077e5da5e9c

File: src/hangar_sim/description/vacuum_urdf.xacro (robot description, xacro)
@@ -46,5 +46,5 @@
       <parent link="vacuum_base"/>
       <child link="grasp_link"/>
-      <origin rpy="0.0 0.0 0.0" xyz="0.0 0.093 0.159"/>
+      <origin rpy="0.0 0.0 3.1415" xyz="0.0 0.093 0.159"/>
     </joint>
   </xacro:macro>
