Commit message: fix linear joints range and joint teleoperate
Former-commit-id: 69bb93c5656ff7b065b804c84026b81eac1751a8

File: src/hangar_sim/description/ur5e_ridgeback.xacro (robot description, xacro)
@@ -65,5 +65,5 @@
     <child link="virtual_rail_link_1" />
     <origin xyz="0 0 0" rpy="0 0 0" />
-    <limit effort="1000.0" lower="-100.0" upper="100.0" velocity="0.175" acceleration="10.0"/>
+    <limit effort="1000.0" lower="-20.0" upper="20.0" velocity="0.175" acceleration="10.0"/>
     <dynamics damping="20.0" friction="500.0" />
   </joint>
@@ -74,5 +74,5 @@
     <child link="virtual_rail_link_2" />
     <origin xyz="0 0 0" rpy="0 0 0" />
-    <limit effort="1000.0" lower="-100.0" upper="100.0" velocity="0.175" acceleration="10.0"/>
+    <limit effort="1000.0" lower="-5.0" upper="55.0" velocity="0.175" acceleration="10.0"/>
     <dynamics damping="20.0" friction="500.0" />
   </joint>

Commit message: Save progress on getting mobile base jtac control working in hangar_sim
Former-commit-id: dc8628665ed3b7b0358d7326991ad2f21de0db59

File: src/hangar_sim/description/ur5e_ridgeback.xacro (robot description, xacro)
@@ -93,3 +93,16 @@
   <!-- MuJoCo Hardware interface -->
   <xacro:picknik_ur_mujoco_ros2_control mujoco_model="$(arg mujoco_model)"/>
+  <!-- Clearpath control hardware interface for controlling mobile base with a JTC -->
+  <ros2_control name="clearpath_controller_interface" type="system">
+    <hardware>
+      <plugin>clearpath_controller_interface/ClearpathControllerInterface</plugin>
+      <param name="odom_topic">/odom</param>
+      <param name="cmd_vel_topic">/platform_velocity_controller/cmd_vel_unstamped</param>
+      <param name="max_linear_velocity">10</param>
+      <param name="max_angular_velocity">10</param>
+    </hardware>
+    <joint name="linear_x_joint"/>
+    <joint name="linear_y_joint"/>
+    <joint name="rotational_yaw_joint"/>
+  </ros2_control>
 </robot>
