Commit message: fix(hangar_sim): widen linear_x_joint limits to ±25 m
The previous ±20 m limit on linear_x_joint was tighter than the hangar
map (X extent: -25 → +25.4 m), so Navigate to Clicked Point could fail
to reach valid points in the environment.

Refs PickNikRobotics/moveit_pro#18745

Co-Authored-By: Claude Opus 4.7 (1M context) <noreply@anthropic.com>

File: src/hangar_sim/description/ur5e_ridgeback.xacro (robot description, xacro)
@@ -66,5 +66,5 @@
     <child link="virtual_rail_link_1" />
     <origin xyz="0 0 0" rpy="0 0 0" />
-    <limit effort="1000.0" lower="-20.0" upper="20.0" velocity="0.175" acceleration="10.0"/>
+    <limit effort="1000.0" lower="-25.0" upper="25.0" velocity="0.175" acceleration="10.0"/>
     <dynamics damping="20.0" friction="500.0" />
   </joint>

Commit message: fix(hangar_sim): derive the base height from the wheel geometry
Co-Authored-By: Claude Opus 5 <noreply@anthropic.com>

File: src/hangar_sim/description/ur5e_ridgeback.xacro (robot description, xacro)
@@ -69,9 +69,9 @@
     <parent link="world" />
     <child link="virtual_rail_link_1" />
-    <!-- z matches the MJCF base_platform_rotation anchor (pos 0 0 -0.048), which is tuned
-         so the wheels contact the floor (the sim base has no z DOF). Without this offset
-         the robot_state_publisher chain renders the robot 48 mm above where the physics
-         (and every sensor frame) actually put it. -->
-    <origin xyz="0 0 -0.048" rpy="0 0 0" />
+    <!-- Height of the base above the floor, from the wheel geometry: the axle sits
+         axle_offset (0.05) above chassis_link and the wheel radius is 0.0759, so the
+         chassis must ride 0.0259 up for the wheels to touch z = 0. Keep in step with
+         the MJCF base_platform_rotation anchor. -->
+    <origin xyz="0 0 0.0259" rpy="0 0 0" />
     <limit effort="1000.0" lower="-25.0" upper="25.0" velocity="0.175" acceleration="10.0"/>
     <dynamics damping="20.0" friction="500.0" />

Commit message: fix(hangar_sim): ride on the roller envelope, not its peak
Co-Authored-By: Claude Opus 5 <noreply@anthropic.com>

File: src/hangar_sim/description/ur5e_ridgeback.xacro (robot description, xacro)
@@ -69,9 +69,12 @@
     <parent link="world" />
     <child link="virtual_rail_link_1" />
-    <!-- Height of the base above the floor, from the wheel geometry: the axle sits
-         axle_offset (0.05) above chassis_link and the wheel radius is 0.0759, so the
-         chassis must ride 0.0259 up for the wheels to touch z = 0. Keep in step with
-         the MJCF base_platform_rotation anchor. -->
-    <origin xyz="0 0 0.0259" rpy="0 0 0" />
+    <!-- Height of the base above the floor, from the wheel geometry. The roller ring is a
+         ring of N=20 spheres of r=0.010 centred at a=0.0659002081, so its envelope
+         ripples between a+r at each sphere and a*cos(pi/N)+r between them. Ride on
+         the lower figure: the base carries no z DOF, so an anchor set to the peak
+         radius leaves a wheel clear of the floor at every angle but bottom dead
+         centre. anchor = a*cos(pi/N) + r - axle_offset = 0.0750889 - 0.05.
+         Keep in step with the MJCF base_platform_rotation anchor. -->
+    <origin xyz="0 0 0.0250889" rpy="0 0 0" />
     <limit effort="1000.0" lower="-25.0" upper="25.0" velocity="0.175" acceleration="10.0"/>
     <dynamics damping="20.0" friction="500.0" />
