Commit message: Expose mujoco viewer in xacro macro
Former-commit-id: 47184bebc7cbdd11f2c4f8ca73aff9303cbca116

File: src/hangar_sim/description/picknik_ur_mujoco_ros2_control.xacro (robot description, xacro)
@@ -1,5 +1,5 @@
 <?xml version="1.0" encoding="utf-8"?>
 <robot xmlns:xacro="http://ros.org/wiki/xacro">
-  <xacro:macro name="picknik_ur_mujoco_ros2_control" params="mujoco_model">
+  <xacro:macro name="picknik_ur_mujoco_ros2_control" params="mujoco_model mujoco_viewer:=false">
     <ros2_control name="ur_mujoco_control" type="system">
       <hardware>
@@ -13,5 +13,5 @@
           <param name="odom_child_frame">ridgeback_base_link</param>
           <param name="odom_zero_z">true</param>
-<!--          <param name="mujoco_viewer">true</param>-->
+          <param name="mujoco_viewer">${mujoco_viewer}</param>
           <param name="mujoco_keyframe">default</param>
       </hardware>

File: src/hangar_sim/description/ur5e_ridgeback.xacro (robot description, xacro)
@@ -19,4 +19,5 @@
   <xacro:arg name="initial_positions_file" default="$(find picknik_ur_base_config)/config/initial_positions.yaml"/>
   <xacro:arg name="mujoco_model" default="description/bar_scene.xml"/>
+  <xacro:arg name="mujoco_viewer" default="false" />
   <!-- Import UR and environment macros -->
   <xacro:include filename="$(find picknik_ur_base_config)/description/picknik_ur_macro.xacro"/>
@@ -92,4 +93,4 @@
   <xacro:vacuum_urdf parent="tool0"/>
   <!-- MuJoCo Hardware interface -->
-  <xacro:picknik_ur_mujoco_ros2_control mujoco_model="$(arg mujoco_model)"/>
+  <xacro:picknik_ur_mujoco_ros2_control mujoco_model="$(arg mujoco_model)" mujoco_viewer="$(arg mujoco_viewer)"/>
 </robot>
