Commit message: Merge pull request #756 from PickNikRobotics/fix/18174-tf-single-owner-base-link
Fix: Make robot_state_publisher the sole owner of the ridgeback_base_link transform in hangar_sim

File: src/hangar_sim/description/picknik_ur_mujoco_ros2_control.xacro (robot description, xacro)
@@ -23,7 +23,20 @@
           <param name="odom_child_frame">ridgeback_base_link</param>
           <param name="odom_rate">150</param>
-          <param name="odom_zero_z">true</param>
+          <!-- Zero z/roll/pitch in /odom for this planar base. The previous tag here,
+               odom_zero_z, is not a recognized odom publisher parameter and was silently
+               ignored; odom_planar is the real one. -->
+          <param name="odom_planar">true</param>
+          <!-- robot_state_publisher owns the live TF to ridgeback_base_link via the
+               virtual-rail joint chain (driven by MuJoCo's own joint states), so the
+               odom publisher must not broadcast a competing odom -> ridgeback_base_link
+               edge. /odom messages keep flowing for Nav2. -->
+          <param name="odom_publish_tf">false</param>
           <param name="odom_frame">odom</param>
           <param name="publish_mj_world_tf">false</param>
+          <!-- Stop the lidar TF fill-in chain at the robot's base instead of walking to
+               the MJCF worldbody. Without this, MuJoCo broadcasts
+               base_platform -> ridgeback_base_link, a second parent for a frame that
+               robot_state_publisher already publishes. -->
+          <param name="base_link_name">ridgeback_base_link</param>
           <param name="mujoco_viewer">${mujoco_viewer}</param>
           <param name="mujoco_keyframe">default</param>

File: src/hangar_sim/description/ur5e_ridgeback.xacro (robot description, xacro)
@@ -20,5 +20,7 @@
   <xacro:arg name="mujoco_model" default="description/bar_scene.xml"/>
   <xacro:arg name="mujoco_viewer" default="false" />
-  <!-- Set to false when use_fuse:=true so fuse is the sole odom → ridgeback_base_link publisher. -->
+  <!-- Publishes /odom messages for Nav2. The odom → ridgeback_base_link TF edge is never
+       broadcast by MuJoCo (odom_publish_tf is false in the ros2_control macro), so this can
+       stay true regardless of use_fuse. -->
   <xacro:arg name="publish_odom" default="true"/>
   <!-- Import UR and environment macros -->
@@ -67,5 +69,9 @@
     <parent link="world" />
     <child link="virtual_rail_link_1" />
-    <origin xyz="0 0 0" rpy="0 0 0" />
+    <!-- z matches the MJCF base_platform_rotation anchor (pos 0 0 -0.048), which is tuned
+         so the wheels contact the floor (the sim base has no z DOF). Without this offset
+         the robot_state_publisher chain renders the robot 48 mm above where the physics
+         (and every sensor frame) actually put it. -->
+    <origin xyz="0 0 -0.048" rpy="0 0 0" />
     <limit effort="1000.0" lower="-25.0" upper="25.0" velocity="0.175" acceleration="10.0"/>
     <dynamics damping="20.0" friction="500.0" />
