Commit message: fix(hangar_sim): prevent dual odom TF publication when use_fuse:=true
When fuse is enabled it must be the sole publisher of odom ->
ridgeback_base_link. MuJoCo's hardware plugin was also publishing
that edge unconditionally, causing jittery interleaved TF updates.

- Make publish_odom a xacro arg (default true) in the MuJoCo hardware
  xacro and forward it through ur5e_ridgeback.xacro
- Expose publish_odom in config.yaml urdf_params so users can set it
  to false when enabling fuse
- Add a launch-time guard (OpaqueFunction) that shuts down with a clear
  error if use_fuse:=true but publish_odom is still true in config.yaml

Fixes #18174

Co-Authored-By: Claude Sonnet 4.6 <noreply@anthropic.com>

File: src/hangar_sim/description/picknik_ur_mujoco_ros2_control.xacro (robot description, xacro)
@@ -1,5 +1,5 @@
 <?xml version="1.0" encoding="utf-8"?>
 <robot xmlns:xacro="http://ros.org/wiki/xacro">
-  <xacro:macro name="picknik_ur_mujoco_ros2_control" params="mujoco_model mujoco_viewer:=false">
+  <xacro:macro name="picknik_ur_mujoco_ros2_control" params="mujoco_model mujoco_viewer:=false publish_odom:=true">
     <ros2_control name="ur_mujoco_control" type="system">
       <!-- Per-LiDAR topic routing. Sensor names match the MJCF site-name prefix
@@ -20,5 +20,5 @@
           <param name="tf_publish_rate">60</param>
           <param name="lidar_publish_rate">10</param>
-          <param name="publish_odom">true</param>
+          <param name="publish_odom">${publish_odom}</param>
           <param name="odom_child_frame">ridgeback_base_link</param>
           <param name="odom_rate">150</param>

File: src/hangar_sim/description/ur5e_ridgeback.xacro (robot description, xacro)
@@ -20,4 +20,6 @@
   <xacro:arg name="mujoco_model" default="description/bar_scene.xml"/>
   <xacro:arg name="mujoco_viewer" default="false" />
+  <!-- Set to false when use_fuse:=true so fuse is the sole odom → ridgeback_base_link publisher. -->
+  <xacro:arg name="publish_odom" default="true"/>
   <!-- Import UR and environment macros -->
   <xacro:include filename="$(find picknik_ur_base_config)/description/picknik_ur_macro.xacro"/>
@@ -93,4 +95,4 @@
   <xacro:vacuum_urdf parent="tool0"/>
   <!-- MuJoCo Hardware interface -->
-  <xacro:picknik_ur_mujoco_ros2_control mujoco_model="$(arg mujoco_model)" mujoco_viewer="$(arg mujoco_viewer)"/>
+  <xacro:picknik_ur_mujoco_ros2_control mujoco_model="$(arg mujoco_model)" mujoco_viewer="$(arg mujoco_viewer)" publish_odom="$(arg publish_odom)"/>
 </robot>

Commit message: feat(hangar_sim): gate the forward stereo pair behind enable_vo
The forward stereo pair exists for visual odometry and has no consumer yet.
MuJoCo renders every fixed MJCF camera on the render timer whether or not
anything subscribes, so the pair cost two 1280x720 offscreen passes at 20 Hz on
every run, and its four image topics sat in the operator's camera picker ahead
of the wrist and scene cameras.

Add an `enable_vo` xacro arg, off by default. When off, the <sensor> blocks
carry `camera_enabled=false` so the plugin drops the cameras entirely, and the
launch file does not start forward_stereo_publisher. The launch file reads the
flag from config.yaml rather than declaring its own launch argument, so the
cameras cannot render with no publisher.

Publish the renders as /forward_stereo/{left,right}/image_raw so all four image
topics group under one camera-picker entry, and keep the plugin's monocular
camera_info off the ROS sibling name of the image topics: it carries P[3]=0, so
a consumer resolving camera_info by the sibling convention would infer infinite
depth from finite disparity.

The MJCF cameras, mount geometry, calibration and both stereo tests stay in the
tree, so turning this back on is one line rather than a revert.

Requires PickNikRobotics/moveit_pro#22676, which adds `camera_enabled`.

Co-Authored-By: Claude Opus 5 (1M context) <noreply@anthropic.com>

File: src/hangar_sim/description/picknik_ur_mujoco_ros2_control.xacro (robot description, xacro)
@@ -1,5 +1,5 @@
 <?xml version="1.0" encoding="utf-8"?>
 <robot xmlns:xacro="http://ros.org/wiki/xacro">
-  <xacro:macro name="picknik_ur_mujoco_ros2_control" params="mujoco_model mujoco_viewer:=false publish_odom:=true">
+  <xacro:macro name="picknik_ur_mujoco_ros2_control" params="mujoco_model mujoco_viewer:=false publish_odom:=true enable_vo:=false">
     <ros2_control name="ur_mujoco_control" type="system">
       <!-- Per-LiDAR topic routing. Sensor names match the MJCF site-name prefix
@@ -13,17 +13,41 @@
         <param name="topic">/scan_rear</param>
       </sensor>
-      <!-- Move the plugin's per-camera monocular camera_info off the ROS sibling
-           name of the stereo source images. That info carries the same K and
-           frame_id as the stereo contract but P[3]=0, so a consumer resolving
-           camera_info as the sibling of /forward_stereo_right/color would read a
-           zero baseline and infer infinite depth from finite disparity, with
-           nothing to flag the mistake. The calibrated stereo contract is
-           published by forward_stereo_publisher on /forward_stereo/{left,right}/. -->
-      <sensor name="forward_stereo_left">
-        <param name="camera_info_topic">/forward_stereo_left/monocular_camera_info</param>
-      </sensor>
-      <sensor name="forward_stereo_right">
-        <param name="camera_info_topic">/forward_stereo_right/monocular_camera_info</param>
-      </sensor>
+      <!-- The forward stereo pair exists for visual odometry and has no other consumer.
+           Off by default: MuJoCo renders every fixed MJCF camera on the render timer
+           whether or not anything subscribes, so leaving the pair on costs two 1280x720
+           offscreen passes at 20 Hz and puts four image topics in the operator's camera
+           picker that nobody can use. `camera_enabled` drops the cameras from the plugin's
+           configs entirely, so they are neither rendered nor advertised. -->
+      <xacro:unless value="${enable_vo}">
+        <sensor name="forward_stereo_left">
+          <param name="camera_enabled">false</param>
+        </sensor>
+        <sensor name="forward_stereo_right">
+          <param name="camera_enabled">false</param>
+        </sensor>
+      </xacro:unless>
+      <!-- Publish MuJoCo's renders as image_raw inside the same /forward_stereo/{left,right}/
+           namespace as the rectified pair, so all four image topics group under one entry in
+           the operator's camera picker instead of splitting across two top-level names. The
+           renders are an rgb8 simulator artifact with no counterpart on a real OAK-D, whose
+           stereo sensors are monochrome; forward_stereo_publisher converts them to the mono8
+           image_rect pair that is the actual contract. Those rectified names are unchanged.
+           The plugin's per-camera camera_info is kept off the ROS sibling name of both image
+           topics. It carries the same K and frame_id as the stereo contract but P[3]=0, so a
+           consumer resolving camera_info by the sibling convention would read a zero baseline
+           and infer infinite depth from finite disparity, with nothing to flag the mistake.
+           The sibling name now resolves to the calibrated stereo camera_info, which describes
+           these renders correctly too: distortion is zero and rectification is identity, so
+           raw and rectified differ only in encoding. -->
+      <xacro:if value="${enable_vo}">
+        <sensor name="forward_stereo_left">
+          <param name="rgb_topic">/forward_stereo/left/image_raw</param>
+          <param name="camera_info_topic">/forward_stereo/left/monocular_camera_info</param>
+        </sensor>
+        <sensor name="forward_stereo_right">
+          <param name="rgb_topic">/forward_stereo/right/image_raw</param>
+          <param name="camera_info_topic">/forward_stereo/right/monocular_camera_info</param>
+        </sensor>
+      </xacro:if>
       <hardware>
           <plugin>picknik_mujoco_ros/MujocoSystem</plugin>

File: src/hangar_sim/description/ur5e_ridgeback.xacro (robot description, xacro)
@@ -24,4 +24,7 @@
        stay true regardless of use_fuse. -->
   <xacro:arg name="publish_odom" default="true"/>
+  <!-- Renders and publishes the forward stereo pair. Off unless a visual odometry
+       consumer is running; see picknik_ur_mujoco_ros2_control.xacro. -->
+  <xacro:arg name="enable_vo" default="false"/>
   <!-- Import UR and environment macros -->
   <xacro:include filename="$(find picknik_ur_base_config)/description/picknik_ur_macro.xacro"/>
@@ -104,4 +107,4 @@
   <xacro:vacuum_urdf parent="tool0"/>
   <!-- MuJoCo Hardware interface -->
-  <xacro:picknik_ur_mujoco_ros2_control mujoco_model="$(arg mujoco_model)" mujoco_viewer="$(arg mujoco_viewer)" publish_odom="$(arg publish_odom)"/>
+  <xacro:picknik_ur_mujoco_ros2_control mujoco_model="$(arg mujoco_model)" mujoco_viewer="$(arg mujoco_viewer)" publish_odom="$(arg publish_odom)" enable_vo="$(arg enable_vo)"/>
 </robot>
