Commit message: Save progress on getting mobile base jtac control working in hangar_sim

File: src/hangar_sim/description/hangar_urdf.xacro (robot description, xacro)
@@ -876,3 +876,15 @@
     </joint>
   </xacro:macro>
+  <ros2_control name="clearpath_controller_interface" type="system">
+    <hardware>
+      <plugin>clearpath_controller_interface/ClearpathControllerInterface</plugin>
+      <param name="odom_topic">/odom</param>
+      <param name="cmd_vel_topic">/platform_velocity_controller/cmd_vel_unstamped</param>
+      <param name="max_linear_velocity">0.2</param>
+      <param name="max_angular_velocity">0.2</param>
+    </hardware>
+    <joint name="linear_x_joint"/>
+    <joint name="linear_y_joint"/>
+    <joint name="rotational_yaw_joint"/>
+  </ros2_control>
 </robot>

Commit message: Fix Invalid URDF Names

File: src/hangar_sim/description/hangar_urdf.xacro (robot description, xacro)
@@ -156,5 +156,5 @@
       </collision>
     </link>
-    <link name="collision_Cube_002.001">
+    <link name="collision_Cube_002_001">
       <collision>
         <origin rpy="0.0 0.0 0.0" xyz="-11.812490463256836 -22.871850967407228 1.300389289855957"/>
@@ -645,7 +645,7 @@
       <origin rpy="0.0 0.0 0.0" xyz="0.0 25.80866050720215 -0.5"/>
     </joint>
-    <joint name="collision_SM_Floor_376_collision_Cube_002.001_joint" type="fixed">
-      <parent link="collision_SM_Floor_376"/>
-      <child link="collision_Cube_002.001"/>
+    <joint name="collision_SM_Floor_376_collision_Cube_002_001_joint" type="fixed">
+      <parent link="collision_SM_Floor_376"/>
+      <child link="collision_Cube_002_001"/>
       <origin rpy="0.0 0.0 0.0" xyz="0.0 25.80866050720215 -0.5"/>
     </joint>

Commit message: need to change to underscore for collision_cube so does not crash on bring up

File: src/hangar_sim/description/hangar_urdf.xacro (robot description, xacro)
@@ -23,10 +23,10 @@
     </joint>
     <link name="collision_SM_Floor_376">
-      <collision>
+<!--      <collision>-->
         <origin rpy="0.0 0.0 0.0" xyz="0.0 25.80866050720215 -0.5"/>
 <!--        <geometry>-->
 <!--          <mesh filename="package://hangar_sim/description/assets/hangar_mesh/collision_SM_Floor_376.obj" scale="1.0 1.0 1.0"/>-->
 <!--        </geometry>-->
-      </collision>
+<!--      </collision>-->
     </link>
     <link name="collision_Cube">
