Commit message: 17708 Add missing collision and visual geometry to planning scene
Add collision_Cube_002.001 (access stand) and fix collision_Cube
(cart) position in the URDF so the planning scene matches the Mujoco
world. Add visual DAE meshes for both objects and SRDF
disable_collisions entries for the new collision link.

Closes PickNikRobotics/moveit_pro#17708

Co-Authored-By: Claude Opus 4.6 (1M context) <noreply@anthropic.com>

File: src/hangar_sim/description/hangar_urdf.xacro (robot description, xacro)
@@ -32,9 +32,15 @@
     <link name="collision_Cube">
       <collision>
-        <origin rpy="0.0 0.0 0.0" xyz="7.231803894042969 -12.968037605285645 1.2229089736938477"/>
+        <origin rpy="0.0 0.0 0.0" xyz="-11.642203330993652 -23.97299122810723 0.93372729420661926"/>
         <geometry>
           <mesh filename="package://hangar_sim/description/assets/hangar_mesh/collision_Cube.obj" scale="1.0 1.0 1.0"/>
         </geometry>
       </collision>
+      <visual>
+        <origin rpy="0.0 0.0 0.0" xyz="-11.641720771789551 -23.939123630523683 0.9243095517158508"/>
+        <geometry>
+          <mesh filename="package://hangar_sim/description/assets/hangar_mesh/SM_Cart_28.dae" scale="1.0 1.0 1.0"/>
+        </geometry>
+      </visual>
     </link>
     <link name="collision_Cube_001">
@@ -150,4 +156,18 @@
       </collision>
     </link>
+    <link name="collision_Cube_002.001">
+      <collision>
+        <origin rpy="0.0 0.0 0.0" xyz="-11.812490463256836 -22.871850967407228 1.300389289855957"/>
+        <geometry>
+          <mesh filename="package://hangar_sim/description/assets/hangar_mesh/collision_Cube_002.001.obj" scale="1.0 1.0 1.0"/>
+        </geometry>
+      </collision>
+      <visual>
+        <origin rpy="0.0 0.0 3.141592653589793" xyz="-11.796743392944336 -22.872787143707277 1.380396664142609"/>
+        <geometry>
+          <mesh filename="package://hangar_sim/description/assets/hangar_mesh/SM_AccessStand_441.001.dae" scale="1.0 1.0 1.0"/>
+        </geometry>
+      </visual>
+    </link>
     <link name="collision_Plane">
       <collision>
@@ -623,4 +643,9 @@
       <parent link="collision_SM_Floor_376"/>
       <child link="collision_Cube_015"/>
+      <origin rpy="0.0 0.0 0.0" xyz="0.0 25.80866050720215 -0.5"/>
+    </joint>
+    <joint name="collision_SM_Floor_376_collision_Cube_002.001_joint" type="fixed">
+      <parent link="collision_SM_Floor_376"/>
+      <child link="collision_Cube_002.001"/>
       <origin rpy="0.0 0.0 0.0" xyz="0.0 25.80866050720215 -0.5"/>
     </joint>

Commit message: fix(hangar_sim): split large visual mesh into 5 files under 10 MB each
The original hangar_floor.dae (42 MB) triggered a large-mesh warning in the
3D viewer. Split into 5 files by grouping the 89 sub-geometries via bin-packing;
the two largest geometries (landing gear, ~12 MB each) are lightly decimated to
85% faces and exported as OBJ (~3.8 MB each) with the original node matrix
flattened in, the remaining 87 are split across three DAE files (each under
10 MB). Original scene appearance is fully preserved.

Co-Authored-By: Claude Sonnet 4.6 <noreply@anthropic.com>

File: src/hangar_sim/description/hangar_urdf.xacro (robot description, xacro)
@@ -8,16 +8,68 @@
       <origin rpy="0.0 0.0 0.0" xyz="0.0 0.0 0.0"/>
     </joint>
-    <!-- Use single link for visual mesh -->
-    <link name="visual_mesh">
+    <!-- Visual mesh split into 5 files to keep each under 10 MB -->
+    <link name="visual_mesh_00">
       <visual>
         <origin rpy="0.0 0.0 0.0" xyz="0.0 0.0 0.0"/>
         <geometry>
-          <mesh filename="package://hangar_sim/description/assets/hangar_floor.dae" scale="1.0 1.0 1.0"/>
+          <mesh filename="package://hangar_sim/description/assets/hangar_floor_00.obj" scale="1.0 1.0 1.0"/>
         </geometry>
       </visual>
     </link>
-    <joint name="collision_SM_Floor_376_visual_mesh" type="fixed">
-      <parent link="collision_SM_Floor_376"/>
-      <child link="visual_mesh"/>
+    <joint name="collision_SM_Floor_376_visual_mesh_00" type="fixed">
+      <parent link="collision_SM_Floor_376"/>
+      <child link="visual_mesh_00"/>
+      <origin rpy="0.0 0.0 0.0" xyz="0.0 0.0 0.0"/>
+    </joint>
+    <link name="visual_mesh_01">
+      <visual>
+        <origin rpy="0.0 0.0 0.0" xyz="0.0 0.0 0.0"/>
+        <geometry>
+          <mesh filename="package://hangar_sim/description/assets/hangar_floor_01.obj" scale="1.0 1.0 1.0"/>
+        </geometry>
+      </visual>
+    </link>
+    <joint name="collision_SM_Floor_376_visual_mesh_01" type="fixed">
+      <parent link="collision_SM_Floor_376"/>
+      <child link="visual_mesh_01"/>
+      <origin rpy="0.0 0.0 0.0" xyz="0.0 0.0 0.0"/>
+    </joint>
+    <link name="visual_mesh_02">
+      <visual>
+        <origin rpy="0.0 0.0 0.0" xyz="0.0 0.0 0.0"/>
+        <geometry>
+          <mesh filename="package://hangar_sim/description/assets/hangar_floor_02.dae" scale="1.0 1.0 1.0"/>
+        </geometry>
+      </visual>
+    </link>
+    <joint name="collision_SM_Floor_376_visual_mesh_02" type="fixed">
+      <parent link="collision_SM_Floor_376"/>
+      <child link="visual_mesh_02"/>
+      <origin rpy="0.0 0.0 0.0" xyz="0.0 0.0 0.0"/>
+    </joint>
+    <link name="visual_mesh_03">
+      <visual>
+        <origin rpy="0.0 0.0 0.0" xyz="0.0 0.0 0.0"/>
+        <geometry>
+          <mesh filename="package://hangar_sim/description/assets/hangar_floor_03.dae" scale="1.0 1.0 1.0"/>
+        </geometry>
+      </visual>
+    </link>
+    <joint name="collision_SM_Floor_376_visual_mesh_03" type="fixed">
+      <parent link="collision_SM_Floor_376"/>
+      <child link="visual_mesh_03"/>
+      <origin rpy="0.0 0.0 0.0" xyz="0.0 0.0 0.0"/>
+    </joint>
+    <link name="visual_mesh_04">
+      <visual>
+        <origin rpy="0.0 0.0 0.0" xyz="0.0 0.0 0.0"/>
+        <geometry>
+          <mesh filename="package://hangar_sim/description/assets/hangar_floor_04.dae" scale="1.0 1.0 1.0"/>
+        </geometry>
+      </visual>
+    </link>
+    <joint name="collision_SM_Floor_376_visual_mesh_04" type="fixed">
+      <parent link="collision_SM_Floor_376"/>
+      <child link="visual_mesh_04"/>
       <origin rpy="0.0 0.0 0.0" xyz="0.0 0.0 0.0"/>
     </joint>
