Commit message: Add boilerplate for push behavior
Signed-off-by: Paul Gesel <paul.gesel@picknik.ai>

Former-commit-id: 9f806c56662d604677bd877cfea4ea46ca2ce032

File: src/pushing_sim/description/picknik_kinova_gen3.xacro (robot description, xacro)
@@ -287,5 +287,5 @@
       <collision>
         <geometry>
-          <mesh filename="package://robotiq_description/meshes/collision/2f_85/robotiq_base.dae"/>
+          <mesh filename="package://robotiq_description/meshes/collision/2f_85/robotiq_base.stl"/>
         </geometry>
       </collision>
@@ -304,5 +304,5 @@
       <collision>
         <geometry>
-          <mesh filename="package://robotiq_description/meshes/collision/2f_85/left_knuckle.dae"/>
+          <mesh filename="package://robotiq_description/meshes/collision/2f_85/left_knuckle.stl"/>
         </geometry>
       </collision>
@@ -321,5 +321,5 @@
       <collision>
         <geometry>
-          <mesh filename="package://robotiq_description/meshes/collision/2f_85/right_knuckle.dae"/>
+          <mesh filename="package://robotiq_description/meshes/collision/2f_85/right_knuckle.stl"/>
         </geometry>
       </collision>
@@ -338,5 +338,5 @@
       <collision>
         <geometry>
-          <mesh filename="package://robotiq_description/meshes/collision/2f_85/left_finger.dae"/>
+          <mesh filename="package://robotiq_description/meshes/collision/2f_85/left_finger.stl"/>
         </geometry>
       </collision>
@@ -355,5 +355,5 @@
       <collision>
         <geometry>
-          <mesh filename="package://robotiq_description/meshes/collision/2f_85/right_finger.dae"/>
+          <mesh filename="package://robotiq_description/meshes/collision/2f_85/right_finger.stl"/>
         </geometry>
       </collision>
@@ -372,5 +372,5 @@
       <collision>
         <geometry>
-          <mesh filename="package://robotiq_description/meshes/collision/2f_85/left_inner_knuckle.dae"/>
+          <mesh filename="package://robotiq_description/meshes/collision/2f_85/left_inner_knuckle.stl"/>
         </geometry>
       </collision>
@@ -389,5 +389,5 @@
       <collision>
         <geometry>
-          <mesh filename="package://robotiq_description/meshes/collision/2f_85/right_inner_knuckle.dae"/>
+          <mesh filename="package://robotiq_description/meshes/collision/2f_85/right_inner_knuckle.stl"/>
         </geometry>
       </collision>
@@ -406,5 +406,5 @@
       <collision>
         <geometry>
-          <mesh filename="package://robotiq_description/meshes/collision/2f_85/left_finger_tip.dae"/>
+          <mesh filename="package://robotiq_description/meshes/collision/2f_85/left_finger_tip.stl"/>
         </geometry>
         <surface>
@@ -441,5 +441,5 @@
       <collision>
         <geometry>
-          <mesh filename="package://robotiq_description/meshes/collision/2f_85/right_finger_tip.dae"/>
+          <mesh filename="package://robotiq_description/meshes/collision/2f_85/right_finger_tip.stl"/>
         </geometry>
         <surface>
