Commit message: Add camera calibration config and objectives to align with new camera calibration behaviors and how-to guide in Pro.
Former-commit-id: 5f6b7241fa214657cbb125d3f43ac29ec7b1b4e7

File: src/moveit_pro_kinova_configs/space_satellite_sim_camera_cal/description/space_satellite_sim.xacro (robot description, xacro)
@@ -4,5 +4,5 @@
   <xacro:arg name="arm" default="gen3" />
   <xacro:arg name="dof" default="7" />
-  <xacro:arg name="mujoco_keyframe" default="default" />
+  <!-- <xacro:arg name="mujoco_keyframe" default="default" /> -->
   <xacro:arg name="mujoco_model" default="description/mujoco/scene.xml" />
   <xacro:arg name="mujoco_viewer" default="false" />
@@ -536,4 +536,63 @@
     <origin xyz="0 0 0.15" rpy="0 0 0"/>
   </joint>
+  <!-- Calibration tool -->
+  <link name="calibration_tool_link">
+    <visual>
+      <geometry>
+        <mesh filename="file://$(find space_satellite_sim_camera_cal)/description/mujoco/assets/calibration_tool.stl"/>
+      </geometry>
+    </visual>
+  </link>
+  <joint name="calibration_tool_joint" type="fixed">
+    <parent link="robotiq_85_base_link"/>
+    <child link="calibration_tool_link"/>
+    <origin xyz="0 0 0.169" rpy="0 0 0"/>
+  </joint>
+  <link name="calibration_tag_right">
+    <visual>
+      <origin xyz="0 0 0" rpy="0 1.5708 0"/>
+      <geometry>
+        <mesh filename="package://picknik_accessories/descriptions/ar_markers/Marker0.dae" scale=".05 .102 .102"/>
+        <!-- .dae tag side len = 0.5m, and tag size is 0.051m -> scale=0.102m -->
+      </geometry>
+    </visual>
+  </link>
+  <joint name="calibration_tag_right_joint" type="fixed">
+    <parent link="calibration_tool_link"/>
+    <child link="calibration_tag_right"/>
+    <origin xyz="-0.08625 -0.04925 -0.01" rpy="0 0 0"/>
+  </joint>
+  <link name="calibration_tag_left">
+    <visual>
+      <origin xyz="0 0 0" rpy="0 1.5708 0"/>
+      <geometry>
+        <mesh filename="package://picknik_accessories/descriptions/ar_markers/Marker1.dae" scale=".05 .102 .102"/>
+      </geometry>
+    </visual>
+  </link>
+  <joint name="calibration_tag_left_joint" type="fixed">
+    <parent link="calibration_tool_link"/>
+    <child link="calibration_tag_left"/>
+    <origin xyz="0.08625 -0.04925 -0.01" rpy="0 0 0"/>
+  </joint>
+  <link name="calibration_tag_bottom">
+    <visual>
+      <origin xyz="0 0 0" rpy="0 1.5708 0"/>
+      <geometry>
+        <mesh filename="package://picknik_accessories/descriptions/ar_markers/Marker2.dae" scale=".05 .102 .102"/>
+      </geometry>
+    </visual>
+  </link>
+  <joint name="calibration_tag_bottom_joint" type="fixed">
+    <parent link="calibration_tool_link"/>
+    <child link="calibration_tag_bottom"/>
+    <origin xyz="0.0 -0.18125 -0.01" rpy="0 0 0"/>
+  </joint>
+  <link name="calibration_tool_frame"/>
+  <joint name="calibration_tool_frame_joint" type="fixed">
+    <parent link="calibration_tool_link"/>
+    <child link = "calibration_tool_frame"/>
+    <origin xyz="0 -0.09325 -0.01" rpy="0 ${pi} ${pi}"/>
+  </joint>
   <!-- Servicer Camera -->
   <link name="servicer_camera_mount_link" />
@@ -663,7 +722,7 @@
     <hardware>
       <plugin>picknik_mujoco_ros/MujocoSystem</plugin>
-      <param name="mujoco_keyframe">$(arg mujoco_keyframe)</param>
+      <!-- <param name="mujoco_keyframe">$(arg mujoco_keyframe)</param> -->
       <param name="mujoco_model">$(arg mujoco_model)</param>
-      <param name="mujoco_model_package">space_satellite_sim</param>
+      <param name="mujoco_model_package">space_satellite_sim_camera_cal</param>
       <param name="mujoco_viewer">$(arg mujoco_viewer)</param>
       <param name="render_publish_rate">10</param>

Commit message: Fix 2cm baselink offset, update servicer cam to realsense.

File: src/moveit_pro_kinova_configs/space_satellite_sim_camera_cal/description/space_satellite_sim.xacro (robot description, xacro)
@@ -545,7 +545,7 @@
   </link>
   <joint name="calibration_tool_joint" type="fixed">
-    <parent link="grasp_link"/>
+    <parent link="robotiq_85_base_link"/>
     <child link="calibration_tool_link"/>
-    <origin xyz="0 0 0.019" rpy="0 0 0"/>
+    <origin xyz="0 0 0.169" rpy="0 0 0"/>
   </joint>
   <link name="calibration_tag_right">
@@ -595,12 +595,22 @@
     <origin xyz="0 -0.09325 -0.01" rpy="0 ${pi} ${pi}"/>
   </joint>
-  <!-- Camera External -->
-  <link name="external_camera_link" />
-  <joint name="external_camera_joint" type="fixed">
+  <!-- Servicer Camera -->
+  <link name="servicer_camera_mount_link" />
+  <joint name="servicer_camera_mount_joint" type="fixed">
     <parent link="world" />
-    <child link="external_camera_link" />
+    <child link="servicer_camera_mount_link" />
+    <origin xyz=" 0.585021 0.966828 -0.0111449" rpy="0.00122423 0.00171265 -0.426171" />
+  </joint>
+  <xacro:realsense_d415 parent="servicer_camera_mount_link" name="servicer_camera">
+    <origin xyz="0 0 0" rpy="0 0 0" />
+  </xacro:realsense_d415>
+  <!-- Scene Camera -->
+  <link name="scene_camera_mount_link" />
+  <joint name="scene_camera_mount_joint" type="fixed">
+    <parent link="world" />
+    <child link="scene_camera_mount_link" />
     <origin xyz="-0.3 0.3 1.0" rpy="0 0.5236 0" />
   </joint>
-  <xacro:realsense_d415 parent="external_camera_link" name="scene_camera">
+  <xacro:realsense_d415 parent="scene_camera_mount_link" name="scene_camera">
     <origin xyz="0 0 0" rpy="0 0 0" />
   </xacro:realsense_d415>
