Commit message: feat(space_satellite_sim_camera_cal): use CalibrateCameraPosePnp for scene camera cal
Rewire the scene-camera calibration leaf to GetImage + GetCameraInfo +
CalibrateCameraPosePnp (single joint PnP over all tag corners), replacing the
DetectAprilTags + per-tag GetDetectionPose + CalibrateCameraPose path.

Replace the decorative calibration_tag_right/left/bottom links with TF-only
calibration_tag_0/1/2 frames that reproduce the MuJoCo-rendered AprilTag poses
exactly (via a calibration_tags_root matching MuJoCo's calibration_tool body),
so the behavior's per-id TF lookups resolve to what the camera actually sees.

File: src/moveit_pro_kinova_configs/space_satellite_sim_camera_cal/description/space_satellite_sim.xacro (robot description, xacro)
@@ -549,43 +549,36 @@
     <origin xyz="0 0 0.169" rpy="0 0 0"/>
   </joint>
-  <link name="calibration_tag_right">
-    <visual>
-      <origin xyz="0 0 0" rpy="0 1.5708 0"/>
-      <geometry>
-        <mesh filename="package://picknik_accessories/descriptions/ar_markers/Marker0.dae" scale=".05 .102 .102"/>
-        <!-- .dae tag side len = 0.5m, and tag size is 0.051m -> scale=0.102m -->
-      </geometry>
-    </visual>
-  </link>
-  <joint name="calibration_tag_right_joint" type="fixed">
+  <!--
+    AprilTag TF frames consumed by CalibrateCameraPosePnp. Frame calibration_tag_<id>
+    is the pose of the physical tag with detected id <id>, origin at the tag center and
+    +Z out of the tag face. These reproduce the tags rendered in simulation (see
+    description/mujoco/gen3_7dof_body.xml) so the frames stay coincident with what the
+    camera sees: the MuJoCo "calibration_tool" body applies a -90 deg yaw that
+    calibration_tool_link does not, so the tags hang off a matching intermediate frame.
+    Detected ids follow the MuJoCo materials: 0 = tool left, 1 = tool right, 2 = bottom.
+  -->
+  <link name="calibration_tags_root"/>
+  <joint name="calibration_tags_root_joint" type="fixed">
     <parent link="calibration_tool_link"/>
-    <child link="calibration_tag_right"/>
-    <origin xyz="-0.08625 -0.04925 -0.01" rpy="0 0 0"/>
-  </joint>
-  <link name="calibration_tag_left">
-    <visual>
-      <origin xyz="0 0 0" rpy="0 1.5708 0"/>
-      <geometry>
-        <mesh filename="package://picknik_accessories/descriptions/ar_markers/Marker1.dae" scale=".05 .102 .102"/>
-      </geometry>
-    </visual>
-  </link>
-  <joint name="calibration_tag_left_joint" type="fixed">
-    <parent link="calibration_tool_link"/>
-    <child link="calibration_tag_left"/>
-    <origin xyz="0.08625 -0.04925 -0.01" rpy="0 0 0"/>
-  </joint>
-  <link name="calibration_tag_bottom">
-    <visual>
-      <origin xyz="0 0 0" rpy="0 1.5708 0"/>
-      <geometry>
-        <mesh filename="package://picknik_accessories/descriptions/ar_markers/Marker2.dae" scale=".05 .102 .102"/>
-      </geometry>
-    </visual>
-  </link>
-  <joint name="calibration_tag_bottom_joint" type="fixed">
-    <parent link="calibration_tool_link"/>
-    <child link="calibration_tag_bottom"/>
-    <origin xyz="0.0 -0.18125 -0.01" rpy="0 0 0"/>
+    <child link="calibration_tags_root"/>
+    <origin xyz="0 0 0" rpy="0 0 -1.5708"/>
+  </joint>
+  <link name="calibration_tag_0"/>
+  <joint name="calibration_tag_0_joint" type="fixed">
+    <parent link="calibration_tags_root"/>
+    <child link="calibration_tag_0"/>
+    <origin xyz="0.08625 -0.04925 -0.01" rpy="3.14159 0 0"/>
+  </joint>
+  <link name="calibration_tag_1"/>
+  <joint name="calibration_tag_1_joint" type="fixed">
+    <parent link="calibration_tags_root"/>
+    <child link="calibration_tag_1"/>
+    <origin xyz="-0.08625 -0.04925 -0.01" rpy="3.14159 0 0"/>
+  </joint>
+  <link name="calibration_tag_2"/>
+  <joint name="calibration_tag_2_joint" type="fixed">
+    <parent link="calibration_tags_root"/>
+    <child link="calibration_tag_2"/>
+    <origin xyz="0.0 -0.18125 -0.01" rpy="3.14159 0 0"/>
   </joint>
   <link name="calibration_tool_frame"/>

Commit message: fix(space_satellite_sim_camera_cal): correct calibration tag frames for PnP
Part B's tag frames added a spurious Rz(-90) parent rotation
(calibration_tags_root) that displaced the tag positions from where they
render in MuJoCo. CalibrateCameraPosePnp uses tag corners (orientation-
and position-sensitive), so this made it drift to a different phantom
camera pose at each waypoint, whereas the old center-only
CalibrateCameraPose tolerated it.

Parent calibration_tag_0/1/2 directly to calibration_tool_link at the
proven tag-center offsets (same values the original centers-based
calibration used); rpy="3.14159 0 0" keeps +Z out of the tag face for
the corner PnP solve. Verified in sim: recovered optical pose is now
consistent across all waypoints and the saved mount matches the URDF
scene camera mount within noise.

File: src/moveit_pro_kinova_configs/space_satellite_sim_camera_cal/description/space_satellite_sim.xacro (robot description, xacro)
@@ -550,21 +550,15 @@
   </joint>
   <!--
-    AprilTag TF frames consumed by CalibrateCameraPosePnp. Frame calibration_tag_<id>
-    is the pose of the physical tag with detected id <id>, origin at the tag center and
-    +Z out of the tag face. These reproduce the tags rendered in simulation (see
-    description/mujoco/gen3_7dof_body.xml) so the frames stay coincident with what the
-    camera sees: the MuJoCo "calibration_tool" body applies a -90 deg yaw that
-    calibration_tool_link does not, so the tags hang off a matching intermediate frame.
-    Detected ids follow the MuJoCo materials: 0 = tool left, 1 = tool right, 2 = bottom.
+    AprilTag TF frames consumed by CalibrateCameraPosePnp. Frame calibration_tag_<id> is the
+    pose of the physical tag with detected id <id>: origin at the tag center, +Z out of the tag
+    face. These reproduce the tags rendered in simulation (description/mujoco/gen3_7dof_body.xml)
+    so the frames stay coincident with what the camera sees. The tag-center positions are the
+    same values the original center-based CalibrateCameraPose used (proven correct in sim); the
+    rpy flips Z so +Z points out of the tag face, which the corner-based PnP solve needs. Detected
+    ids follow the MuJoCo materials: 0 = tool left, 1 = tool right, 2 = bottom.
   -->
-  <link name="calibration_tags_root"/>
-  <joint name="calibration_tags_root_joint" type="fixed">
-    <parent link="calibration_tool_link"/>
-    <child link="calibration_tags_root"/>
-    <origin xyz="0 0 0" rpy="0 0 -1.5708"/>
-  </joint>
   <link name="calibration_tag_0"/>
   <joint name="calibration_tag_0_joint" type="fixed">
-    <parent link="calibration_tags_root"/>
+    <parent link="calibration_tool_link"/>
     <child link="calibration_tag_0"/>
     <origin xyz="0.08625 -0.04925 -0.01" rpy="3.14159 0 0"/>
@@ -572,5 +566,5 @@
   <link name="calibration_tag_1"/>
   <joint name="calibration_tag_1_joint" type="fixed">
-    <parent link="calibration_tags_root"/>
+    <parent link="calibration_tool_link"/>
     <child link="calibration_tag_1"/>
     <origin xyz="-0.08625 -0.04925 -0.01" rpy="3.14159 0 0"/>
@@ -578,5 +572,5 @@
   <link name="calibration_tag_2"/>
   <joint name="calibration_tag_2_joint" type="fixed">
-    <parent link="calibration_tags_root"/>
+    <parent link="calibration_tool_link"/>
     <child link="calibration_tag_2"/>
     <origin xyz="0.0 -0.18125 -0.01" rpy="3.14159 0 0"/>

Commit message: feat(space_satellite_sim_camera_cal): add wrist-camera (eye-in-hand) PnP calibration
Add a "Calibrate Wrist Camera" objective that calibrates the wrist-mounted
camera against three static satellite AprilTags, reusing the same
CalibrateCameraPosePnp subtree as the scene-camera (eye-to-hand) calibration.
Only the frames, topics, tag prefix, and waypoints differ.

- Scene/URDF: three tag36h11 markers (ids 3/4/5, distinct from the tool plate
  0/1/2) as angled plates on the drum top, plus a wrist_camera_mount_link frame
  on the flange to receive the calibrated extrinsics.
- Objectives: thread tag_frame_prefix, mounting_pose_parent_frame, and
  waypoint_N_name through the shared subtrees (defaults preserve the scene-camera
  path unchanged); new thin calibrate_wrist_camera.xml wires the wrist ports.
- Per-waypoint fix: express each waypoint's optical pose in the mount-parent
  frame before averaging. For a moving (eye-in-hand) camera the optical pose in
  base_link differs per waypoint, so averaging it directly biased the result;
  the mount-parent frame is rigid to the camera, so the cross-waypoint average is
  unbiased. This is a no-op for the eye-to-hand case (parent == base_link).

Verified in sim: recovers the declared wrist mount [0, -0.056, -0.058] Ry180 to
sub-millimeter, with per-waypoint PnP reprojection RMS ~0.38 px.

File: src/moveit_pro_kinova_configs/space_satellite_sim_camera_cal/description/space_satellite_sim.xacro (robot description, xacro)
@@ -602,4 +602,37 @@
     <origin xyz="0 0 0" rpy="0 0 0" />
   </xacro:realsense_d415>
+  <!-- Wrist Camera mount (eye-in-hand calibration). The nominal flange-to-camera pose
+       that the "Calibrate Wrist Camera" objective solves for; paste its result here to
+       correct the extrinsics. For the sim, mount == optical: bracelet_link -> optical is
+       Ry(180 deg) at [0, -0.056, -0.058] (MuJoCo renders /wrist_camera/* from this). -->
+  <link name="wrist_camera_mount_link" />
+  <joint name="wrist_camera_mount_joint" type="fixed">
+    <parent link="bracelet_link" />
+    <child link="wrist_camera_mount_link" />
+    <origin xyz="0 -0.056 -0.058" rpy="0 3.14159265358979 0" />
+  </joint>
+  <!-- Satellite calibration tags (static, world-fixed) for the wrist camera. tag36h11
+       ids 3/4/5, mounted as angled plates on the drum top facing the servicer arm; the
+       rpy tilt (Ry 30 deg) points +Z out of the tag face for the corner-based PnP solve.
+       Poses match the MuJoCo satellite_tags geoms in description/mujoco/scene.xml. The
+       "Calibrate Wrist Camera" objective looks up frame 'sat_tag_<id>'. -->
+  <link name="sat_tag_3" />
+  <joint name="sat_tag_3_joint" type="fixed">
+    <parent link="world" />
+    <child link="sat_tag_3" />
+    <origin xyz="0.42 0.46 0.274" rpy="0 0.5236 0" />
+  </joint>
+  <link name="sat_tag_4" />
+  <joint name="sat_tag_4_joint" type="fixed">
+    <parent link="world" />
+    <child link="sat_tag_4" />
+    <origin xyz="0.42 0.66 0.274" rpy="0 0.5236 0" />
+  </joint>
+  <link name="sat_tag_5" />
+  <joint name="sat_tag_5_joint" type="fixed">
+    <parent link="world" />
+    <child link="sat_tag_5" />
+    <origin xyz="0.20 0.56 0.274" rpy="0 0.5236 0" />
+  </joint>
   <ros2_control name="kinova_mujoco_simulation" type="system">
     <joint name="joint_1">

Commit message: refactor(space_satellite_sim_camera_cal): flat front-face wrist-cal tags + diverse waypoints
Mount the three satellite AprilTags flat and coplanar on the servicer's front
(+x) gold face, on the arm-base side of the docking mechanism, replacing the
tilted drum-top placement (scene.xml geoms + matching sat_tag_* URDF frames;
Ry90 so +Z exits the tag face). Regenerate the four wrist-camera waypoints for
diverse, collision-free views that keep all three tags clear of the end
effector. Sim-verified: every waypoint detects all 3 tags and the recovered
wrist mount matches the URDF to ~0.6 mm / 0.02 deg.

File: src/moveit_pro_kinova_configs/space_satellite_sim_camera_cal/description/space_satellite_sim.xacro (robot description, xacro)
@@ -613,13 +613,14 @@
   </joint>
   <!-- Satellite calibration tags (static, world-fixed) for the wrist camera. tag36h11
-       ids 3/4/5, mounted as angled plates on the drum top facing the servicer arm; the
-       rpy tilt (Ry 30 deg) points +Z out of the tag face for the corner-based PnP solve.
-       Poses match the MuJoCo satellite_tags geoms in description/mujoco/scene.xml. The
-       "Calibrate Wrist Camera" objective looks up frame 'sat_tag_<id>'. -->
+       ids 3/4/5, mounted flat and coplanar on the servicer's front (+x) gold face, on
+       the arm-base side of the central docking mechanism. rpy (Ry 90 deg) points +Z out
+       of the tag face (normal +x) for the corner-based PnP solve. Poses match the MuJoCo
+       satellite_tags geoms in description/mujoco/scene.xml. The "Calibrate Wrist Camera"
+       objective looks up frame 'sat_tag_<id>'. -->
   <link name="sat_tag_3" />
   <joint name="sat_tag_3_joint" type="fixed">
     <parent link="world" />
     <child link="sat_tag_3" />
-    <origin xyz="0.42 0.46 0.274" rpy="0 0.5236 0" />
+    <origin xyz="0.50 0.45 0.04" rpy="0 1.5708 0" />
   </joint>
   <link name="sat_tag_4" />
@@ -627,5 +628,5 @@
     <parent link="world" />
     <child link="sat_tag_4" />
-    <origin xyz="0.42 0.66 0.274" rpy="0 0.5236 0" />
+    <origin xyz="0.50 0.27 0.04" rpy="0 1.5708 0" />
   </joint>
   <link name="sat_tag_5" />
@@ -633,5 +634,5 @@
     <parent link="world" />
     <child link="sat_tag_5" />
-    <origin xyz="0.20 0.56 0.274" rpy="0 0.5236 0" />
+    <origin xyz="0.50 0.36 -0.12" rpy="0 1.5708 0" />
   </joint>
   <ros2_control name="kinova_mujoco_simulation" type="system">
