Commit message: Add servicer platform to xacro, fix arm mounting transform
Former-commit-id: 886e15dead24614c4e41abdb2b0a7bce0e52df7f

File: src/moveit_pro_kinova_configs/space_satellite_sim/description/space_satellite_sim.xacro (robot description, xacro)
@@ -1,666 +1,663 @@
 <?xml version="1.0"?>
 <robot name="gen3" xmlns:xacro="http://ros.org/wiki/xacro">
-    <!-- Arguments for Kinova -->
-    <xacro:arg name="arm" default="gen3" />
-    <xacro:arg name="dof" default="7" />
-    <xacro:arg name="mujoco_keyframe" default="default" />
-    <xacro:arg name="mujoco_model" default="description/mujoco/scene.xml" />
-    <xacro:arg name="mujoco_viewer" default="false" />
-    <!-- Import macros for main hardware components -->
-    <xacro:include filename="$(find kortex_description)/arms/$(arg arm)/$(arg dof)dof/urdf/$(arg arm)_macro.xacro" />
-    <xacro:include filename="$(find picknik_accessories)/descriptions/sensors/realsense_d415.urdf.xacro"/>
-    <!-- Import environment macros -->
-    <xacro:include filename="$(find picknik_accessories)/descriptions/geometry/cube.urdf.xacro"/>
-    <!-- World is centered under base_link of the robot, on the ground -->
-    <link name="world"/>
-    <!-- initial position for simulations (Mock Hardware, Gazebo, Ignition) -->
-    <xacro:arg name="initial_positions_file" default="$(find kinova_sim)/config/initial_positions.yaml"/>
-    <xacro:property name="initial_positions_file" default="$(arg initial_positions_file)"/>
-    <!-- Load the arm -->
-    <joint name="base_joint" type="fixed">
-      <origin rpy="0 0 0" xyz="0 0 0.02"/>
-      <parent link="world"/>
-      <child link="base_link"/>
-    </joint>
-    <link name="base_link">
-      <inertial>
-        <origin rpy="0 0 0" xyz="-0.000648 -0.000166 0.084487"/>
-        <mass value="1.697"/>
-        <inertia ixx="0.004622" ixy="9E-06" ixz="6E-05" iyy="0.004495" iyz="9E-06" izz="0.002079"/>
-      </inertial>
-      <visual>
-        <origin rpy="0 0 0" xyz="0 0 0"/>
-        <geometry>
-          <mesh filename="package://kortex_description/arms/gen3/7dof/meshes/base_link.STL"/>
-        </geometry>
-        <material name="">
-          <color rgba="0.75294 0.75294 0.75294 1"/>
-        </material>
-      </visual>
-      <collision>
-        <origin rpy="0 0 0" xyz="0 0 0"/>
-        <geometry>
-          <mesh filename="package://kortex_description/arms/gen3/7dof/meshes/base_link.STL"/>
-        </geometry>
-      </collision>
-    </link>
-    <link name="shoulder_link">
-      <inertial>
-        <origin rpy="0 0 0" xyz="-2.3E-05 -0.010364 -0.07336"/>
-        <mass value="1.3773"/>
-        <inertia ixx="0.00457" ixy="1E-06" ixz="2E-06" iyy="0.004831" iyz="0.000448" izz="0.001409"/>
-      </inertial>
-      <visual>
-        <origin rpy="0 0 0" xyz="0 0 0"/>
-        <geometry>
-          <mesh filename="package://kortex_description/arms/gen3/7dof/meshes/shoulder_link.STL"/>
-        </geometry>
-        <material name="">
-          <color rgba="0.75294 0.75294 0.75294 1"/>
-        </material>
-      </visual>
-      <collision>
-        <origin rpy="0 0 0" xyz="0 0 0"/>
-        <geometry>
-          <mesh filename="package://kortex_description/arms/gen3/7dof/meshes/shoulder_link.STL"/>
-        </geometry>
-      </collision>
-    </link>
-    <joint name="joint_1" type="continuous">
-      <origin rpy="3.1416 2.7629E-18 -4.9305E-36" xyz="0 0 0.15643"/>
-      <parent link="base_link"/>
-      <child link="shoulder_link"/>
-      <axis xyz="0 0 1"/>
-      <limit effort="39" velocity="1.3963"/>
-    </joint>
-    <link name="half_arm_1_link">
-      <inertial>
-        <origin rpy="0 0 0" xyz="-4.4E-05 -0.09958 -0.013278"/>
-        <mass value="1.1636"/>
-        <inertia ixx="0.011088" ixy="5E-06" ixz="0" iyy="0.001072" iyz="-0.000691" izz="0.011255"/>
-      </inertial>
-      <visual>
-        <origin rpy="0 0 0" xyz="0 0 0"/>
-        <geometry>
-          <mesh filename="package://kortex_description/arms/gen3/7dof/meshes/half_arm_1_link.STL"/>
-        </geometry>
-        <material name="">
-          <color rgba="0.75294 0.75294 0.75294 1"/>
-        </material>
-      </visual>
-      <collision>
-        <origin rpy="0 0 0" xyz="0 0 0"/>
-        <geometry>
-          <mesh filename="package://kortex_description/arms/gen3/7dof/meshes/half_arm_1_link.STL"/>
-        </geometry>
-      </collision>
-    </link>
-    <joint name="joint_2" type="revolute">
-      <origin rpy="1.5708 2.1343E-17 -1.1102E-16" xyz="0 0.005375 -0.12838"/>
-      <parent link="shoulder_link"/>
-      <child link="half_arm_1_link"/>
-      <axis xyz="0 0 1"/>
-      <limit effort="39" lower="-2.41" upper="2.41" velocity="1.3963"/>
-    </joint>
-    <link name="half_arm_2_link">
-      <inertial>
-        <origin rpy="0 0 0" xyz="-4.4E-05 -0.006641 -0.117892"/>
-        <mass value="1.1636"/>
-        <inertia ixx="0.010932" ixy="0" ixz="-7E-06" iyy="0.011127" iyz="0.000606" izz="0.001043"/>
-      </inertial>
-      <visual>
-        <origin rpy="0 0 0" xyz="0 0 0"/>
-        <geometry>
-          <mesh filename="package://kortex_description/arms/gen3/7dof/meshes/half_arm_2_link.STL"/>
-        </geometry>
-        <material name="">
-          <color rgba="0.75294 0.75294 0.75294 1"/>
-        </material>
-      </visual>
-      <collision>
-        <origin rpy="0 0 0" xyz="0 0 0"/>
-        <geometry>
-          <mesh filename="package://kortex_description/arms/gen3/7dof/meshes/half_arm_2_link.STL"/>
-        </geometry>
-      </collision>
-    </link>
-    <joint name="joint_3" type="continuous">
-      <origin rpy="-1.5708 1.2326E-32 -2.9122E-16" xyz="0 -0.21038 -0.006375"/>
-      <parent link="half_arm_1_link"/>
-      <child link="half_arm_2_link"/>
-      <axis xyz="0 0 1"/>
-      <limit effort="39" velocity="1.3963"/>
-    </joint>
-    <link name="forearm_link">
-      <inertial>
-        <origin rpy="0 0 0" xyz="-1.8E-05 -0.075478 -0.015006"/>
-        <mass value="0.9302"/>
-        <inertia ixx="0.008147" ixy="-1E-06" ixz="0" iyy="0.000631" iyz="-0.0005" izz="0.008316"/>
-      </inertial>
-      <visual>
-        <origin rpy="0 0 0" xyz="0 0 0"/>
-        <geometry>
-          <mesh filename="package://kortex_description/arms/gen3/7dof/meshes/forearm_link.STL"/>
-        </geometry>
-        <material name="">
-          <color rgba="0.75294 0.75294 0.75294 1"/>
-        </material>
-      </visual>
-      <collision>
-        <origin rpy="0 0 0" xyz="0 0 0"/>
-        <geometry>
-          <mesh filename="package://kortex_description/arms/gen3/7dof/meshes/forearm_link.STL"/>
-        </geometry>
-      </collision>
-    </link>
-    <joint name="joint_4" type="revolute">
-      <origin rpy="1.5708 -6.6954E-17 -1.6653E-16" xyz="0 0.006375 -0.21038"/>
-      <parent link="half_arm_2_link"/>
-      <child link="forearm_link"/>
-      <axis xyz="0 0 1"/>
-      <limit effort="39" lower="-2.66" upper="2.66" velocity="1.3963"/>
-    </joint>
-    <link name="spherical_wrist_1_link">
-      <inertial>
-        <origin rpy="0 0 0" xyz="1E-06 -0.009432 -0.063883"/>
-        <mass value="0.6781"/>
-        <inertia ixx="0.001596" ixy="0" ixz="0" iyy="0.001607" iyz="0.000256" izz="0.000399"/>
-      </inertial>
-      <visual>
-        <origin rpy="0 0 0" xyz="0 0 0"/>
-        <geometry>
-          <mesh filename="package://kortex_description/arms/gen3/7dof/meshes/spherical_wrist_1_link.STL"/>
-        </geometry>
-        <material name="">
-          <color rgba="0.75294 0.75294 0.75294 1"/>
-        </material>
-      </visual>
-      <collision>
-        <origin rpy="0 0 0" xyz="0 0 0"/>
-        <geometry>
-          <mesh filename="package://kortex_description/arms/gen3/7dof/meshes/spherical_wrist_1_link.STL"/>
-        </geometry>
-      </collision>
-    </link>
-    <joint name="joint_5" type="continuous">
-      <origin rpy="-1.5708 2.2204E-16 -6.373E-17" xyz="0 -0.20843 -0.006375"/>
-      <parent link="forearm_link"/>
-      <child link="spherical_wrist_1_link"/>
-      <axis xyz="0 0 1"/>
-      <limit effort="9" velocity="1.2218"/>
-    </joint>
-    <link name="spherical_wrist_2_link">
-      <inertial>
-        <origin rpy="0 0 0" xyz="1E-06 -0.045483 -0.00965"/>
-        <mass value="0.6781"/>
-        <inertia ixx="0.001641" ixy="0" ixz="0" iyy="0.00041" iyz="-0.000278" izz="0.001641"/>
-      </inertial>
-      <visual>
-        <origin rpy="0 0 0" xyz="0 0 0"/>
-        <geometry>
-          <mesh filename="package://kortex_description/arms/gen3/7dof/meshes/spherical_wrist_2_link.STL"/>
-        </geometry>
-        <material name="">
-          <color rgba="0.75294 0.75294 0.75294 1"/>
-        </material>
-      </visual>
-      <collision>
-        <origin rpy="0 0 0" xyz="0 0 0"/>
-        <geometry>
-          <mesh filename="package://kortex_description/arms/gen3/7dof/meshes/spherical_wrist_2_link.STL"/>
-        </geometry>
-      </collision>
-    </link>
-    <joint name="joint_6" type="revolute">
-      <origin rpy="1.5708 9.2076E-28 -8.2157E-15" xyz="0 0.00017505 -0.10593"/>
-      <parent link="spherical_wrist_1_link"/>
-      <child link="spherical_wrist_2_link"/>
-      <axis xyz="0 0 1"/>
-      <limit effort="9" lower="-2.23" upper="2.23" velocity="1.2218"/>
-    </joint>
-    <link name="bracelet_link">
-      <inertial>
-        <origin rpy="0 0 0" xyz="-9.3E-05 0.000132 -0.022905"/>
-        <mass value="0.364"/>
-        <inertia ixx="0.000214" ixy="0" ixz="1E-06" iyy="0.000223" iyz="-2E-06" izz="0.00024"/>
-      </inertial>
-      <visual>
-        <origin rpy="0 0 0" xyz="0 0 0"/>
-        <geometry>
-          <mesh filename="package://kortex_description/arms/gen3/7dof/meshes/bracelet_with_vision_link.STL"/>
-        </geometry>
-        <material name="">
-          <color rgba="0.75294 0.75294 0.75294 1"/>
-        </material>
-      </visual>
-      <collision>
-        <origin rpy="0 0 0" xyz="0 0 0"/>
-        <geometry>
-          <mesh filename="package://kortex_description/arms/gen3/7dof/meshes/bracelet_with_vision_link.STL"/>
-        </geometry>
-      </collision>
-    </link>
-    <joint name="joint_7" type="continuous">
-      <origin rpy="-1.5708 -5.5511E-17 9.6396E-17" xyz="0 -0.10593 -0.00017505"/>
-      <parent link="spherical_wrist_2_link"/>
-      <child link="bracelet_link"/>
-      <axis xyz="0 0 1"/>
-      <limit effort="9" velocity="1.2218"/>
-    </joint>
-    <link name="end_effector_link"/>
-    <joint name="end_effector" type="fixed">
-      <origin rpy="3.14159265358979 1.09937075168372E-32 0" xyz="0 0 -0.0615250000000001"/>
-      <parent link="bracelet_link"/>
-      <child link="end_effector_link"/>
-      <axis xyz="0 0 0"/>
-    </joint>
-    <link name="fts_link"/>
-    <joint name="fts_joint" type="fixed">
-      <origin rpy="0.0 0.0 3.14159265358979" xyz="0 0 0.0"/>
-      <parent link="end_effector_link"/>
-      <child link="fts_link"/>
-      <axis xyz="0 0 0"/>
-    </joint>
-    <!-- Add robotiq 2f 85 gripper model -->
-    <link name="robotiq_85_base_link">
-      <visual>
-        <geometry>
-          <mesh filename="package://robotiq_description/meshes/visual/2f_85/robotiq_base.dae"/>
-        </geometry>
-      </visual>
-      <collision>
-        <geometry>
-          <mesh filename="package://robotiq_description/meshes/collision/2f_85/robotiq_base.stl"/>
-        </geometry>
-      </collision>
-      <inertial>
-        <origin rpy="0 0 0" xyz="0.0 2.274e-05 0.03232288"/>
-        <mass value="6.6320197e-01"/>
-        <inertia ixx="5.1617816e-04" ixy="2.936e-8" ixz="0.0" iyy="5.8802208e-04" iyz="-3.2296e-7" izz="3.9462776e-04"/>
-      </inertial>
-    </link>
-    <link name="robotiq_85_left_knuckle_link">
-      <visual>
-        <geometry>
-          <mesh filename="package://robotiq_description/meshes/visual/2f_85/left_knuckle.dae"/>
-        </geometry>
-      </visual>
-      <collision>
-        <geometry>
-          <mesh filename="package://robotiq_description/meshes/collision/2f_85/left_knuckle.stl"/>
-        </geometry>
-      </collision>
-      <inertial>
-        <origin rpy="0 0 0" xyz="0.01213197 0.0002 -0.00058647"/>
-        <mass value="1.384773208e-02"/>
-        <inertia ixx="3.5232e-7" ixy="0.0" ixz="1.1744e-7" iyy="2.31944e-6" iyz="0" izz="2.23136e-6"/>
-      </inertial>
-    </link>
-    <link name="robotiq_85_right_knuckle_link">
-      <visual>
-        <geometry>
-          <mesh filename="package://robotiq_description/meshes/visual/2f_85/right_knuckle.dae"/>
-        </geometry>
-      </visual>
-      <collision>
-        <geometry>
-          <mesh filename="package://robotiq_description/meshes/collision/2f_85/right_knuckle.stl"/>
-        </geometry>
-      </collision>
-      <inertial>
-        <origin rpy="0 0 0" xyz="-0.01213197 0.0002 -0.00058647"/>
-        <mass value="1.384773208e-02"/>
-        <inertia ixx="3.5232e-7" ixy="0.0" ixz="-1.1744e-7" iyy="2.31944e-6" iyz="0.0" izz="2.23136e-6"/>
-      </inertial>
-    </link>
-    <link name="robotiq_85_left_finger_link">
-      <visual>
-        <geometry>
-          <mesh filename="package://robotiq_description/meshes/visual/2f_85/left_finger.dae"/>
-        </geometry>
-      </visual>
-      <collision>
-        <geometry>
-          <mesh filename="package://robotiq_description/meshes/collision/2f_85/left_finger.stl"/>
-        </geometry>
-      </collision>
-      <inertial>
-        <origin rpy="0 0 0" xyz="0.00346899 -0.00079447 0.01867121"/>
-        <mass value="4.260376752e-02"/>
-        <inertia ixx="1.385792000000000e-05" ixy="0.0" ixz="-2.17264e-06" iyy="1.183208e-05" iyz="0.0" izz="5.19672e-06"/>
-      </inertial>
-    </link>
-    <link name="robotiq_85_right_finger_link">
-      <visual>
-        <geometry>
-          <mesh filename="package://robotiq_description/meshes/visual/2f_85/right_finger.dae"/>
-        </geometry>
-      </visual>
-      <collision>
-        <geometry>
-          <mesh filename="package://robotiq_description/meshes/collision/2f_85/right_finger.stl"/>
-        </geometry>
-      </collision>
-      <inertial>
-        <origin rpy="0 0 0" xyz="-0.00346899 -5.53e-06 0.01867121"/>
-        <mass value="4.260376752000000e-02"/>
-        <inertia ixx="1.385792e-05" ixy="0.0" ixz="2.17264e-06" iyy="1.183208e-05" iyz="0.0" izz="5.19672e-06"/>
-      </inertial>
-    </link>
-    <link name="robotiq_85_left_inner_knuckle_link">
-      <visual>
-        <geometry>
-          <mesh filename="package://robotiq_description/meshes/visual/2f_85/left_inner_knuckle.dae"/>
-        </geometry>
-      </visual>
-      <collision>
-        <geometry>
-          <mesh filename="package://robotiq_description/meshes/collision/2f_85/left_inner_knuckle.stl"/>
-        </geometry>
-      </collision>
-      <inertial>
-        <origin rpy="0 0 0" xyz="0.01897699 0.00015001 0.02247101"/>
-        <mass value="2.969376448e-02"/>
-        <inertia ixx="9.57136e-06" ixy="0.0" ixz="-3.93424e-06" iyy="8.69056e-06" iyz="0.0" izz="8.19144e-06"/>
-      </inertial>
-    </link>
-    <link name="robotiq_85_right_inner_knuckle_link">
-      <visual>
-        <geometry>
-          <mesh filename="package://robotiq_description/meshes/visual/2f_85/right_inner_knuckle.dae"/>
-        </geometry>
-      </visual>
-      <collision>
-        <geometry>
-          <mesh filename="package://robotiq_description/meshes/collision/2f_85/right_inner_knuckle.stl"/>
-        </geometry>
-      </collision>
-      <inertial>
-        <origin rpy="0 0 0" xyz="-0.01926824 5.001e-05 0.02222178"/>
-        <mass value="2.969376448e-02"/>
-        <inertia ixx="9.42456e-06" ixy="0.0" ixz="3.9636e-06" iyy="8.69056e-06" iyz="0.0" izz="8.33824e-06"/>
-      </inertial>
-    </link>
-    <link name="robotiq_85_left_finger_tip_link">
-      <visual>
-        <geometry>
-          <mesh filename="package://robotiq_description/meshes/visual/2f_85/left_finger_tip.dae"/>
-        </geometry>
-      </visual>
-      <collision>
-        <geometry>
-          <mesh filename="package://robotiq_description/meshes/collision/2f_85/left_finger_tip.stl"/>
-        </geometry>
-        <surface>
-          <friction>
-            <ode>
-              <mu1>100000.0</mu1>
-              <mu2>100000.0</mu2>
-            </ode>
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
Commit message: Update for Pro detection to be primary, and to use ports instead of params.

File: src/moveit_pro_kinova_configs/space_satellite_sim/description/space_satellite_sim.xacro (robot description, xacro)
@@ -536,12 +536,22 @@
     <origin xyz="0 0 0.15" rpy="0 0 0"/>
   </joint>
-  <!-- Camera External -->
-  <link name="external_camera_link" />
-  <joint name="external_camera_joint" type="fixed">
+  <!-- Servicer Camera -->
+  <link name="servicer_camera_mount_link" />
+  <joint name="servicer_camera_mount_joint" type="fixed">
     <parent link="world" />
-    <child link="external_camera_link" />
+    <child link="servicer_camera_mount_link" />
+    <origin xyz=" 0.585021 0.966828 -0.0111449" rpy="0.00122423 0.00171265 -0.426171" />
+  </joint>
+  <xacro:realsense_d415 parent="servicer_camera_mount_link" name="servicer_camera">
+    <origin xyz="0 0 0" rpy="0 0 0" />
+  </xacro:realsense_d415>
+  <!-- Scene Camera -->
+  <link name="scene_camera_mount_link" />
+  <joint name="scene_camera_mount_joint" type="fixed">
+    <parent link="world" />
+    <child link="scene_camera_mount_link" />
     <origin xyz="-0.3 0.3 1.0" rpy="0 0.5236 0" />
   </joint>
-  <xacro:realsense_d415 parent="external_camera_link" name="scene_camera">
+  <xacro:realsense_d415 parent="scene_camera_mount_link" name="scene_camera">
     <origin xyz="0 0 0" rpy="0 0 0" />
   </xacro:realsense_d415>
