Commit message: Pivot to new HW interface approach!

File: src/moveit_pro_franka_configs/franka_dual_arm_config_hw/description/franka.urdf.xacro (robot description, xacro)
@@ -1,6 +1,6 @@
 <?xml version='1.0' encoding='utf-8'?>
 <robot xmlns:xacro="http://www.ros.org/wiki/xacro" name="franka">
-  <xacro:arg name="right_robot_ip" default="172.16.0.2" />
-  <xacro:arg name="left_robot_ip" default="172.16.0.3" />
+  <xacro:arg name="right_robot_ip" default="192.168.1.22" />
+  <xacro:arg name="left_robot_ip" default="192.168.1.21" />
   <xacro:arg name="ee_id" default="franka_hand" />
   <xacro:arg name="rpy_ee" default="0 0 -0.785" />
@@ -11,5 +11,5 @@
      <parent link="world"/>
      <child link = "right_mount"/>
-    <origin xyz="0 -0.06 0.342" rpy="0.8936 -0.1746 0.4636"/>
+    <origin xyz="0.035 -0.050681 0.356" rpy="0.8936 -0.1746 0.4636"/>
   </joint>
   <xacro:franka_robot arm_id="fr3"
@@ -40,5 +40,5 @@
      <parent link="world"/>
      <child link = "left_mount"/>
-    <origin xyz="0 0.06 0.342" rpy="-0.8936 -0.1746 -0.4636"/>
+    <origin xyz="0.035 0.050681 0.356" rpy="-0.8936 -0.1746 -0.4636"/>
   </joint>
   <xacro:franka_robot arm_id="fr3"

Commit message: Update franka dual arm hw config

File: src/moveit_pro_franka_configs/franka_dual_arm_config_hw/description/franka.urdf.xacro (robot description, xacro)
@@ -1,6 +1,6 @@
 <?xml version='1.0' encoding='utf-8'?>
 <robot xmlns:xacro="http://www.ros.org/wiki/xacro" name="franka">
-  <xacro:arg name="right_robot_ip" default="192.168.1.22" />
-  <xacro:arg name="left_robot_ip" default="192.168.1.21" />
+  <xacro:arg name="right_robot_ip" default="172.16.15.102" />
+  <xacro:arg name="left_robot_ip" default="172.16.0.4" />
   <xacro:arg name="ee_id" default="franka_hand" />
   <xacro:arg name="rpy_ee" default="0 0 -0.785" />
@@ -11,5 +11,5 @@
      <parent link="world"/>
      <child link = "right_mount"/>
-    <origin xyz="0.035 -0.050681 0.356" rpy="0.8936 -0.1746 0.4636"/>
+    <origin xyz="-0.6 -0.050681 0.356" rpy="0 0 0"/>
   </joint>
   <xacro:franka_robot arm_id="fr3"
@@ -40,5 +40,5 @@
      <parent link="world"/>
      <child link = "left_mount"/>
-    <origin xyz="0.035 0.050681 0.356" rpy="-0.8936 -0.1746 -0.4636"/>
+    <origin xyz="0.6 0.050681 0.356" rpy="0 0 0"/>
   </joint>
   <xacro:franka_robot arm_id="fr3"
