Commit message: wip
Former-commit-id: ebe3cb8b4042634abc9ec027813ea0c60d187352

File: src/moveit_pro_kuka_configs/moveit_pro_kr16/description/kr16.xacro (robot description, xacro)
@@ -6,4 +6,10 @@
   <xacro:arg name="use_fake_hardware" default="true" />
   <xacro:include filename="$(find kuka_cybertech_support)/urdf/kr16_r2010_2.urdf.xacro" />
+  <link name="grasp_link"/>
+  <joint name="grasp_link_joint" type="fixed">
+    <origin rpy="0 0 0" xyz="0.0 0.0 0.0"/>
+    <parent link="link_6"/>
+    <child link="grasp_link"/>
+  </joint>
   <ros2_control name="mujoco_control" type="system">
     <hardware>

Commit message: wip
Former-commit-id: 8bedbdf957fdea8156d81c5d7216534801a28e0d

File: src/moveit_pro_kuka_configs/moveit_pro_kr16/description/kr16.xacro (robot description, xacro)
@@ -5,4 +5,8 @@
   <!-- Import kr16 urdf file -->
   <xacro:arg name="use_fake_hardware" default="true" />
+  <xacro:arg
+    name="initial_positions_file"
+    default="$(find moveit_pro_kr16)/config/initial_positions.yaml"
+  />
   <xacro:include filename="$(find moveit_pro_kr16)/description/kr16_r2010_2.urdf.xacro" />
   <link name="grasp_link"/>
@@ -12,18 +16,3 @@
     <child link="grasp_link"/>
   </joint>
-  <ros2_control name="mujoco_control" type="system">
-    <hardware>
-      <plugin>picknik_mujoco_ros/MujocoSystem</plugin>
-      <param name="mujoco_model">$(arg mujoco_model)</param>
-      <param name="mujoco_model_package">moveit_pro_kr16</param>
-      <!-- The rate <camera> data is published at -->
-      <param name="render_publish_rate">10</param>
-      <!-- The rate transforms to <site> poses are published at -->
-      <param name="tf_publish_rate">60</param>
-      <!-- The rate <rangefinder> data is published at -->
-      <param name="lidar_publish_rate">10</param>
-      <!-- Whether to launch the MuJoCo interactive viewer -->
-      <param name="mujoco_viewer">$(arg mujoco_viewer)</param>
-    </hardware>
-  </ros2_control>
 </robot>

File: src/moveit_pro_kuka_configs/moveit_pro_kr16/description/kr16_r2010_2.urdf.xacro (robot description, xacro)
@@ -1,20 +1,25 @@
 <?xml version="1.0"?>
 <robot xmlns:xacro="http://www.ros.org/wiki/xacro" name="kr16_r2010_2">
-  <!-- Import urdf file  -->
-  <xacro:include filename="$(find moveit_pro_kr16)/description/kr16_r2010_2_macro.xacro"/>
-  <!-- Read additional arguments  -->
-  <xacro:arg name="use_fake_hardware" default="false"/>
-  <xacro:arg name="roundtrip_time" default="0"/>
-  <xacro:arg name="client_ip" default="0.0.0.0"/>
-  <xacro:arg name="client_port" default="59152"/>
-  <xacro:arg name="prefix" default=""/>
-  <xacro:arg name="x" default="0"/>
-  <xacro:arg name="y" default="0"/>
-  <xacro:arg name="z" default="0"/>
-  <xacro:arg name="roll" default="0"/>
-  <xacro:arg name="pitch" default="0"/>
-  <xacro:arg name="yaw" default="0"/>
-  <xacro:kuka_kr16_r2010_2_robot client_ip="$(arg client_ip)" client_port="$(arg client_port)" prefix="$(arg prefix)" use_fake_hardware="$(arg use_fake_hardware)" roundtrip_time="$(arg roundtrip_time)">
-    <origin xyz="$(arg x) $(arg y) $(arg z)" rpy="$(arg roll) $(arg pitch) $(arg yaw)"/>
-  </xacro:kuka_kr16_r2010_2_robot>
+    <!-- Import urdf file  -->
+    <xacro:include filename="$(find moveit_pro_kr16)/description/kr16_r2010_2_macro.xacro" />
+    <!-- Read additional arguments  -->
+    <xacro:arg name="use_fake_hardware" default="false" />
+    <xacro:arg name="roundtrip_time" default="0" />
+    <xacro:arg name="client_ip" default="0.0.0.0" />
+    <xacro:arg name="client_port" default="59152" />
+    <xacro:arg name="prefix" default="" />
+    <xacro:arg name="x" default="0" />
+    <xacro:arg name="y" default="0" />
+    <xacro:arg name="z" default="0" />
+    <xacro:arg name="roll" default="0" />
+    <xacro:arg name="pitch" default="0" />
+    <xacro:arg name="yaw" default="0" />
+    <xacro:arg name="initial_positions_file"
+        default="$(find moveit_pro_kr16)/config/initial_positions.yaml" />
+    <xacro:kuka_kr16_r2010_2_robot client_ip="$(arg client_ip)" client_port="$(arg client_port)"
+        prefix="$(arg prefix)" use_fake_hardware="$(arg use_fake_hardware)"
+        roundtrip_time="$(arg roundtrip_time)"
+        initial_positions_file="$(arg initial_positions_file)">
+        <origin xyz="$(arg x) $(arg y) $(arg z)" rpy="$(arg roll) $(arg pitch) $(arg yaw)" />
+    </xacro:kuka_kr16_r2010_2_robot>
 </robot>

File: src/moveit_pro_kuka_configs/moveit_pro_kr16/description/kr16_r2010_2_macro.xacro (robot description, xacro)
@@ -1,9 +1,9 @@
 <?xml version="1.0"?>
 <robot xmlns:xacro="http://wiki.ros.org/xacro">
-  <xacro:include filename="$(find kuka_cybertech_support)/urdf/kr_cybertech_ros2_control.xacro"/>
+  <xacro:include filename="$(find moveit_pro_kr16)/description/kr16_ros2_control.xacro"/>
   <xacro:include filename="$(find kuka_cybertech_support)/urdf/kr_cybertech_transmission.xacro"/>
-  <xacro:macro name="kuka_kr16_r2010_2_robot" params="client_ip client_port prefix use_fake_hardware roundtrip_time *origin">
+  <xacro:macro name="kuka_kr16_r2010_2_robot" params="client_ip client_port prefix use_fake_hardware roundtrip_time initial_positions_file *origin">
     <!-- ros2 control instance -->
-    <xacro:kuka_cybertech_ros2_control name="${prefix}kr16_r2010_2" client_ip="${client_ip}" client_port="${client_port}" prefix="${prefix}" use_fake_hardware="${use_fake_hardware}" roundtrip_time="${roundtrip_time}"/>
+    <xacro:kuka_cybertech_ros2_control name="${prefix}kr16_r2010_2" client_ip="${client_ip}" client_port="${client_port}" prefix="${prefix}" use_fake_hardware="${use_fake_hardware}" roundtrip_time="${roundtrip_time}" initial_positions_file="${initial_positions_file}"/>
     <link name="world"/>
     <link name="${prefix}base_link">
