Commit message: Update mounting position, format & update sim srdf

File: src/moveit_pro_franka_configs/franka_dual_arm_config/description/franka.urdf.xacro (robot description, xacro)
@@ -10,5 +10,5 @@
      <parent link="world"/>
      <child link = "right_mount"/>
-    <origin xyz="0 -0.06 0.342" rpy="0.8936 -0.1746 0.4636"/>
+    <origin xyz="0.035 -0.050681 0.356" rpy="0.8936 -0.1746 0.4636"/>
   </joint>
   <xacro:franka_robot arm_id="fr3"
@@ -39,5 +39,5 @@
      <parent link="world"/>
      <child link = "left_mount"/>
-    <origin xyz="0 0.06 0.342" rpy="-0.8936 -0.1746 -0.4636"/>
+    <origin xyz="0.035 0.050681 0.356" rpy="-0.8936 -0.1746 -0.4636"/>
   </joint>
   <xacro:franka_robot arm_id="fr3"

File: src/moveit_pro_franka_configs/franka_dual_arm_config_hw/description/franka.urdf.xacro (robot description, xacro)
@@ -11,5 +11,5 @@
      <parent link="world"/>
      <child link = "right_mount"/>
-    <origin xyz="-0.6 -0.050681 0.356" rpy="0 0 0"/>
+    <origin xyz="0.035 -0.050681 0.356" rpy="0.8936 -0.1746 0.4636"/>
   </joint>
   <xacro:franka_robot arm_id="fr3"
@@ -40,5 +40,5 @@
      <parent link="world"/>
      <child link = "left_mount"/>
-    <origin xyz="0.6 0.050681 0.356" rpy="0 0 0"/>
+    <origin xyz="0.035 0.050681 0.356" rpy="-0.8936 -0.1746 -0.4636"/>
   </joint>
   <xacro:franka_robot arm_id="fr3"
