Commit message: config working now
Signed-off-by: Paul Gesel <paul.gesel@picknik.ai>

Former-commit-id: 49ae79bd892295b482f2fb5eccc1eff8d36193f6

File: src/fanuc_config/description/crx10ia.urdf.xacro (robot description, xacro)
@@ -9,6 +9,6 @@
   <xacro:include filename="$(find fanuc_hardware_interface)/robot/fanuc_joint_control.xacro"/>
   <link name="world"/>
-  <link name="end_effector"/>
-  <xacro:crx10ia parent="world" child="end_effector">
+  <link name="grasp_link"/>
+  <xacro:crx10ia parent="world" child="grasp_link">
     <origin xyz="0 0 0" rpy="0 0 0"/>
   </xacro:crx10ia>

Commit message: update moveit config branch
Signed-off-by: Paul Gesel <paul.gesel@picknik.ai>

Former-commit-id: 1f66641f2306929b6714ddcba692ded86b839a3c

File: src/fanuc_config/description/crx10ia.urdf.xacro (robot description, xacro)
@@ -1,5 +1,5 @@
 <?xml version="1.0" ?>
 <robot name="crx10ia" xmlns:xacro="http://wiki.ros.org/xacro">
-  <xacro:arg name="robot_ip" default="192.168.1.100"/>
+  <xacro:arg name="robot_ip" default="$(arg robot_ip)"/>
   <xacro:arg name="rmi_port" default="16001"/>
   <xacro:arg name="stream_motion_port" default="60015"/>
@@ -7,5 +7,5 @@
   <xacro:arg name="payload_schedule" default="1"/>
   <xacro:include filename="$(find fanuc_crx_description)/urdf/crx10ia_macro.xacro"/>
-  <xacro:include filename="$(find fanuc_hardware_interface)/robot/fanuc_joint_control.xacro"/>
+  <xacro:include filename="$(find fanuc_hardware_interface)/robot/fanuc_control.xacro"/>
   <link name="world"/>
   <link name="grasp_link"/>
@@ -13,19 +13,4 @@
     <origin xyz="0 0 0" rpy="0 0 0"/>
   </xacro:crx10ia>
-  <ros2_control name="crx10ia" type="system">
-    <joint name="J1"/>
-    <joint name="J2"/>
-    <joint name="J3"/>
-    <joint name="J4"/>
-    <joint name="J5"/>
-    <joint name="J6"/>
-    <hardware>
-      <plugin>fanuc_robot_driver/FanucHardwareInterface</plugin>
-      <param name="robot_ip">$(arg robot_ip)</param>
-      <param name="rmi_port">$(arg rmi_port)</param>
-      <param name="stream_motion_port">$(arg stream_motion_port)</param>
-      <param name="io_configuration">$(arg io_configuration)</param>
-      <param name="payload_schedule">$(arg payload_schedule)</param>
-    </hardware>
-  </ros2_control>
+  <xacro:fanuc_control name="crx10ia"/>
 </robot>
