Commit message: Update mounting position, format & update sim srdf
Former-commit-id: 2c895e3acfedf77712b72c15692c1e6416c16bc9

File: src/moveit_pro_franka_configs/franka_dual_arm_sim/description/franka.urdf.xacro (robot description, xacro)
@@ -10,5 +10,5 @@
      <parent link="world"/>
      <child link = "right_mount"/>
-    <origin xyz="0 -0.06 0.342" rpy="0.8936 -0.1746 0.4636"/>
+    <origin xyz="0.035 -0.050681 0.356" rpy="0.8936 -0.1746 0.4636"/>
   </joint>
   <xacro:franka_robot arm_id="fr3"
@@ -39,5 +39,5 @@
      <parent link="world"/>
      <child link = "left_mount"/>
-    <origin xyz="0 0.06 0.342" rpy="-0.8936 -0.1746 -0.4636"/>
+    <origin xyz="0.035 0.050681 0.356" rpy="-0.8936 -0.1746 -0.4636"/>
   </joint>
   <xacro:franka_robot arm_id="fr3"

Commit message: Implemented gripper functionality for Franka dual arm sim.
Former-commit-id: d13d425541706b4711881b3e7658be65f1b72452

File: src/moveit_pro_franka_configs/franka_dual_arm_sim/description/franka.urdf.xacro (robot description, xacro)
@@ -30,7 +30,8 @@
                       connected_to= "right_mount">
   </xacro:franka_robot>
+  <!-- This link aligns the axes of the grasp frame to our required convention for motion planning tasks. -->
   <link name="right_grasp_link" />
   <joint name="right_grasp_link_joint" type="fixed">
-     <parent link="right_fr3_link8"/>
+     <parent link="right_fr3_hand_tcp"/>
      <child link = "right_grasp_link"/>
      <origin xyz="0 0 0" rpy="0 0 -1.5708"/>
@@ -59,8 +60,8 @@
                       connected_to= "left_mount">
   </xacro:franka_robot>
-    <!-- This link aligns the axes of the grasp frame to our required convention for motion planning tasks. -->
+   <!-- This link aligns the axes of the grasp frame to our required convention for motion planning tasks. -->
    <link name="left_grasp_link" />
    <joint name="left_grasp_link_joint" type="fixed">
-      <parent link="world"/>
+      <parent link="left_fr3_hand_tcp"/>
       <child link = "left_grasp_link"/>
       <origin xyz="0 0 0" rpy="0 0 -1.5708"/>
@@ -144,4 +145,15 @@
         <state_interface name="effort"/>
       </joint>
+      <joint name="right_fr3_finger_joint1">
+        <command_interface name="position">
+          <param name="min">-0.0</param>
+          <param name="max">0.04</param>
+        </command_interface>
+        <state_interface name="position">
+          <param name="initial_value">0.035</param>
+        </state_interface>
+        <state_interface name="velocity"/>
+        <state_interface name="effort"/>
+      </joint>
       <joint name="left_fr3_joint1">
         <command_interface name="position">
@@ -217,4 +229,15 @@
         <state_interface name="position">
           <param name="initial_value">0.7853</param>
+        </state_interface>
+        <state_interface name="velocity"/>
+        <state_interface name="effort"/>
+      </joint>
+      <joint name="left_fr3_finger_joint1">
+        <command_interface name="position">
+          <param name="min">-0.0</param>
+          <param name="max">0.04</param>
+        </command_interface>
+        <state_interface name="position">
+          <param name="initial_value">0.035</param>
         </state_interface>
         <state_interface name="velocity"/>
@@ -227,6 +250,6 @@
         <param name="render_publish_rate">10</param>
         <param name="tf_publish_rate">60</param>
-        <param name="mujoco_viewer">false</param>
         <param name="mujoco_keyframe">home</param>
+        <param name="mujoco_viewer">$(arg mujoco_viewer)</param>
       </hardware>
     </ros2_control>
