Commit message: Update Franka description repo and upgrade Franka meshes.
Former-commit-id: 11e17194b0f836edb3f0df7fa48b1f841a87ce1f

File: src/moveit_pro_franka_configs/dual_arm_sim/description/franka.urdf.xacro (robot description, xacro)
@@ -4,11 +4,20 @@
   <xacro:arg name="ee_id" default="franka_hand" />
   <xacro:arg name="rpy_ee" default="0 0 -0.785" />
+  <!-- Load Franka Duo Mount -->
+  <xacro:include filename="$(find franka_description)/robots/fr3_duo/fr3_duo_mount/fr3_duo_mount.xacro"/>
+  <xacro:property name="mount_kinematics" value="${xacro.load_yaml('$(find franka_description)/robots/fr3_duo/fr3_duo_mount/kinematics.yaml')}" />
   <!-- Load Franka robot -->
   <xacro:include filename="$(find franka_description)/robots/common/franka_robot.xacro"/>
   <link name="world" />
+  <xacro:mount name="fr3_duo"
+               parent="world"
+               inertials="${xacro.load_yaml('$(find franka_description)/robots/fr3_duo/fr3_duo_mount/inertials.yaml')}">
+    <origin xyz="0.0 0.0 0.305115" rpy="0 0 0" />
+  </xacro:mount>
   <joint name="right_mount_joint" type="fixed">
-     <parent link="world"/>
+     <parent link="mount_link"/>
      <child link = "right_mount"/>
-    <origin xyz="0.035 -0.050681 0.356" rpy="0.8936 -0.1746 0.4636"/>
+     <origin xyz="${mount_kinematics['right']['kinematic']['x']} ${mount_kinematics['right']['kinematic']['y']} ${mount_kinematics['right']['kinematic']['z']}"
+             rpy="${mount_kinematics['right']['kinematic']['roll']} ${mount_kinematics['right']['kinematic']['pitch']} ${mount_kinematics['right']['kinematic']['yaw']}"/>
   </joint>
   <xacro:franka_robot arm_id="fr3"
@@ -19,4 +28,5 @@
                       gazebo="false"
                       hand="true"
+                      tcp_xyz="0 0 0.1034"
                       ee_id="$(arg ee_id)"
                       with_sc="false"
@@ -27,6 +37,6 @@
                       gazebo_effort="false"
                       no_prefix="false"
-                      arm_prefix="right"
-                      connected_to= "right_mount">
+                      arm_prefix="right_"
+                      connected_to= "right_mount"> <!-- This also creates the link right_mount -->
   </xacro:franka_robot>
   <!-- This link aligns the axes of the grasp frame to our required convention for motion planning tasks. -->
@@ -38,7 +48,8 @@
   </joint>
   <joint name="left_mount_joint" type="fixed">
-     <parent link="world"/>
+     <parent link="mount_link"/>
      <child link = "left_mount"/>
-    <origin xyz="0.035 0.050681 0.356" rpy="-0.8936 -0.1746 -0.4636"/>
+     <origin xyz="${mount_kinematics['left']['kinematic']['x']} ${mount_kinematics['left']['kinematic']['y']} ${mount_kinematics['left']['kinematic']['z']}"
+             rpy="${mount_kinematics['left']['kinematic']['roll']} ${mount_kinematics['left']['kinematic']['pitch']} ${mount_kinematics['left']['kinematic']['yaw']}"/>
   </joint>
   <xacro:franka_robot arm_id="fr3"
@@ -49,4 +60,5 @@
                       gazebo="false"
                       hand="true"
+                      tcp_xyz="0 0 0.1034"
                       ee_id="$(arg ee_id)"
                       with_sc="false"
@@ -57,6 +69,6 @@
                       gazebo_effort="false"
                       no_prefix="false"
-                      arm_prefix="left"
-                      connected_to= "left_mount">
+                      arm_prefix="left_"
+                      connected_to= "left_mount"> <!-- This also creates the link left_mount -->
   </xacro:franka_robot>
    <!-- This link aligns the axes of the grasp frame to our required convention for motion planning tasks. -->

File: src/moveit_pro_franka_configs/franka_arm_hw/description/franka.urdf.xacro (robot description, xacro)
@@ -13,4 +13,5 @@
                       gazebo="false"
                       hand="true"
+                      tcp_xyz="0 0 0.1034"
                       ee_id="$(arg ee_id)"
                       with_sc="false"

File: src/moveit_pro_franka_configs/franka_dual_arm_hw/description/franka.urdf.xacro (robot description, xacro)
@@ -20,4 +20,5 @@
                       gazebo="false"
                       hand="true"
+                      tcp_xyz="0 0 0.1034"
                       ee_id="$(arg ee_id)"
                       with_sc="false"
@@ -28,5 +29,5 @@
                       gazebo_effort="false"
                       no_prefix="false"
-                      arm_prefix="right"
+                      arm_prefix="right_"
                       connected_to= "right_mount">
   </xacro:franka_robot>
@@ -49,4 +50,5 @@
                       gazebo="false"
                       hand="true"
+                      tcp_xyz="0 0 0.1034"
                       ee_id="$(arg ee_id)"
                       with_sc="false"
@@ -57,5 +59,5 @@
                       gazebo_effort="false"
                       no_prefix="false"
-                      arm_prefix="left"
+                      arm_prefix="left_"
                       connected_to= "left_mount">
   </xacro:franka_robot>

File: src/moveit_pro_franka_configs/kitchen_sim/description/franka.urdf.xacro (robot description, xacro)
@@ -13,4 +13,5 @@
                       gazebo="false"
                       hand="true"
+                      tcp_xyz="0 0 0.1034"
                       ee_id="$(arg ee_id)"
                       with_sc="false"
