Commit message: fix(viz): decimate d415 camera mesh under the 10 MB URDF load gate
The realsense2_description d415.stl is a 425k-triangle / 21 MB Catia export
that trips the MoveIt Pro UI's 10 MB-per-mesh URDF load gate (moveit_pro#19448),
so configs with use_mesh=true fail to render the camera in the 3D view.

- Vendor a quadric-decimated d415.stl into picknik_accessories
  (descriptions/sensors/, 85k tris / ~4.1 MB, bbox preserved within ~0.5%).
- Repoint the shared realsense_d415.urdf.xacro mesh from
  package://realsense2_description/meshes/d415.stl to the vendored copy,
  fixing every config that uses the mesh (UR, Kinova, satellite) in one line.
  realsense2_description stays a dep for its _materials / _usb_plug includes.

The phoebe_ws submodule has its own realsense2_description d415 reference; it
is a separate repo and out of scope here.

Co-Authored-By: Claude Opus 4.8 (1M context) <noreply@anthropic.com>

File: src/picknik_accessories/descriptions/sensors/realsense_d415.urdf.xacro (robot description, xacro)
@@ -46,5 +46,5 @@
           <origin xyz="${d415_cam_mount_from_center_offset} ${-d415_cam_depth_py} 0" rpy="${M_PI/2} 0 ${M_PI/2}"/>
           <geometry>
-            <mesh filename="package://realsense2_description/meshes/d415.stl" />
+            <mesh filename="package://picknik_accessories/descriptions/sensors/d415.stl" />
           </geometry>
         </xacro:if>
