Commit message: Add test of scan and plan example - generating mesh normals works, but I really need just a half mesh if I want planning to be feasible
Former-commit-id: 76143c17150c796f97d428ef3c133ec543d544d0

File: src/lab_sim/description/picknik_ur.xacro (robot description, xacro)
@@ -1187,7 +1187,31 @@
     <origin rpy="0 0 0" xyz="0 1 0.45" />
   </joint>
+  <link name="workpiece">
+    <visual>
+      <origin rpy="0 0 0" xyz="0 0 0" />
+      <geometry>
+        <mesh
+          filename="package://ur_description/meshes/ur5e/collision/forearm.stl"
+        />
+      </geometry>
+    </visual>
+    <collision>
+      <origin rpy="0 0 0" xyz="0 0 0" />
+      <geometry>
+        <mesh
+          filename="package://ur_description/meshes/ur5e/collision/forearm.stl"
+        />
+      </geometry>
+    </collision>
+  </link>
+  <joint name="workpiece_joint" type="fixed">
+    <parent link="world" />
+    <child link="workpiece" />
+    <origin rpy="0 0 0" xyz="0 0.5 0.75" />
+  </joint>
   <ros2_control name="ur_mujoco_control" type="system">
     <hardware>
       <plugin>picknik_mujoco_ros/MujocoSystem</plugin>
+      <param name="mujoco_viewer">false</param>
       <param name="mujoco_model">$(arg mujoco_model)</param>
       <param name="mujoco_model_package">lab_sim</param>

Commit message: turn the realsense camera into a box
Former-commit-id: e6a1fb1512c81c6e7106bf31e8109e98169fa6ad

File: src/lab_sim/description/picknik_ur.xacro (robot description, xacro)
@@ -104,13 +104,19 @@
   <link name="wrist_mounted_camera_link">
     <visual>
-      <origin
-        rpy="1.5707963267948966 0 1.5707963267948966"
-        xyz="0.00987 -0.02 0"
-      />
-      <geometry>
-        <mesh filename="package://realsense2_description/meshes/d415.stl" />
+      <origin rpy="0 0 0" xyz="0 -0.02 0" />
+      <geometry>
+        <box size="0.02005 0.099 0.023" />
       </geometry>
       <material name="rs_aluminum">
         <color rgba="0.5 0.5 0.5 1.0" />
+      </material>
+    </visual>
+    <visual>
+      <origin rpy="0 0 0" xyz="0.010525 -0.02 0" />
+      <geometry>
+        <box size="0.001 0.099 0.023" />
+      </geometry>
+      <material name="black">
+        <color rgba="0.0 0.0 0.0 1.0" />
       </material>
     </visual>

File: src/moveit_pro_kinova_configs/kinova_gen3_base_config/description/robotiq_2f_85_gripper.urdf (robot description, URDF)
Before this commit: robot ur5e_gripper_and_camera, 28 links, 27 joints
Links:
- link wrist_mounted_camera_link: geometry collision box size=0.02005 0.099 0.023; visual box size=0.001 0.099 0.023

Commit message: remove table from urdf
Former-commit-id: 55cba0b96341205e59ec12807a5a2a72cbbc4a36

File: src/lab_sim/description/picknik_ur.xacro (robot description, xacro)
@@ -1173,24 +1173,4 @@
     <dynamics damping="20.0" friction="500.0" />
   </joint>
-  <!-- Table -->
-  <link name="table">
-    <visual>
-      <origin rpy="0 0 0" xyz="0 0 -0.45" />
-      <geometry>
-        <box size="3.5 1 0.9" />
-      </geometry>
-    </visual>
-    <collision>
-      <origin rpy="0 0 0" xyz="0 0 -0.45" />
-      <geometry>
-        <box size="3.5 1 0.9" />
-      </geometry>
-    </collision>
-  </link>
-  <joint name="table_joint" type="fixed">
-    <parent link="world" />
-    <child link="table" />
-    <origin rpy="0 0 0" xyz="0 1 0.45" />
-  </joint>
   <ros2_control name="ur_mujoco_control" type="system">
     <hardware>

Commit message: Update bottle mesh and reduced gripper force
Former-commit-id: 61ac16fd8246f0385e2fe66fcd13c1d52201d85c

File: src/lab_sim/description/picknik_ur.xacro (robot description, xacro)
@@ -598,5 +598,5 @@
     <axis xyz="0 -1 0" />
     <origin rpy="0 0 0" xyz="0.03060114 0.0 0.05490452" />
-    <limit effort="50" lower="0.0" upper="0.8" velocity="0.5" />
+    <limit effort="3" lower="0.0" upper="0.8" velocity="0.5" />
   </joint>
   <joint name="robotiq_85_right_knuckle_joint" type="revolute">
@@ -605,5 +605,5 @@
     <axis xyz="0 1 0" />
     <origin rpy="0 0 0" xyz="-0.03060114 0.0 0.05490452" />
-    <limit effort="50" lower="0.0" upper="0.8" velocity="0.5" />
+    <limit effort="3" lower="0.0" upper="0.8" velocity="0.5" />
     <mimic joint="robotiq_85_left_knuckle_joint" multiplier="1" />
   </joint>

Commit message: Apply suggestions from code review
Former-commit-id: f2ae8240078218964e49cb25ec915586cba997f9

File: src/lab_sim/description/picknik_ur.xacro (robot description, xacro)
@@ -598,5 +598,5 @@
     <axis xyz="0 -1 0" />
     <origin rpy="0 0 0" xyz="0.03060114 0.0 0.05490452" />
-    <limit effort="3" lower="0.0" upper="0.8" velocity="0.5" />
+    <limit effort="20" lower="0.0" upper="0.8" velocity="0.5" />
   </joint>
   <joint name="robotiq_85_right_knuckle_joint" type="revolute">
@@ -605,5 +605,5 @@
     <axis xyz="0 1 0" />
     <origin rpy="0 0 0" xyz="-0.03060114 0.0 0.05490452" />
-    <limit effort="3" lower="0.0" upper="0.8" velocity="0.5" />
+    <limit effort="20" lower="0.0" upper="0.8" velocity="0.5" />
     <mimic joint="robotiq_85_left_knuckle_joint" multiplier="1" />
   </joint>

Commit message: Changes to replicate  move_group error

File: src/lab_sim/description/picknik_ur.xacro (robot description, xacro)
@@ -655,5 +655,6 @@
   <link name="grasp_link" />
   <joint name="grasp_link_joint" type="fixed">
-    <parent link="robotiq_85_base_link" />
+    <!-- <parent link="robotiq_85_base_link" /> -->
+    <parent link="gripper_mount_link" />
     <child link="grasp_link" />
     <origin rpy="0.0 0.0 3.141592653589793" xyz="0.0 0.0 0.134" />

Commit message: feat(lab_sim): improve scene render quality
- scene.xml: add 4x MSAA + 4096px shadows to the <visual> block
- lab_desk granite table top: replace the black checker texture with a
  solid polished dark granite (specular/shininess + reflectance="0.7")
- linear rail: make the three rail geoms opaque (alpha 0.4 -> 1)
- robot pedestal: anodized-aluminum look in both the MuJoCo scene and the
  URDF (matching "pedestal_metal" color; base_link previously had no
  material). Solid shaded color + specular sheen rather than a procedural
  texture, since high-frequency texture aliases/shimmers under minification
  as the pedestal moves toward/away from the camera.

File: src/lab_sim/description/picknik_ur.xacro (robot description, xacro)
@@ -11,4 +11,7 @@
   <material name="offwhite">
     <color rgba="0.01 0.01 0.01 1" />
+  </material>
+  <material name="pedestal_metal">
+    <color rgba="0.22 0.23 0.25 1" />
   </material>
   <link name="world" />
@@ -778,4 +781,5 @@
         <box size="0.16 0.2 0.4" />
       </geometry>
+      <material name="pedestal_metal" />
     </visual>
     <collision>
