Commit message: Add collision geometry to base_link in lab_sim URDF
The base_link pedestal had a visual box but no collision element,
causing KeepOutZone collision checking to miss the robot platform.

Fixes #16960

Co-Authored-By: Claude Opus 4.6 <noreply@anthropic.com>

File: src/lab_sim/description/picknik_ur.xacro (robot description, xacro)
@@ -779,4 +779,10 @@
       </geometry>
     </visual>
+    <collision>
+      <origin rpy="0 0 0" xyz="0.0 0.0 -0.2" />
+      <geometry>
+        <box size="0.16 0.2 0.4" />
+      </geometry>
+    </collision>
   </link>
   <link name="base_link_inertia">

Commit message: Add lab desk objects, adjust collision wall/tray positions, and clean up lab_sim
Co-Authored-By: Claude Opus 4.6 <noreply@anthropic.com>

File: src/lab_sim/description/picknik_ur.xacro (robot description, xacro)
@@ -664,5 +664,5 @@
       <origin rpy="0 0 0" xyz="0 0 0" />
       <geometry>
-        <box size="5.0 0.6 0.30" />
+        <box size="5.0 0.2 0.30" />
       </geometry>
       <material name="grey">
@@ -673,5 +673,5 @@
       <origin rpy="0 0 0" xyz="0 0.14 0.125" />
       <geometry>
-        <box size="5.0 0.2 0.5" />
+        <box size="5.0 0.12 0.5" />
       </geometry>
       <material name="grey">
@@ -682,5 +682,5 @@
       <origin rpy="0 0 0" xyz="0 -0.22 0.125" />
       <geometry>
-        <box size="5.0 0.12 0.5" />
+        <box size="5.0 0.08 0.5" />
       </geometry>
       <material name="grey">
@@ -691,5 +691,5 @@
       <origin rpy="0 0 0" xyz="0 0 0" />
       <geometry>
-        <box size="5.0 0.6 0.3" />
+        <box size="5.0 0.2 0.3" />
       </geometry>
       <material name="grey">
@@ -700,5 +700,5 @@
       <origin rpy="0 0 0" xyz="0 0.14 0.125" />
       <geometry>
-        <box size="5.0 0.2 0.5" />
+        <box size="5.0 0.12 0.5" />
       </geometry>
       <material name="grey">
@@ -709,5 +709,5 @@
       <origin rpy="0 0 0" xyz="0 -0.22 0.125" />
       <geometry>
-        <box size="5.0 0.12 0.5" />
+        <box size="5.0 0.08 0.5" />
       </geometry>
       <material name="grey">

Commit message: feat(lab_sim): select the camera renderer from one setting
MOVEIT_PRO_CAMERA_RENDERER picks mujoco (the default), nyx, or both. The
robot description resolves the MuJoCo camera and point-cloud rates from it
and runtime.launch.xml reads the same variable to decide whether to start
picknik_nyx_renderer, so the two halves cannot disagree.

The point-cloud rate has to follow the render rate rather than stand alone:
the cloud timer publishes what the render timer produced, so running it
against a stopped renderer reports every camera as never having rendered.
Nyx has no depth output, so selecting it gives up point clouds.

An unrecognized value fails the description rather than leaving the config
with no cameras and no explanation.

Needs the Nyx renderer package, which is not in a released image yet, so
anything other than the default requires a moveit_pro build that carries it.

Co-Authored-By: Claude Opus 5 (1M context) <noreply@anthropic.com>
Claude-Session: https://claude.ai/code/session_019YCk2yNsEQkVUSvhAmsJ4m

File: src/lab_sim/description/picknik_ur.xacro (robot description, xacro)
@@ -3,4 +3,13 @@
   <xacro:arg name="mujoco_model" default="description/scene.xml" />
   <xacro:arg name="mujoco_model_package" default="lab_sim" />
+  <!-- Which renderer produces this config's camera topics: mujoco (the default), nyx, or both on separate topics. runtime.launch.xml reads the same variable to decide whether to start the Nyx node, so the two halves cannot disagree. An unrecognized value fails the description rather than leaving the config with no cameras. -->
+  <xacro:arg
+    name="camera_renderer"
+    default="$(optenv MOVEIT_PRO_CAMERA_RENDERER mujoco)"
+  />
+  <xacro:property
+    name="mujoco_cameras"
+    value="${ dict(mujoco=True, nyx=False, both=True)['$(arg camera_renderer)'] }"
+  />
   <xacro:arg
     name="point_cloud_publish_rate"
@@ -1196,8 +1205,8 @@
       <param name="mujoco_model">$(arg mujoco_model)</param>
       <param name="mujoco_model_package">$(arg mujoco_model_package)</param>
-      <!-- The rate <camera> data is published at -->
-      <param name="render_publish_rate">10</param>
-      <!-- The rate point clouds generated from depth images are published at -->
-      <param name="point_cloud_publish_rate">$(arg point_cloud_publish_rate)</param>
+      <!-- The rate <camera> data is published at. Zero switches MuJoCo's cameras off: the image timer is only created for a non-zero rate. -->
+      <param name="render_publish_rate">${10 if mujoco_cameras else 0}</param>
+      <!-- The rate point clouds generated from depth images are published at. Zero for the same reason, and it follows the render rate rather than standing alone: the cloud timer publishes what the render timer produced, so against a stopped renderer it would report every camera as never having rendered. Nyx has no depth output, so selecting it gives up point clouds. -->
+      <param name="point_cloud_publish_rate">${$(arg point_cloud_publish_rate) if mujoco_cameras else 0}</param>
       <!-- The rate transforms to <site> poses are published at -->
       <param name="tf_publish_rate">60</param>

Commit message: fix(lab_sim): harden the camera renderer selector
An empty MOVEIT_PRO_CAMERA_RENDERER failed the robot description.
moveit_pro's validator accepts an empty value and docker-compose forwards
it as-is, so a bare assignment in the workspace .env took the description
down. The value is now bound to a property and read as data, with an
empty value treated as opengl, which also keeps a quote in the value from
closing the string literal and being evaluated instead of compared.

The lab_sim and april_tag_sim integration tests pin the renderer to
opengl so colcon test does not depend on a developer's exported value,
and .nyx_scenes/ is ignored, where nyx_export_scene writes hundreds of
megabytes inside $USER_WS.

Co-Authored-By: Claude Opus 5 (1M context) <noreply@anthropic.com>

File: src/lab_sim/description/picknik_ur.xacro (robot description, xacro)
@@ -8,4 +8,5 @@
     default="$(optenv MOVEIT_PRO_CAMERA_RENDERER opengl)"
   />
+  <xacro:property name="camera_renderer" value="$(arg camera_renderer)" />
   <xacro:arg
     name="point_cloud_publish_rate"
@@ -1214,5 +1215,5 @@
     <!-- nyx: the Nyx nodes publish <camera>/color and camera_info, so MuJoCo publishes only depth and points. -->
     <xacro:if
-      value="${ dict(opengl=False, nyx=True, both=False)['$(arg camera_renderer)'] }"
+      value="${ dict(opengl=False, nyx=True, both=False)[camera_renderer or 'opengl'] }"
     >
       <sensor name="scene_camera">
@@ -1225,5 +1226,5 @@
     <!-- both: each renderer's color image goes under its own prefix, so no consumer reads one renderer while expecting the other. Depth and points stay unprefixed. -->
     <xacro:if
-      value="${ dict(opengl=False, nyx=False, both=True)['$(arg camera_renderer)'] }"
+      value="${ dict(opengl=False, nyx=False, both=True)[camera_renderer or 'opengl'] }"
     >
       <sensor name="scene_camera">

Commit message: refactor(picknik_accessories): share the camera renderer sensors macro
MOVEIT_PRO_CAMERA_RENDERER applies to every MuJoCo config, so the arg,
the validation and the per-camera <sensor> blocks move into
picknik_accessories, which the configs already depend on, and lab_sim
includes them and passes its camera list. A config with other cameras
sets nyx_cameras in urdf_params or calls the macro with its own list.

Co-Authored-By: Claude Opus 5 (1M context) <noreply@anthropic.com>

File: src/lab_sim/description/picknik_ur.xacro (robot description, xacro)
@@ -3,10 +3,9 @@
   <xacro:arg name="mujoco_model" default="description/scene.xml" />
   <xacro:arg name="mujoco_model_package" default="lab_sim" />
-  <!-- Which renderer produces the cameras' color topics. runtime.launch.xml starts a Nyx node per camera. -->
-  <xacro:arg
-    name="camera_renderer"
-    default="$(optenv MOVEIT_PRO_CAMERA_RENDERER opengl)"
+  <xacro:include
+    filename="$(find picknik_accessories)/descriptions/sensors/camera_renderer.urdf.xacro"
   />
-  <xacro:property name="camera_renderer" value="$(arg camera_renderer)" />
+  <!-- The cameras MOVEIT_PRO_CAMERA_RENDERER applies to. A config reusing this description with other cameras sets nyx_cameras in urdf_params, and its runtime.launch.xml starts one Nyx node per name. -->
+  <xacro:arg name="nyx_cameras" default="scene_camera wrist_camera" />
   <xacro:arg
     name="point_cloud_publish_rate"
@@ -1213,28 +1212,5 @@
       <param name="mujoco_viewer">$(arg mujoco_viewer)</param>
     </hardware>
-    <!-- nyx: the Nyx nodes publish <camera>/color and camera_info, so MuJoCo publishes only depth and points. -->
-    <xacro:if
-      value="${ dict(opengl=False, nyx=True, both=False)[camera_renderer or 'opengl'] }"
-    >
-      <sensor name="scene_camera">
-        <param name="color_enabled">false</param>
-      </sensor>
-      <sensor name="wrist_camera">
-        <param name="color_enabled">false</param>
-      </sensor>
-    </xacro:if>
-    <!-- both: each renderer's color image goes under its own prefix, so no consumer reads one renderer while expecting the other. Depth and points stay unprefixed. -->
-    <xacro:if
-      value="${ dict(opengl=False, nyx=False, both=True)[camera_renderer or 'opengl'] }"
-    >
-      <sensor name="scene_camera">
-        <param name="rgb_topic">scene_camera/opengl/color</param>
-        <param name="camera_info_topic">scene_camera/opengl/camera_info</param>
-      </sensor>
-      <sensor name="wrist_camera">
-        <param name="rgb_topic">wrist_camera/opengl/color</param>
-        <param name="camera_info_topic">wrist_camera/opengl/camera_info</param>
-      </sensor>
-    </xacro:if>
+    <xacro:camera_renderer_sensors cameras="$(arg nyx_cameras)" />
   </ros2_control>
 </robot>
