Commit message: fix(kinova_vla_test_sim): fork local SRDF to drop dangling camera/gripper warnings, fix serve_policy docs
The xacro dropped the RealSense mesh/scene_camera link but the SRDF (shared
verbatim from kinova_sim) still referenced it in disable_collisions entries,
and the gripper's non-mimic finger joints were never marked passive or given
group_state values. Fork a local SRDF so this config's collision matrix and
group_state actually match its own URDF, and drop the now-unused
external_camera/wrist_realsense urdf_params.

Also document --service-ports on the serve_policy run command; docker compose
run does not publish a service's ports by default, so omitting it left the
bridge unable to reach the inference server.

Co-Authored-By: Claude Sonnet 5 <noreply@anthropic.com>

File: src/moveit_pro_kinova_configs/kinova_vla_test_sim/description/picknik_kinova_gen3.xacro (robot description, xacro)
@@ -553,14 +553,4 @@
       <origin xyz="0 0 0.15" rpy="0 0 0"/>
     </joint>
-    <!-- Camera External -->
-    <link name="external_camera_link" />
-    <joint name="external_camera_joint" type="fixed">
-      <parent link="world" />
-      <child link="external_camera_link" />
-      <origin xyz="-0.3 0.3 1.0" rpy="0.0 0.4 0" />
-    </joint>
-    <xacro:realsense_d415 parent="external_camera_link" name="scene_camera">
-      <origin xyz="0 0 0" rpy="0 0 0" />
-    </xacro:realsense_d415>
     <ros2_control name="kinova_mujoco_simulation" type="system">
       <joint name="joint_1">
