Commit message: fix(husky_a300_mock): correct ground-contact frame and lint test_depends
Captain-ruled fix for the base-footprint-above-ground finding: the
vendored A300 description's own base_footprint_joint sits 0.30 m above
true ground contact (an upstream clearpath_common authoring bug, not
introduced here). Keep the vendored file byte-identical to upstream;
add a workspace-local "footprint" frame as base_link's parent, carrying
the FK-measured 0.13597 m ground-contact offset, and repoint
platform_velocity_controller's base_frame_id at it so TF, the 3D
Visualizer, and future Nav2 costmaps all agree the wheels sit on the
grid.

Also declares the sibling-package-convention lint test_depends
(ament_cmake_copyright, ament_cmake_lint_cmake, ament_flake8,
picknik_ament_copyright) so the BUILD_TESTING lint block isn't inert.

File: src/husky_a300_mock/description/husky_a300_blank_world.xacro (robot description, xacro)
@@ -17,4 +17,22 @@
   <xacro:include filename="$(find clearpath_platform_description)/urdf/a300/a300.urdf.xacro" />
   <xacro:a300 control="diff_4wd" front_wheels="outdoor" rear_wheels="outdoor" />
+  <!-- Known upstream artifact: a300.urdf.xacro's own base_footprint_joint (chassis_link ->
+       base_footprint, origin z=front_wheel_radius) puts base_footprint 0.30 m ABOVE true ground
+       contact instead of on it - the sign should carry the wheel-center offset the other way.
+       FK-measured against this file's own generated URDF: base_link=[0,0,0], front wheel
+       centers=[...,0.0291], wheel radius=0.1651 -> true ground contact is 0.13597 m BELOW
+       base_link. We can't fix that vendored joint in place (it would mean editing the vendored
+       clearpath_platform_description package, which this file keeps byte-identical to upstream)
+       and we can't add a second link literally named "base_footprint" either (URDF requires
+       unique link names; confirmed check_urdf rejects the duplicate). So this adds a
+       REP105-shaped ground frame under a different name, "footprint", that becomes base_link's
+       real parent - the wheel-radius/wheel-center numbers above are the platform_velocity_
+       controller's own SRDF/description geometry, not customer-specific measurements. -->
+  <link name="footprint" />
+  <joint name="footprint_joint" type="fixed">
+    <parent link="footprint" />
+    <child link="base_link" />
+    <origin xyz="0 0 0.13597" rpy="0 0 0" />
+  </joint>
   <!-- Attachments: the standard A300 accessory kit (front/rear bumper, sensor enclosure, sensor
        arch), for visual/body fidelity with the real robot. No sensors are mounted - sensors are out
