Commit message: feat(so101_sim): replace the stock SO-101 jaws with the XLeRobot fin gripper
The maintainer's bench arm runs XLeRobot's soft fin-ray gripper, so the mock
twin should show the same hand. `hardware/SO101_soft_fin.stl` upstream is one
binary STL holding three disconnected bodies on a print plate; they split into
the fixed-jaw body (52 x 48.6 x 65.2 mm), the moving-jaw body
(36.7 x 20.3 x 48 mm) and the TPU fin-ray finger (67.2 x 24.2 x 24.1 mm), which
is used twice, once per jaw.

Both jaw bodies are the stock parts with the moulded finger cut off and a
two-screw fork added; the servo bracket and the pivot yoke are untouched. Each
was rigidly registered onto the part it replaces and is stored in that part's
mesh frame, so the URDF reuses the visual origin the stock mesh already used.
83% of the fin fixed-jaw surface and 64% of the fin moving-jaw surface land
within 0.1 mm of the stock geometry; the rest is the new fork.

The finger is stored once in a frame built from its own screw bores, so each of
its two placements is just that jaw's bore frame. The bores fix the pose up to a
180 degree spin about the finger's long axis; the two fins are mirrored, ribs
facing inward across the grasp, matching XLeRobot's photo of the assembled
gripper.

Mock only: no MuJoCo, no compliance modelling. The fins are rigid meshes.

The single revolute `gripper` joint, its axis and limits, the ros2_control
block, the controllers and config.yaml are all untouched.

Co-Authored-By: Claude Opus 5 <noreply@anthropic.com>

File: src/so101_sim/description/so101.urdf.xacro (robot description, xacro)
@@ -33,4 +33,7 @@
     <color rgba="0.1 0.1 0.1 1.0"/>
   </material>
+  <material name="tpu_fin">
+    <color rgba="0.12 0.12 0.13 1.0"/>
+  </material>
   <!-- Link overhead camera mount -->
   <link name="overhead_camera_mount_link">
@@ -376,9 +379,12 @@
       </geometry>
     </collision>
-    <!-- Part wrist_roll_follower_so101_v1 -->
+    <!-- Part soft_fin_fixed_jaw: the XLeRobot fin-gripper replacement for
+         wrist_roll_follower_so101_v1. Same servo bracket and the same mesh
+         frame as the stock part, so this keeps the stock part's origin; the
+         moulded fixed finger is gone, replaced by the fork below. -->
     <visual>
       <origin xyz="8.32667e-17 -0.000218214 0.000949706" rpy="-3.14159 -5.55112e-17 0"/>
       <geometry>
-        <mesh filename="package://so101_sim/description/assets/wrist_roll_follower_so101_v1.stl"/>
+        <mesh filename="package://so101_sim/description/assets/soft_fin_fixed_jaw.stl"/>
       </geometry>
       <material name="3d_printed"><color rgba="0.05 0.05 0.05 1.0"/></material>
@@ -387,5 +393,21 @@
       <origin xyz="8.32667e-17 -0.000218214 0.000949706" rpy="-3.14159 -5.55112e-17 0"/>
       <geometry>
-        <mesh filename="package://so101_sim/description/assets/wrist_roll_follower_so101_v1.stl"/>
+        <mesh filename="package://so101_sim/description/assets/soft_fin_fixed_jaw_collision.stl"/>
+      </geometry>
+    </collision>
+    <!-- Part soft_fin_finger, fixed side. The finger mesh is stored in a frame
+         built from its own screw pair, so this origin is just the fixed jaw's
+         two-bore frame. -->
+    <visual>
+      <origin xyz="-0.02275 0.000781901 -0.0425503" rpy="2.66224e-06 -0.0806329 -2.14431e-07"/>
+      <geometry>
+        <mesh filename="package://so101_sim/description/assets/soft_fin_finger.stl"/>
+      </geometry>
+      <material name="tpu_fin"><color rgba="0.12 0.12 0.13 1.0"/></material>
+    </visual>
+    <collision>
+      <origin xyz="-0.02275 0.000781901 -0.0425503" rpy="2.66224e-06 -0.0806329 -2.14431e-07"/>
+      <geometry>
+        <mesh filename="package://so101_sim/description/assets/soft_fin_finger.stl"/>
       </geometry>
     </collision>
@@ -457,9 +479,12 @@
       <inertia ixx="6.61427e-06" ixy="-3.19807e-07" ixz="-5.90717e-09" iyy="1.89032e-06" iyz="-1.09945e-07" izz="5.28738e-06"/>
     </inertial>
-    <!-- Part moving_jaw_so101_v1 -->
+    <!-- Part soft_fin_moving_jaw: the XLeRobot fin-gripper replacement for
+         moving_jaw_so101_v1. Same pivot yoke and mesh frame as the stock part,
+         so this keeps the stock part's origin; the moulded blade is gone,
+         replaced by the fork below. -->
     <visual>
       <origin xyz="-5.55112e-17 -5.55112e-17 0.0189" rpy="9.53145e-17 6.93889e-18 1.24077e-24"/>
       <geometry>
-        <mesh filename="package://so101_sim/description/assets/moving_jaw_so101_v1.stl"/>
+        <mesh filename="package://so101_sim/description/assets/soft_fin_moving_jaw.stl"/>
       </geometry>
       <material name="3d_printed"><color rgba="0.05 0.05 0.05 1.0"/></material>
@@ -468,5 +493,19 @@
       <origin xyz="-5.55112e-17 -5.55112e-17 0.0189" rpy="9.53145e-17 6.93889e-18 1.24077e-24"/>
       <geometry>
-        <mesh filename="package://so101_sim/description/assets/moving_jaw_so101_v1.stl"/>
+        <mesh filename="package://so101_sim/description/assets/soft_fin_moving_jaw_collision.stl"/>
+      </geometry>
+    </collision>
+    <!-- Part soft_fin_finger, moving side: the moving jaw's two-bore frame. -->
+    <visual>
+      <origin xyz="-0.00115 -0.0222 0.0181" rpy="1.5708 -1.07812e-17 3.10121"/>
+      <geometry>
+        <mesh filename="package://so101_sim/description/assets/soft_fin_finger.stl"/>
+      </geometry>
+      <material name="tpu_fin"><color rgba="0.12 0.12 0.13 1.0"/></material>
+    </visual>
+    <collision>
+      <origin xyz="-0.00115 -0.0222 0.0181" rpy="1.5708 -1.07812e-17 3.10121"/>
+      <geometry>
+        <mesh filename="package://so101_sim/description/assets/soft_fin_finger.stl"/>
       </geometry>
     </collision>

Commit message: feat(so101_sim): drive the physical arm over the Feetech STS3215 bus
Fill in the `hardware_interface:=real` branch of the SO-101 URDF so MoveIt
Pro's controllers reach the follower arm's servos, and document the bench
procedure for bringing it up. Mock is untouched and stays the default.

- `feetech_ros2_driver` 0.2.2 is a released Jazzy package, so it is an
  `exec_depend` rather than a vendored snapshot: the Dockerfile's existing
  rosdep pass installs `ros-jazzy-feetech-ros2-driver` from the base image's
  pinned apt snapshot. No Dockerfile edit, no external_dependencies entry.
- xacro args `usb_port` (default `/dev/so101_follower`) and `calibration_file`.
  Servo IDs and per-joint zero offsets live in the calibration YAML instead of
  twelve args, mirroring how `initial_positions.yaml` is already loaded. Baud
  is not an arg: the driver hardwires 1 Mbaud, the SO-101 factory setting.
- `config/udev/99-so101.rules` for stable `/dev/so101_{leader,follower}`.
- `effort` is declared on the mock branch only, and `joint_state_broadcaster`
  no longer asks for it. The driver's `export_state_interfaces()` returns
  position and velocity only, and because that override is non-empty the
  framework does not add the URDF-declared interfaces, so declaring `effort`
  on `real` makes `validate_storage()` reject the component at load with
  "Discrepancy between robot description file (urdf) and actually exported
  HW interfaces" and no controller ever claims an interface. Mock's expansion
  is unchanged.
- `stopped_velocity_tolerance` is 0.0: the driver decodes Present Speed as an
  unsigned word, so a joint moving negative reports ~+50.27 rad/s and the
  goal check would abort on velocity with every position in tolerance. The
  README's "Known gaps in the driver" list carries this and the missing
  effort feedback.

Teleop jog reaches the servos on this branch too: both jog controllers command
`position`, the one command interface the driver exports, so the teleop change
merged in #928 needs nothing further for real hardware.

The Mirror SO101 Follower Objective is the wiggle test on both branches: the
bridge's sine is `wiggle_amplitude_rad` (0.1 rad by default, a ROS parameter)
either side of the pose read once from `/joint_states` when mirroring starts,
clamped to the URDF limits, so it is a joint-by-joint "alive and turning the
right way" check that is safe on the powered follower rather than a sweep
through a fixed pose. The sine subtracts its own phase term so every joint
starts at exactly the sampled pose rather than an amplitude away from it, and
mirroring refuses to start without a complete six-joint `JointState` newer
than `joint_states_timeout_s`.

The bench procedure covers udev install, servo IDs and LeRobot calibration
(including that tick 2048 means the pose held during homing, not URDF zero,
and the per-joint offset correction), power-before-start on `real`, the
first-activation checks, and falling back to mock.

Proven without hardware: the workspace builds with the driver; the mock path
runs unchanged; both branches expand and parse; and the real branch was driven
against a pty-backed STS3215 emulator through load, `validate_storage`,
activation, `/joint_states`, and a successful trajectory goal. Not proven:
anything requiring the physical bus - real servo IDs, calibration offsets and
the leader arm.

Co-Authored-By: Claude Opus 5 <noreply@anthropic.com>

File: src/so101_sim/description/so101.urdf.xacro (robot description, xacro)
@@ -19,4 +19,20 @@
     value="${xacro.load_yaml('$(arg initial_positions_file)')['initial_positions']}"
   />
+  <!--
+    Feetech STS3215 bus, used only when hardware_interface:=real.
+    `usb_port` is the follower bus; keep it a udev symlink rather than a
+    /dev/ttyACM* that renumbers (config/udev/99-so101.rules). The baud rate is
+    not an argument: feetech_ros2_driver hardwires 1 Mbaud, which is the SO-101
+    factory setting.
+  -->
+  <xacro:arg name="usb_port" default="/dev/so101_follower" />
+  <xacro:arg
+    name="calibration_file"
+    default="$(find so101_sim)/config/so101_follower_calibration.yaml"
+  />
+  <xacro:property
+    name="calibration"
+    value="${xacro.load_yaml('$(arg calibration_file)')['joints']}"
+  />
   <!-- The arm is bolted to the bench; `world` is the planning frame. -->
   <link name="world" />
@@ -562,4 +578,13 @@
   <xacro:macro name="so101_joint" params="name lower upper">
     <joint name="${name}">
+      <!--
+        Servo identity and zero, from config/so101_follower_calibration.yaml.
+        The driver reads `id` to address the servo and treats `offset` as the
+        raw tick that means 0 rad. Absent on mock, where they mean nothing.
+      -->
+      <xacro:if value="${'$(arg hardware_interface)' == 'real'}">
+        <param name="id">${calibration[name]['id']}</param>
+        <param name="offset">${calibration[name]['offset']}</param>
+      </xacro:if>
       <command_interface name="position">
         <param name="min">${lower}</param>
@@ -570,5 +595,16 @@
       </state_interface>
       <state_interface name="velocity" />
-      <state_interface name="effort" />
+      <!--
+        Mock only. feetech_ros2_driver overrides export_state_interfaces() and
+        exports position and velocity alone, and ros2_control's
+        validate_storage() rejects a hardware component whose URDF declares a
+        state interface it did not export ("Discrepancy between robot
+        description file (urdf) and actually exported HW interfaces"). An
+        effort declaration on the real branch is therefore fatal at load, not
+        inert; that is also why joint_state_broadcaster does not ask for one.
+      -->
+      <xacro:if value="${'$(arg hardware_interface)' == 'mock'}">
+        <state_interface name="effort" />
+      </xacro:if>
     </joint>
   </xacro:macro>
@@ -582,5 +618,14 @@
     </xacro:if>
     <xacro:if value="${'$(arg hardware_interface)' == 'real'}">
-      <!-- Phase two: a Feetech STS3215 bus hardware interface goes here. -->
+      <hardware>
+        <!--
+          One serial bus, six STS3215 servos daisy-chained, position command
+          and position/velocity feedback. The plugin ships as the Jazzy binary
+          ros-jazzy-feetech-ros2-driver; `feetech_ros2_driver` is an
+          exec_depend so rosdep installs it into the workspace image.
+        -->
+        <plugin>feetech_ros2_driver/FeetechHardwareInterface</plugin>
+        <param name="usb_port">$(arg usb_port)</param>
+      </hardware>
     </xacro:if>
     <!-- Limits are the upstream LeRobot calibration, in radians. -->
