Commit message: refactor(so101): split so101_sim into so101_base_config + mock overlay
Mirrors the workspace's picknik_ur_base_config + mock_sim precedent.
so101_base_config now owns the robot description, all STL assets,
Feetech ros2_control hardware config, SRDF/joint limits/IK/jog,
initial positions, calibration file, udev rule, and the general
Objectives (Move to Waypoint, Close/Open Gripper, Teleoperate); it is
the package a real-arm deployment points MoveIt Pro at, defaulting to
hardware_interface: mock.

so101_sim becomes a thin `based_on_package: so101_base_config` overlay
that only forces hardware_interface: mock and keeps the wiggle-test
bridge (script/so101_arm_bridge.py) and its Mirror SO101 Follower
Objective, per the split this package's own README already called out
under "Later phases". Moves use `git mv` so history follows; xacro
`so101_sim` package references were mechanically renamed to
so101_base_config. Adds test_config_inheritance.py, which fails if the
overlay stops inheriting from the base package.

PR 932 (torque lifecycle) is still open against so101_sim's config.yaml/
xacro/README/package.xml/CMakeLists.txt/test_hardware_plugin.py; this
branch is cut from main before it merges and will need a rebase to
carry its changes into the new layout.

Co-Authored-By: Claude Sonnet 5 <noreply@anthropic.com>

File: src/so101_base_config/description/so101.urdf.xacro (robot description, xacro)
@@ -13,5 +13,5 @@
   <xacro:arg
     name="initial_positions_file"
-    default="$(find so101_sim)/config/initial_positions.yaml"
+    default="$(find so101_base_config)/config/initial_positions.yaml"
   />
   <xacro:property
@@ -29,5 +29,5 @@
   <xacro:arg
     name="calibration_file"
-    default="$(find so101_sim)/config/so101_follower_calibration.yaml"
+    default="$(find so101_base_config)/config/so101_follower_calibration.yaml"
   />
   <xacro:property
@@ -63,12 +63,12 @@
       <origin xyz="0 0 0" rpy="1.5708 0 1.5708"/>
       <geometry>
-        <mesh filename="package://so101_sim/description/assets/arm_base.stl"/>
-      </geometry>
-      <material name="3d_printed"><color rgba="0.05 0.05 0.05 1.0"/></material>
-    </visual>
-    <collision>
-      <origin xyz="0 0 0" rpy="1.5708 0 1.5708"/>
-      <geometry>
-        <mesh filename="package://so101_sim/description/assets/arm_base.stl"/>
+        <mesh filename="package://so101_base_config/description/assets/arm_base.stl"/>
+      </geometry>
+      <material name="3d_printed"><color rgba="0.05 0.05 0.05 1.0"/></material>
+    </visual>
+    <collision>
+      <origin xyz="0 0 0" rpy="1.5708 0 1.5708"/>
+      <geometry>
+        <mesh filename="package://so101_base_config/description/assets/arm_base.stl"/>
       </geometry>
     </collision>
@@ -77,12 +77,12 @@
       <origin xyz="0 0 0" rpy="1.5708 0 1.5708"/>
       <geometry>
-        <mesh filename="package://so101_sim/description/assets/cam_mount_bottom.stl"/>
-      </geometry>
-      <material name="3d_printed"><color rgba="0.05 0.05 0.05 1.0"/></material>
-    </visual>
-    <collision>
-      <origin xyz="0 0 0" rpy="1.5708 0 1.5708"/>
-      <geometry>
-        <mesh filename="package://so101_sim/description/assets/cam_mount_bottom.stl"/>
+        <mesh filename="package://so101_base_config/description/assets/cam_mount_bottom.stl"/>
+      </geometry>
+      <material name="3d_printed"><color rgba="0.05 0.05 0.05 1.0"/></material>
+    </visual>
+    <collision>
+      <origin xyz="0 0 0" rpy="1.5708 0 1.5708"/>
+      <geometry>
+        <mesh filename="package://so101_base_config/description/assets/cam_mount_bottom.stl"/>
       </geometry>
     </collision>
@@ -91,12 +91,12 @@
       <origin xyz="0 0 0" rpy="1.5708 0 1.5708"/>
       <geometry>
-        <mesh filename="package://so101_sim/description/assets/cam_mount_middle.stl"/>
-      </geometry>
-      <material name="3d_printed"><color rgba="0.05 0.05 0.05 1.0"/></material>
-    </visual>
-    <collision>
-      <origin xyz="0 0 0" rpy="1.5708 0 1.5708"/>
-      <geometry>
-        <mesh filename="package://so101_sim/description/assets/cam_mount_middle.stl"/>
+        <mesh filename="package://so101_base_config/description/assets/cam_mount_middle.stl"/>
+      </geometry>
+      <material name="3d_printed"><color rgba="0.05 0.05 0.05 1.0"/></material>
+    </visual>
+    <collision>
+      <origin xyz="0 0 0" rpy="1.5708 0 1.5708"/>
+      <geometry>
+        <mesh filename="package://so101_base_config/description/assets/cam_mount_middle.stl"/>
       </geometry>
     </collision>
@@ -105,12 +105,12 @@
       <origin xyz="0 0 0" rpy="1.5708 0 1.5708"/>
       <geometry>
-        <mesh filename="package://so101_sim/description/assets/cam_mount_top.stl"/>
-      </geometry>
-      <material name="3d_printed"><color rgba="0.05 0.05 0.05 1.0"/></material>
-    </visual>
-    <collision>
-      <origin xyz="0 0 0" rpy="1.5708 0 1.5708"/>
-      <geometry>
-        <mesh filename="package://so101_sim/description/assets/cam_mount_top.stl"/>
+        <mesh filename="package://so101_base_config/description/assets/cam_mount_top.stl"/>
+      </geometry>
+      <material name="3d_printed"><color rgba="0.05 0.05 0.05 1.0"/></material>
+    </visual>
+    <collision>
+      <origin xyz="0 0 0" rpy="1.5708 0 1.5708"/>
+      <geometry>
+        <mesh filename="package://so101_base_config/description/assets/cam_mount_top.stl"/>
       </geometry>
     </collision>
@@ -149,5 +149,5 @@
       <origin xyz="-0.00636471 -9.94414e-05 -0.0024" rpy="1.5708 -1.67685e-15 1.5708"/>
       <geometry>
-        <mesh filename="package://so101_sim/description/assets/base_motor_holder_so101_v1.stl"/>
+        <mesh filename="package://so101_base_config/description/assets/base_motor_holder_so101_v1.stl"/>
       </geometry>
       <material name="3d_printed"><color rgba="0.05 0.05 0.05 1.0"/></material>
@@ -156,5 +156,5 @@
       <origin xyz="-0.00636471 -9.94414e-05 -0.0024" rpy="1.5708 -1.67685e-15 1.5708"/>
       <geometry>
-        <mesh filename="package://so101_sim/description/assets/base_motor_holder_so101_v1.stl"/>
+        <mesh filename="package://so101_base_config/description/assets/base_motor_holder_so101_v1.stl"/>
       </geometry>
     </collision>
@@ -163,5 +163,5 @@
       <origin xyz="-0.00636471 -8.97657e-09 -0.0024" rpy="1.5708 -2.78073e-29 1.5708"/>
       <geometry>
-        <mesh filename="package://so101_sim/description/assets/base_so101_v2.stl"/>
+        <mesh filename="package://so101_base_config/description/assets/base_so101_v2.stl"/>
       </geometry>
       <material name="3d_printed"><color rgba="0.05 0.05 0.05 1.0"/></material>
@@ -170,5 +170,5 @@
       <origin xyz="-0.00636471 -8.97657e-09 -0.0024" rpy="1.5708 -2.78073e-29 1.5708"/>
       <geometry>
-        <mesh filename="package://so101_sim/description/assets/base_so101_v2.stl"/>
+        <mesh filename="package://so101_base_config/description/assets/base_so101_v2.stl"/>
       </geometry>
     </collision>
@@ -177,5 +177,5 @@
       <origin xyz="0.0263353 -8.97657e-09 0.0437" rpy="-8.21148e-16 7.84513e-18 1.249e-15"/>
       <geometry>
-        <mesh filename="package://so101_sim/description/assets/sts3215_03a_v1.stl"/>
+        <mesh filename="package://so101_base_config/description/assets/sts3215_03a_v1.stl"/>
       </geometry>
       <material name="sts3215"><color rgba="0.1 0.1 0.1 1.0"/></material>
@@ -184,5 +184,5 @@
       <origin xyz="0.0263353 -8.97657e-09 0.0437" rpy="-8.21148e-16 7.84513e-18 1.249e-15"/>
       <geometry>
-        <mesh filename="package://so101_sim/description/assets/sts3215_03a_v1.stl"/>
+        <mesh filename="package://so101_base_config/description/assets/sts3215_03a_v1.stl"/>
       </geometry>
     </collision>
@@ -191,5 +191,5 @@
       <origin xyz="-0.0309827 -0.000199441 0.0474" rpy="1.5708 -1.35493e-14 1.5708"/>
       <geometry>
-        <mesh filename="package://so101_sim/description/assets/waveshare_mounting_plate_so101_v2.stl"/>
+        <mesh filename="package://so101_base_config/description/assets/waveshare_mounting_plate_so101_v2.stl"/>
       </geometry>
       <material name="3d_printed"><color rgba="0.05 0.05 0.05 1.0"/></material>
@@ -198,5 +198,5 @@
       <origin xyz="-0.0309827 -0.000199441 0.0474" rpy="1.5708 -1.35493e-14 1.5708"/>
       <geometry>
-        <mesh filename="package://so101_sim/description/assets/waveshare_mounting_plate_so101_v2.stl"/>
+        <mesh filename="package://so101_base_config/description/assets/waveshare_mounting_plate_so101_v2.stl"/>
       </geometry>
     </collision>
@@ -213,5 +213,5 @@
       <origin xyz="-0.0303992 0.000422241 -0.0417" rpy="1.5708 1.5708 0"/>
       <geometry>
-        <mesh filename="package://so101_sim/description/assets/sts3215_03a_v1.stl"/>
+        <mesh filename="package://so101_base_config/description/assets/sts3215_03a_v1.stl"/>
       </geometry>
       <material name="sts3215"><color rgba="0.1 0.1 0.1 1.0"/></material>
@@ -220,5 +220,5 @@
       <origin xyz="-0.0303992 0.000422241 -0.0417" rpy="1.5708 1.5708 0"/>
       <geometry>
-        <mesh filename="package://so101_sim/description/assets/sts3215_03a_v1.stl"/>
+        <mesh filename="package://so101_base_config/description/assets/sts3215_03a_v1.stl"/>
       </geometry>
     </collision>
@@ -227,5 +227,5 @@
       <origin xyz="-0.0675992 -0.000177759 0.0158499" rpy="1.5708 -1.5708 0"/>
       <geometry>
-        <mesh filename="package://so101_sim/description/assets/motor_holder_so101_base_v1.stl"/>
+        <mesh filename="package://so101_base_config/description/assets/motor_holder_so101_base_v1.stl"/>
       </geometry>
       <material name="3d_printed"><color rgba="0.05 0.05 0.05 1.0"/></material>
@@ -234,5 +234,5 @@
       <origin xyz="-0.0675992 -0.000177759 0.0158499" rpy="1.5708 -1.5708 0"/>
       <geometry>
-        <mesh filename="package://so101_sim/description/assets/motor_holder_so101_base_v1.stl"/>
+        <mesh filename="package://so101_base_config/description/assets/motor_holder_so101_base_v1.stl"/>
       </geometry>
     </collision>
@@ -241,5 +241,5 @@
       <origin xyz="0.0122008 2.22413e-05 0.0464" rpy="-1.5708 2.35221e-33 0"/>
       <geometry>
-        <mesh filename="package://so101_sim/description/assets/rotation_pitch_so101_v1.stl"/>
+        <mesh filename="package://so101_base_config/description/assets/rotation_pitch_so101_v1.stl"/>
       </geometry>
       <material name="3d_printed"><color rgba="0.05 0.05 0.05 1.0"/></material>
@@ -248,5 +248,5 @@
       <origin xyz="0.0122008 2.22413e-05 0.0464" rpy="-1.5708 2.35221e-33 0"/>
       <geometry>
-        <mesh filename="package://so101_sim/description/assets/rotation_pitch_so101_v1.stl"/>
+        <mesh filename="package://so101_base_config/description/assets/rotation_pitch_so101_v1.stl"/>
       </geometry>
     </collision>
@@ -263,5 +263,5 @@
       <origin xyz="-0.11257 -0.0155 0.0187" rpy="-3.14159 -5.27356e-16 -1.5708"/>
       <geometry>
-        <mesh filename="package://so101_sim/description/assets/sts3215_03a_v1.stl"/>
+        <mesh filename="package://so101_base_config/description/assets/sts3215_03a_v1.stl"/>
       </geometry>
       <material name="sts3215"><color rgba="0.1 0.1 0.1 1.0"/></material>
@@ -270,5 +270,5 @@
       <origin xyz="-0.11257 -0.0155 0.0187" rpy="-3.14159 -5.27356e-16 -1.5708"/>
       <geometry>
-        <mesh filename="package://so101_sim/description/assets/sts3215_03a_v1.stl"/>
+        <mesh filename="package://so101_base_config/description/assets/sts3215_03a_v1.stl"/>
       </geometry>
     </collision>
@@ -277,5 +277,5 @@
       <origin xyz="-0.065085 0.012 0.0182" rpy="3.14159 -0 -1.30911e-30"/>
       <geometry>
-        <mesh filename="package://so101_sim/description/assets/upper_arm_so101_v1.stl"/>
+        <mesh filename="package://so101_base_config/description/assets/upper_arm_so101_v1.stl"/>
       </geometry>
       <material name="3d_printed"><color rgba="0.05 0.05 0.05 1.0"/></material>
@@ -284,5 +284,5 @@
       <origin xyz="-0.065085 0.012 0.0182" rpy="3.14159 -0 -1.30911e-30"/>
       <geometry>
-        <mesh filename="package://so101_sim/description/assets/upper_arm_so101_v1.stl"/>
+        <mesh filename="package://so101_base_config/description/assets/upper_arm_so101_v1.stl"/>
       </geometry>
     </collision>
@@ -299,5 +299,5 @@
       <origin xyz="-0.0648499 -0.032 0.0182" rpy="3.14159 -0 6.67202e-31"/>
       <geometry>
-        <mesh filename="package://so101_sim/description/assets/under_arm_so101_v1.stl"/>
+        <mesh filename="package://so101_base_config/description/assets/under_arm_so101_v1.stl"/>
       </geometry>
       <material name="3d_printed"><color rgba="0.05 0.05 0.05 1.0"/></material>
@@ -306,5 +306,5 @@
       <origin xyz="-0.0648499 -0.032 0.0182" rpy="3.14159 -0 6.67202e-31"/>
       <geometry>
-        <mesh filename="package://so101_sim/description/assets/under_arm_so101_v1.stl"/>
+        <mesh filename="package://so101_base_config/description/assets/under_arm_so101_v1.stl"/>
       </geometry>
     </collision>
@@ -313,5 +313,5 @@
       <origin xyz="-0.0648499 -0.032 0.018" rpy="-3.14159 -2.55351e-15 -1.83387e-30"/>
       <geometry>
-        <mesh filename="package://so101_sim/description/assets/motor_holder_so101_wrist_v1.stl"/>
+        <mesh filename="package://so101_base_config/description/assets/motor_holder_so101_wrist_v1.stl"/>
       </geometry>
       <material name="3d_printed"><color rgba="0.05 0.05 0.05 1.0"/></material>
@@ -320,5 +320,5 @@
       <origin xyz="-0.0648499 -0.032 0.018" rpy="-3.14159 -2.55351e-15 -1.83387e-30"/>
       <geometry>
-        <mesh filename="package://so101_sim/description/assets/motor_holder_so101_wrist_v1.stl"/>
+        <mesh filename="package://so101_base_config/description/assets/motor_holder_so101_wrist_v1.stl"/>
       </geometry>
     </collision>
@@ -327,5 +327,5 @@
       <origin xyz="-0.1224 0.0052 0.0187" rpy="-3.14159 -7.88861e-31 -3.14159"/>
       <geometry>
-        <mesh filename="package://so101_sim/description/assets/sts3215_03a_v1.stl"/>
+        <mesh filename="package://so101_base_config/description/assets/sts3215_03a_v1.stl"/>
       </geometry>
       <material name="sts3215"><color rgba="0.1 0.1 0.1 1.0"/></material>
@@ -334,5 +334,5 @@
       <origin xyz="-0.1224 0.0052 0.0187" rpy="-3.14159 -7.88861e-31 -3.14159"/>
       <geometry>
-        <mesh filename="package://so101_sim/description/assets/sts3215_03a_v1.stl"/>
+        <mesh filename="package://so101_base_config/description/assets/sts3215_03a_v1.stl"/>
       </geometry>
     </collision>
@@ -349,5 +349,5 @@
       <origin xyz="8.32667e-17 -0.0424 0.0306" rpy="1.5708 1.5708 0"/>
       <geometry>
-        <mesh filename="package://so101_sim/description/assets/sts3215_03a_no_horn_v1.stl"/>
+        <mesh filename="package://so101_base_config/description/assets/sts3215_03a_no_horn_v1.stl"/>
       </geometry>
       <material name="sts3215"><color rgba="0.1 0.1 0.1 1.0"/></material>
@@ -356,5 +356,5 @@
       <origin xyz="8.32667e-17 -0.0424 0.0306" rpy="1.5708 1.5708 0"/>
       <geometry>
-        <mesh filename="package://so101_sim/description/assets/sts3215_03a_no_horn_v1.stl"/>
+        <mesh filename="package://so101_base_config/description/assets/sts3215_03a_no_horn_v1.stl"/>
       </geometry>
     </collision>
@@ -363,5 +363,5 @@
       <origin xyz="0 -0.028 0.0181" rpy="-1.5708 -1.5708 0"/>
       <geometry>
-        <mesh filename="package://so101_sim/description/assets/wrist_roll_pitch_so101_v2.stl"/>
+        <mesh filename="package://so101_base_config/description/assets/wrist_roll_pitch_so101_v2.stl"/>
       </geometry>
       <material name="3d_printed"><color rgba="0.05 0.05 0.05 1.0"/></material>
@@ -370,5 +370,5 @@
       <origin xyz="0 -0.028 0.0181" rpy="-1.5708 -1.5708 0"/>
       <geometry>
-        <mesh filename="package://so101_sim/description/assets/wrist_roll_pitch_so101_v2.stl"/>
+        <mesh filename="package://so101_base_config/description/assets/wrist_roll_pitch_so101_v2.stl"/>
       </geometry>
     </collision>
@@ -385,5 +385,5 @@
       <origin xyz="0.0077 0.0001 -0.0234" rpy="-1.5708 -5.19179e-17 -1.66533e-16"/>
       <geometry>
-        <mesh filename="package://so101_sim/description/assets/sts3215_03a_v1.stl"/>
+        <mesh filename="package://so101_base_config/description/assets/sts3215_03a_v1.stl"/>
       </geometry>
       <material name="sts3215"><color rgba="0.1 0.1 0.1 1.0"/></material>
@@ -392,5 +392,5 @@
       <origin xyz="0.0077 0.0001 -0.0234" rpy="-1.5708 -5.19179e-17 -1.66533e-16"/>
       <geometry>
-        <mesh filename="package://so101_sim/description/assets/sts3215_03a_v1.stl"/>
+        <mesh filename="package://so101_base_config/description/assets/sts3215_03a_v1.stl"/>
       </geometry>
     </collision>
@@ -402,5 +402,5 @@
       <origin xyz="8.32667e-17 -0.000218214 0.000949706" rpy="-3.14159 -5.55112e-17 0"/>
       <geometry>
-        <mesh filename="package://so101_sim/description/assets/soft_fin_fixed_jaw.stl"/>
+        <mesh filename="package://so101_base_config/description/assets/soft_fin_fixed_jaw.stl"/>
       </geometry>
       <material name="3d_printed"><color rgba="0.05 0.05 0.05 1.0"/></material>
@@ -409,5 +409,5 @@
       <origin xyz="8.32667e-17 -0.000218214 0.000949706" rpy="-3.14159 -5.55112e-17 0"/>
       <geometry>
-        <mesh filename="package://so101_sim/description/assets/soft_fin_fixed_jaw_collision.stl"/>
+        <mesh filename="package://so101_base_config/description/assets/soft_fin_fixed_jaw_collision.stl"/>
       </geometry>
     </collision>
@@ -418,5 +418,5 @@
       <origin xyz="-0.02275 0.000781901 -0.0425503" rpy="2.66224e-06 -0.0806329 -2.14431e-07"/>
       <geometry>
-        <mesh filename="package://so101_sim/description/assets/soft_fin_finger.stl"/>
+        <mesh filename="package://so101_base_config/description/assets/soft_fin_finger.stl"/>
       </geometry>
       <material name="tpu_fin"><color rgba="0.12 0.12 0.13 1.0"/></material>
@@ -425,5 +425,5 @@
       <origin xyz="-0.02275 0.000781901 -0.0425503" rpy="2.66224e-06 -0.0806329 -2.14431e-07"/>
       <geometry>
-        <mesh filename="package://so101_sim/description/assets/soft_fin_finger.stl"/>
+        <mesh filename="package://so101_base_config/description/assets/soft_fin_finger.stl"/>
       </geometry>
     </collision>
@@ -440,5 +440,5 @@
       <origin xyz="8.32667e-17 -0.000218214 0.000949706" rpy="-3.14159 -5.55112e-17 0"/>
       <geometry>
-        <mesh filename="package://so101_sim/description/assets/camera_wrist_mount.stl"/>
+        <mesh filename="package://so101_base_config/description/assets/camera_wrist_mount.stl"/>
       </geometry>
       <material name="3d_printed"><color rgba="0.05 0.05 0.05 1.0"/></material>
@@ -447,5 +447,5 @@
       <origin xyz="8.32667e-17 -0.000218214 0.000949706" rpy="-3.14159 -5.55112e-17 0"/>
       <geometry>
-        <mesh filename="package://so101_sim/description/assets/camera_wrist_mount.stl"/>
+        <mesh filename="package://so101_base_config/description/assets/camera_wrist_mount.stl"/>
       </geometry>
     </collision>
@@ -502,5 +502,5 @@
       <origin xyz="-5.55112e-17 -5.55112e-17 0.0189" rpy="9.53145e-17 6.93889e-18 1.24077e-24"/>
       <geometry>
-        <mesh filename="package://so101_sim/description/assets/soft_fin_moving_jaw.stl"/>
+        <mesh filename="package://so101_base_config/description/assets/soft_fin_moving_jaw.stl"/>
       </geometry>
       <material name="3d_printed"><color rgba="0.05 0.05 0.05 1.0"/></material>
@@ -509,5 +509,5 @@
       <origin xyz="-5.55112e-17 -5.55112e-17 0.0189" rpy="9.53145e-17 6.93889e-18 1.24077e-24"/>
       <geometry>
-        <mesh filename="package://so101_sim/description/assets/soft_fin_moving_jaw_collision.stl"/>
+        <mesh filename="package://so101_base_config/description/assets/soft_fin_moving_jaw_collision.stl"/>
       </geometry>
     </collision>
@@ -516,5 +516,5 @@
       <origin xyz="-0.00115 -0.0222 0.0181" rpy="1.5708 -1.07812e-17 3.10121"/>
       <geometry>
-        <mesh filename="package://so101_sim/description/assets/soft_fin_finger.stl"/>
+        <mesh filename="package://so101_base_config/description/assets/soft_fin_finger.stl"/>
       </geometry>
       <material name="tpu_fin"><color rgba="0.12 0.12 0.13 1.0"/></material>
@@ -523,5 +523,5 @@
       <origin xyz="-0.00115 -0.0222 0.0181" rpy="1.5708 -1.07812e-17 3.10121"/>
       <geometry>
-        <mesh filename="package://so101_sim/description/assets/soft_fin_finger.stl"/>
+        <mesh filename="package://so101_base_config/description/assets/soft_fin_finger.stl"/>
       </geometry>
     </collision>
