Commit message: style(so101): change 3D-printed parts from near-black to off-white
Co-Authored-By: Claude Fable 5.1 <noreply@anthropic.com>

File: src/so101_base_config/description/so101.urdf.xacro (robot description, xacro)
@@ -44,5 +44,5 @@
   <!-- Materials -->
   <material name="3d_printed">
-    <color rgba="0.05 0.05 0.05 1.0"/>
+    <color rgba="0.88 0.87 0.83 1.0"/>
   </material>
   <material name="sts3215">
@@ -65,5 +65,5 @@
         <mesh filename="package://so101_base_config/description/assets/arm_base.stl"/>
       </geometry>
-      <material name="3d_printed"><color rgba="0.05 0.05 0.05 1.0"/></material>
+      <material name="3d_printed"><color rgba="0.88 0.87 0.83 1.0"/></material>
     </visual>
     <collision>
@@ -79,5 +79,5 @@
         <mesh filename="package://so101_base_config/description/assets/cam_mount_bottom.stl"/>
       </geometry>
-      <material name="3d_printed"><color rgba="0.05 0.05 0.05 1.0"/></material>
+      <material name="3d_printed"><color rgba="0.88 0.87 0.83 1.0"/></material>
     </visual>
     <collision>
@@ -93,5 +93,5 @@
         <mesh filename="package://so101_base_config/description/assets/cam_mount_middle.stl"/>
       </geometry>
-      <material name="3d_printed"><color rgba="0.05 0.05 0.05 1.0"/></material>
+      <material name="3d_printed"><color rgba="0.88 0.87 0.83 1.0"/></material>
     </visual>
     <collision>
@@ -107,5 +107,5 @@
         <mesh filename="package://so101_base_config/description/assets/cam_mount_top.stl"/>
       </geometry>
-      <material name="3d_printed"><color rgba="0.05 0.05 0.05 1.0"/></material>
+      <material name="3d_printed"><color rgba="0.88 0.87 0.83 1.0"/></material>
     </visual>
     <collision>
@@ -151,5 +151,5 @@
         <mesh filename="package://so101_base_config/description/assets/base_motor_holder_so101_v1.stl"/>
       </geometry>
-      <material name="3d_printed"><color rgba="0.05 0.05 0.05 1.0"/></material>
+      <material name="3d_printed"><color rgba="0.88 0.87 0.83 1.0"/></material>
     </visual>
     <collision>
@@ -165,5 +165,5 @@
         <mesh filename="package://so101_base_config/description/assets/base_so101_v2.stl"/>
       </geometry>
-      <material name="3d_printed"><color rgba="0.05 0.05 0.05 1.0"/></material>
+      <material name="3d_printed"><color rgba="0.88 0.87 0.83 1.0"/></material>
     </visual>
     <collision>
@@ -193,5 +193,5 @@
         <mesh filename="package://so101_base_config/description/assets/waveshare_mounting_plate_so101_v2.stl"/>
       </geometry>
-      <material name="3d_printed"><color rgba="0.05 0.05 0.05 1.0"/></material>
+      <material name="3d_printed"><color rgba="0.88 0.87 0.83 1.0"/></material>
     </visual>
     <collision>
@@ -229,5 +229,5 @@
         <mesh filename="package://so101_base_config/description/assets/motor_holder_so101_base_v1.stl"/>
       </geometry>
-      <material name="3d_printed"><color rgba="0.05 0.05 0.05 1.0"/></material>
+      <material name="3d_printed"><color rgba="0.88 0.87 0.83 1.0"/></material>
     </visual>
     <collision>
@@ -243,5 +243,5 @@
         <mesh filename="package://so101_base_config/description/assets/rotation_pitch_so101_v1.stl"/>
       </geometry>
-      <material name="3d_printed"><color rgba="0.05 0.05 0.05 1.0"/></material>
+      <material name="3d_printed"><color rgba="0.88 0.87 0.83 1.0"/></material>
     </visual>
     <collision>
@@ -279,5 +279,5 @@
         <mesh filename="package://so101_base_config/description/assets/upper_arm_so101_v1.stl"/>
       </geometry>
-      <material name="3d_printed"><color rgba="0.05 0.05 0.05 1.0"/></material>
+      <material name="3d_printed"><color rgba="0.88 0.87 0.83 1.0"/></material>
     </visual>
     <collision>
@@ -301,5 +301,5 @@
         <mesh filename="package://so101_base_config/description/assets/under_arm_so101_v1.stl"/>
       </geometry>
-      <material name="3d_printed"><color rgba="0.05 0.05 0.05 1.0"/></material>
+      <material name="3d_printed"><color rgba="0.88 0.87 0.83 1.0"/></material>
     </visual>
     <collision>
@@ -315,5 +315,5 @@
         <mesh filename="package://so101_base_config/description/assets/motor_holder_so101_wrist_v1.stl"/>
       </geometry>
-      <material name="3d_printed"><color rgba="0.05 0.05 0.05 1.0"/></material>
+      <material name="3d_printed"><color rgba="0.88 0.87 0.83 1.0"/></material>
     </visual>
     <collision>
@@ -365,5 +365,5 @@
         <mesh filename="package://so101_base_config/description/assets/wrist_roll_pitch_so101_v2.stl"/>
       </geometry>
-      <material name="3d_printed"><color rgba="0.05 0.05 0.05 1.0"/></material>
+      <material name="3d_printed"><color rgba="0.88 0.87 0.83 1.0"/></material>
     </visual>
     <collision>
@@ -404,5 +404,5 @@
         <mesh filename="package://so101_base_config/description/assets/soft_fin_fixed_jaw.stl"/>
       </geometry>
-      <material name="3d_printed"><color rgba="0.05 0.05 0.05 1.0"/></material>
+      <material name="3d_printed"><color rgba="0.88 0.87 0.83 1.0"/></material>
     </visual>
     <collision>
@@ -442,5 +442,5 @@
         <mesh filename="package://so101_base_config/description/assets/camera_wrist_mount.stl"/>
       </geometry>
-      <material name="3d_printed"><color rgba="0.05 0.05 0.05 1.0"/></material>
+      <material name="3d_printed"><color rgba="0.88 0.87 0.83 1.0"/></material>
     </visual>
     <collision>
@@ -504,5 +504,5 @@
         <mesh filename="package://so101_base_config/description/assets/soft_fin_moving_jaw.stl"/>
       </geometry>
-      <material name="3d_printed"><color rgba="0.05 0.05 0.05 1.0"/></material>
+      <material name="3d_printed"><color rgba="0.88 0.87 0.83 1.0"/></material>
     </visual>
     <collision>
