Commit message: market_sim: let the base travel the whole store
The planar base joints were limited to the parent sim's 10 m room, so the
base stopped at x = -10 m on its way to aisle A1. A new base_travel_limit
argument in the vendored mobile_fr3_duo_mock URDF (default unchanged) sets the
MoveIt limit, and market_sim's robot model copy widens the MuJoCo range to
match; a test keeps the two equal.

File: src/external_dependencies/moveit_pro_franka_ws/src/mobile_fr3_duo_mock/description/mobile_fr3_duo.urdf.xacro (robot description, xacro)
@@ -11,4 +11,6 @@
   <xacro:arg name="ground_truth_odom_frame" default="mj_world"/>
   <xacro:arg name="base_link_name" default="base_link"/>
+  <!-- Modified by PickNik Inc.: base travel from odom along x and y, in metres; a larger site widens it. -->
+  <xacro:arg name="base_travel_limit" default="10.0"/>
   <xacro:include filename="$(find franka_description)/robots/mobile_fr3_duo_v0_2/mobile_fr3_duo_v0_2.xacro"/>
   <!-- Frames: world -> map (fixed) -> odom -> planar joints -> base_link. The URDF starts at odom. -->
@@ -21,5 +23,5 @@
     <child link="virtual_x"/>
     <axis xyz="1 0 0"/>
-    <limit lower="-10.0" upper="10.0" effort="1000.0" velocity="0.35"/>
+    <limit lower="${-$(arg base_travel_limit)}" upper="$(arg base_travel_limit)" effort="1000.0" velocity="0.35"/>
   </joint>
   <joint name="planar_y" type="prismatic">
@@ -27,5 +29,5 @@
     <child link="virtual_y"/>
     <axis xyz="0 1 0"/>
-    <limit lower="-10.0" upper="10.0" effort="1000.0" velocity="0.35"/>
+    <limit lower="${-$(arg base_travel_limit)}" upper="$(arg base_travel_limit)" effort="1000.0" velocity="0.35"/>
   </joint>
   <joint name="planar_theta" type="continuous">
