Commit message: feat(franka_description): vendor 2.9.0; move kitchen_sim and dual_arm_sim to its macros
franka_description 2.9.0 drops the joint-limit, kinematics, inertial and
ros2_control arguments of franka_robot and moves the FR3 Duo mount to
accessories/fr3_duo_mount_v0_3. The vendored copy keeps only the FR3, FR3
v2, TMR v0.2 base and FR3 Duo spine, head and mount files this workspace
uses, plus the hand SRDF that the FR3, FR3 v2 and FR3 Duo SRDF macros
include. UPSTREAM.yaml notes that the mobile Duo URDF's default arms name
the pruned fr3v2_1; configs here pass fr3v2. dual_arm_sim's MuJoCo arm
mounts take the rotation the new mount gives.

File: src/dual_arm_sim/description/franka.urdf.xacro (robot description, xacro)
@@ -4,27 +4,22 @@
   <xacro:arg name="ee_id" default="franka_hand" />
   <xacro:arg name="rpy_ee" default="0 0 -0.785" />
-  <!-- Load Franka Duo Mount -->
-  <xacro:include filename="$(find franka_description)/robots/fr3_duo/fr3_duo_mount/fr3_duo_mount.xacro"/>
-  <xacro:property name="mount_kinematics" value="${xacro.load_yaml('$(find franka_description)/robots/fr3_duo/fr3_duo_mount/kinematics.yaml')}" />
+  <!-- Load Franka Duo Mount (franka_description 2.9.0 accessory) -->
+  <xacro:include filename="$(find franka_description)/accessories/fr3_duo_mount_v0_3/fr3_duo_mount.xacro"/>
   <!-- Load Franka robot -->
   <xacro:include filename="$(find franka_description)/robots/common/franka_robot.xacro"/>
   <link name="world" />
-  <xacro:mount name="fr3_duo"
-               parent="world"
-               inertials="${xacro.load_yaml('$(find franka_description)/robots/fr3_duo/fr3_duo_mount/inertials.yaml')}">
-    <origin xyz="0.0 0.0 0.305115" rpy="0 0 0" />
-  </xacro:mount>
+  <!-- The mount macro attaches with an identity joint, so the pedestal height goes on this link. -->
+  <link name="mount_base" />
+  <joint name="mount_base_joint" type="fixed">
+     <parent link="world"/>
+     <child link="mount_base"/>
+     <origin xyz="0.0 0.0 0.305115" rpy="0 0 0" />
+  </joint>
+  <xacro:mount name="fr3_duo" parent="mount_base" left_prefix="left" right_prefix="right" />
   <joint name="right_mount_joint" type="fixed">
-     <parent link="mount_link"/>
+     <parent link="fr3_duo_mount_right"/>
      <child link = "right_mount"/>
-     <origin xyz="${mount_kinematics['right']['kinematic']['x']} ${mount_kinematics['right']['kinematic']['y']} ${mount_kinematics['right']['kinematic']['z']}"
-             rpy="${mount_kinematics['right']['kinematic']['roll']} ${mount_kinematics['right']['kinematic']['pitch']} ${mount_kinematics['right']['kinematic']['yaw']}"/>
   </joint>
   <xacro:franka_robot robot_type="fr3"
-                      joint_limits="${xacro.load_yaml('$(find franka_description)/robots/fr3/joint_limits.yaml')}"
-                      inertials="${xacro.load_yaml('$(find franka_description)/robots/fr3/inertials.yaml')}"
-                      kinematics="${xacro.load_yaml('$(find franka_description)/robots/fr3/kinematics.yaml')}"
-                      dynamics="${xacro.load_yaml('$(find franka_description)/robots/fr3/dynamics.yaml')}"
-                      gazebo="false"
                       hand="true"
                       tcp_xyz="0 0 0.1034"
@@ -32,9 +27,4 @@
                       rpy_ee="$(arg rpy_ee)"
                       with_sc="false"
-                      ros2_control="false"
-                      robot_ip=""
-                      use_fake_hardware="false"
-                      fake_sensor_commands="false"
-                      gazebo_effort="false"
                       no_prefix="false"
                       arm_prefix="right_"
@@ -49,15 +39,8 @@
   </joint>
   <joint name="left_mount_joint" type="fixed">
-     <parent link="mount_link"/>
+     <parent link="fr3_duo_mount_left"/>
      <child link = "left_mount"/>
-     <origin xyz="${mount_kinematics['left']['kinematic']['x']} ${mount_kinematics['left']['kinematic']['y']} ${mount_kinematics['left']['kinematic']['z']}"
-             rpy="${mount_kinematics['left']['kinematic']['roll']} ${mount_kinematics['left']['kinematic']['pitch']} ${mount_kinematics['left']['kinematic']['yaw']}"/>
   </joint>
   <xacro:franka_robot robot_type="fr3"
-                      joint_limits="${xacro.load_yaml('$(find franka_description)/robots/fr3/joint_limits.yaml')}"
-                      inertials="${xacro.load_yaml('$(find franka_description)/robots/fr3/inertials.yaml')}"
-                      kinematics="${xacro.load_yaml('$(find franka_description)/robots/fr3/kinematics.yaml')}"
-                      dynamics="${xacro.load_yaml('$(find franka_description)/robots/fr3/dynamics.yaml')}"
-                      gazebo="false"
                       hand="true"
                       tcp_xyz="0 0 0.1034"
@@ -65,9 +48,4 @@
                       rpy_ee="$(arg rpy_ee)"
                       with_sc="false"
-                      ros2_control="false"
-                      robot_ip=""
-                      use_fake_hardware="false"
-                      fake_sensor_commands="false"
-                      gazebo_effort="false"
                       no_prefix="false"
                       arm_prefix="left_"

File: src/kitchen_sim/description/franka.urdf.xacro (robot description, xacro)
@@ -6,10 +6,6 @@
   <!-- Load Franka robot -->
   <xacro:include filename="$(find franka_description)/robots/common/franka_robot.xacro"/>
+  <!-- franka_description 2.9.0 loads the FR3 limits, inertials, kinematics and dynamics itself. -->
   <xacro:franka_robot robot_type="fr3"
-                      joint_limits="${xacro.load_yaml('$(find franka_description)/robots/fr3/joint_limits.yaml')}"
-                      inertials="${xacro.load_yaml('$(find franka_description)/robots/fr3/inertials.yaml')}"
-                      kinematics="${xacro.load_yaml('$(find franka_description)/robots/fr3/kinematics.yaml')}"
-                      dynamics="${xacro.load_yaml('$(find franka_description)/robots/fr3/dynamics.yaml')}"
-                      gazebo="false"
                       hand="true"
                       tcp_xyz="0 0 0.1034"
@@ -17,9 +13,4 @@
                       rpy_ee="$(arg rpy_ee)"
                       with_sc="false"
-                      ros2_control="false"
-                      robot_ip=""
-                      use_fake_hardware="false"
-                      fake_sensor_commands="false"
-                      gazebo_effort="false"
                       no_prefix="false"
                       arm_prefix=""
