Commit message: feat: add PBR materials and the camera renderer switch to every MuJoCo sim config
Co-Authored-By: Claude Opus 5.5 <noreply@anthropic.com>

File: src/moveit_pro_kinova_configs/space_satellite_sim/description/space_satellite_sim.xacro (robot description, xacro)
@@ -1,12 +1,15 @@
 <?xml version="1.0"?>
 <robot name="gen3" xmlns:xacro="http://ros.org/wiki/xacro">
+  <!-- Which renderer produces the cameras' color topics: opengl (the default), nyx, or both, as documented in lab_sim's picknik_ur.xacro; both is for side-by-side comparison only, since nothing then publishes <camera>/color. runtime.launch.xml reads the same variable to start one Nyx node per camera. An empty value means opengl; an unrecognized one fails the description rather than leaving the config with no camera. -->
+  <xacro:arg
+    name="camera_renderer"
+    default="$(optenv MOVEIT_PRO_CAMERA_RENDERER opengl)"
+  />
+  <xacro:if value="${'$(arg camera_renderer)' not in ('', 'opengl', 'nyx', 'both')}">${xacro.fatal("MOVEIT_PRO_CAMERA_RENDERER is '$(arg camera_renderer)' for the robot description; set it to opengl, nyx or both, or leave it unset for opengl.")}</xacro:if>
   <!-- Arguments for Kinova -->
-  <xacro:arg name="arm" default="gen3" />
-  <xacro:arg name="dof" default="7" />
   <xacro:arg name="mujoco_keyframe" default="default" />
   <xacro:arg name="mujoco_model" default="description/mujoco/scene.xml" />
   <xacro:arg name="mujoco_viewer" default="false" />
   <!-- Import macros for main hardware components -->
-  <xacro:include filename="$(find kortex_description)/arms/$(arg arm)/$(arg dof)dof/urdf/$(arg arm)_macro.xacro" />
   <xacro:include filename="$(find picknik_accessories)/descriptions/sensors/realsense_d415.urdf.xacro"/>
   <!-- Import service platform macro -->
@@ -541,5 +544,5 @@
     <parent link="world" />
     <child link="servicer_camera_mount_link" />
-    <origin xyz=" 0.585021 0.966828 -0.0111449" rpy="0.00122423 0.00171265 -0.426171" />
+    <origin xyz="0.765189 0.582408 -0.0111449" rpy="0.00122423 0.00171265 -0.426171" />
   </joint>
   <xacro:realsense_d415 parent="servicer_camera_mount_link" name="servicer_camera">
@@ -551,5 +554,6 @@
     <parent link="world" />
     <child link="scene_camera_mount_link" />
-    <origin xyz="-0.3 0.3 1.0" rpy="0 0.5236 0" />
+    <!-- Puts scene_camera_color_optical_frame on the MJCF's scene_camera_optical_frame site. -->
+    <origin xyz="5.57611 5.50201 4.36204" rpy="0 0.523593 -2.44346" />
   </joint>
   <xacro:realsense_d415 parent="scene_camera_mount_link" name="scene_camera">
@@ -670,4 +674,35 @@
       <param name="tf_publish_rate">60</param>
     </hardware>
+    <!-- nyx: the Nyx nodes publish each camera's color and camera_info, so MuJoCo publishes only depth and points. -->
+    <xacro:if
+      value="${ dict(opengl=False, nyx=True, both=False)['$(arg camera_renderer)' or 'opengl'] }"
+    >
+      <sensor name="scene_camera">
+        <param name="color_enabled">false</param>
+      </sensor>
+      <sensor name="servicer_camera">
+        <param name="color_enabled">false</param>
+      </sensor>
+      <sensor name="wrist_camera">
+        <param name="color_enabled">false</param>
+      </sensor>
+    </xacro:if>
+    <!-- both: each renderer's color image goes under its own prefix, so no consumer reads one renderer while expecting the other. Depth and points stay unprefixed. -->
+    <xacro:if
+      value="${ dict(opengl=False, nyx=False, both=True)['$(arg camera_renderer)' or 'opengl'] }"
+    >
+      <sensor name="scene_camera">
+        <param name="rgb_topic">scene_camera/opengl/color</param>
+        <param name="camera_info_topic">scene_camera/opengl/camera_info</param>
+      </sensor>
+      <sensor name="servicer_camera">
+        <param name="rgb_topic">servicer_camera/opengl/color</param>
+        <param name="camera_info_topic">servicer_camera/opengl/camera_info</param>
+      </sensor>
+      <sensor name="wrist_camera">
+        <param name="rgb_topic">wrist_camera/opengl/color</param>
+        <param name="camera_info_topic">wrist_camera/opengl/camera_info</param>
+      </sensor>
+    </xacro:if>
   </ros2_control>
 </robot>

File: src/rebot_bench_sim/description/rebot_bench_sim.urdf.xacro (robot description, xacro)
@@ -10,4 +10,19 @@
   <xacro:arg name="mujoco_keyframe" default="default" />
   <xacro:arg name="mujoco_viewer" default="false" />
+  <!-- Which renderer produces the cameras' color topics: opengl (the default), nyx, or both, as documented in lab_sim's picknik_ur.xacro; both is for side-by-side comparison only, since nothing then publishes the real color topics. runtime.launch.xml reads the same variable to start one Nyx node per camera, remapped onto the real cameras' topics. An empty value means opengl; an unrecognized one fails the description rather than leaving the config with no camera. -->
+  <xacro:arg
+    name="camera_renderer"
+    default="$(optenv MOVEIT_PRO_CAMERA_RENDERER opengl)"
+  />
+  <xacro:if value="${'$(arg camera_renderer)' not in ('', 'opengl', 'nyx', 'both')}">${xacro.fatal("MOVEIT_PRO_CAMERA_RENDERER is '$(arg camera_renderer)' for the robot description; set it to opengl, nyx or both, or leave it unset for opengl.")}</xacro:if>
+  <xacro:property name="camera_renderer" value="${'$(arg camera_renderer)' or 'opengl'}" />
+  <xacro:property
+    name="mujoco_color_on_real_topic"
+    value="${ dict(opengl=True, nyx=False, both=False)[camera_renderer] }"
+  />
+  <xacro:property
+    name="mujoco_color_under_opengl"
+    value="${ dict(opengl=False, nyx=False, both=True)[camera_renderer] }"
+  />
   <xacro:property name="layout" value="${xacro.load_yaml('$(arg layout)')}" />
   <!-- An xacro:arg keeps its first declaration, so these defaults win over
@@ -40,12 +55,32 @@
          "_optical_frame", so the cameras are named after the real frames. -->
     <sensor name="d435_color">
-      <param name="rgb_topic">/wrist_mounted_camera/color/image_raw</param>
-      <param name="camera_info_topic">/wrist_mounted_camera/color/camera_info</param>
+      <xacro:if value="${mujoco_color_on_real_topic}">
+        <param name="rgb_topic">/wrist_mounted_camera/color/image_raw</param>
+        <param name="camera_info_topic">/wrist_mounted_camera/color/camera_info</param>
+      </xacro:if>
+      <xacro:if value="${mujoco_color_under_opengl}">
+        <param name="rgb_topic">/wrist_mounted_camera/opengl/color/image_raw</param>
+        <param name="camera_info_topic">/wrist_mounted_camera/opengl/color/camera_info</param>
+      </xacro:if>
+      <!-- nyx: the Nyx node publishes color and camera_info on the real topics instead. -->
+      <xacro:unless value="${mujoco_color_on_real_topic or mujoco_color_under_opengl}">
+        <param name="color_enabled">false</param>
+      </xacro:unless>
       <param name="depth_topic">/wrist_mounted_camera/depth/image_rect_raw</param>
       <param name="points_topic">/wrist_mounted_camera/depth/color/points</param>
     </sensor>
     <sensor name="scene_camera_color">
-      <param name="rgb_topic">/scene_camera/color/image_raw</param>
-      <param name="camera_info_topic">/scene_camera/color/camera_info</param>
+      <xacro:if value="${mujoco_color_on_real_topic}">
+        <param name="rgb_topic">/scene_camera/color/image_raw</param>
+        <param name="camera_info_topic">/scene_camera/color/camera_info</param>
+      </xacro:if>
+      <xacro:if value="${mujoco_color_under_opengl}">
+        <param name="rgb_topic">/scene_camera/opengl/color/image_raw</param>
+        <param name="camera_info_topic">/scene_camera/opengl/color/camera_info</param>
+      </xacro:if>
+      <!-- nyx: the Nyx node publishes color and camera_info on the real topics instead. -->
+      <xacro:unless value="${mujoco_color_on_real_topic or mujoco_color_under_opengl}">
+        <param name="color_enabled">false</param>
+      </xacro:unless>
       <param name="depth_topic">/scene_camera/depth/image_rect_raw</param>
       <param name="points_topic">/scene_camera/depth/color/points</param>

File: src/vla_sim/description/picknik_kinova_gen3.xacro (robot description, xacro)
@@ -1,4 +1,10 @@
 <?xml version="1.0"?>
 <robot name="gen3" xmlns:xacro="http://ros.org/wiki/xacro">
+  <!-- Which renderer produces the cameras' color topics: opengl (the default), nyx, or both, as documented in lab_sim's picknik_ur.xacro; both is for side-by-side comparison only, since nothing then publishes <camera>/color. runtime.launch.xml reads the same variable to start one Nyx node per camera. An empty value means opengl; an unrecognized one fails the description rather than leaving the config with no camera. -->
+  <xacro:arg
+    name="camera_renderer"
+    default="$(optenv MOVEIT_PRO_CAMERA_RENDERER opengl)"
+  />
+  <xacro:if value="${'$(arg camera_renderer)' not in ('', 'opengl', 'nyx', 'both')}">${xacro.fatal("MOVEIT_PRO_CAMERA_RENDERER is '$(arg camera_renderer)' for the robot description; set it to opengl, nyx or both, or leave it unset for opengl.")}</xacro:if>
     <xacro:arg name="mujoco_model" default="description/mujoco/cube_stack_scene.xml" />
     <xacro:arg name="mujoco_viewer" default="false" />
@@ -668,4 +674,35 @@
         <param name="mujoco_viewer">$(arg mujoco_viewer)</param>
       </hardware>
+      <!-- nyx: the Nyx nodes publish each camera's color and camera_info, so MuJoCo publishes only depth and points. -->
+      <xacro:if
+        value="${ dict(opengl=False, nyx=True, both=False)['$(arg camera_renderer)' or 'opengl'] }"
+      >
+        <sensor name="overview_camera">
+          <param name="color_enabled">false</param>
+        </sensor>
+        <sensor name="scene_camera">
+          <param name="color_enabled">false</param>
+        </sensor>
+        <sensor name="wrist_camera">
+          <param name="color_enabled">false</param>
+        </sensor>
+      </xacro:if>
+      <!-- both: each renderer's color image goes under its own prefix, so no consumer reads one renderer while expecting the other. Depth and points stay unprefixed. -->
+      <xacro:if
+        value="${ dict(opengl=False, nyx=False, both=True)['$(arg camera_renderer)' or 'opengl'] }"
+      >
+        <sensor name="overview_camera">
+          <param name="rgb_topic">overview_camera/opengl/color</param>
+          <param name="camera_info_topic">overview_camera/opengl/camera_info</param>
+        </sensor>
+        <sensor name="scene_camera">
+          <param name="rgb_topic">scene_camera/opengl/color</param>
+          <param name="camera_info_topic">scene_camera/opengl/camera_info</param>
+        </sensor>
+        <sensor name="wrist_camera">
+          <param name="rgb_topic">wrist_camera/opengl/color</param>
+          <param name="camera_info_topic">wrist_camera/opengl/camera_info</param>
+        </sensor>
+      </xacro:if>
     </ros2_control>
 </robot>
