Commit message: fix(rebot): validate mock execution from the zeroed rest pose

File: src/rebot_bench_mock/description/rebot.urdf (robot description, URDF)
Before this commit: robot rebot_b601_rs, 15 links, 14 joints
Joints:
- joint gripper_joint1: limit lower=0 upper=0.043284165449 effort=500 velocity=0.0024 -> lower=0 upper=0.04328416544945937 effort=500 velocity=0.0024
- joint gripper_joint2: limit lower=0 upper=0.043284165449 effort=500 velocity=0.0024 -> lower=0 upper=0.04328416544945937 effort=500 velocity=0.0024
- joint joint7: limit lower=0 upper=5.410520681182 effort=14 velocity=0.3 -> lower=0 upper=5.410520681182422 effort=14 velocity=0.3

Commit message: feat(rebot_bench_mock): add optional wrist and scene RGB cameras

File: src/rebot_bench_mock/description/rebot.urdf (robot description, URDF)
Before this commit: robot rebot_b601_rs, 15 links, 14 joints
Links:
- added link scene_camera_color_optical_frame
- added link scene_camera_link
Joints:
- added joint scene_camera_mount_joint: type fixed, parent world, child scene_camera_link, origin xyz=0 0 0 rpy=0 0 0
- added joint scene_camera_optical_joint: type fixed, parent scene_camera_link, child scene_camera_color_optical_frame, origin xyz=0 0 0 rpy=-1.5707963267948966 0 -1.5707963267948966
