Commit message: chore(deps): refresh vendored franka_config to 7aeeddc449edf8d62b594f9e36a81da53e7796f9

File: src/external_dependencies/franka_config/franka_description/end_effectors/common/ee_with_one_link.xacro (robot description, xacro)
@@ -2,8 +2,8 @@
 <robot xmlns:xacro="http://www.ros.org/wiki/xacro" name="ee_with_one_link">
   <!-- safety_distance: Minimum safety distance in [m] by which the collision volumes are expanded and which is enforced during robot motions -->
-  <xacro:macro name="ee_with_one_link" params="connected_to:='' robot_type arm_prefix:='' ee_id ee_inertials rpy_ee:='0 0 0' xyz_ee:='0 0 0' tcp_xyz:='0 0 0' tcp_rpy:='0 0 0' safety_distance:=0 gazebo:=false description_pkg:=franka_description with_sc:=false">
+  <xacro:macro name="ee_with_one_link" params="connected_to:='' robot_type arm_prefix:='' ee_id ee_inertials rpy_ee:='0 0 0' xyz_ee:='0 0 0' tcp_xyz:='0 0 0' tcp_rpy:='0 0 0' safety_distance:=0 include_self_collision_geometry:=true description_pkg:=franka_description with_sc:=false no_prefix:=false">
     <xacro:property name="ee_prefix" default="robot_"/>
     <xacro:unless value="${robot_type == ''}">
-      <xacro:property name="ee_prefix" value="${arm_prefix}${robot_type}_" />
+      <xacro:property name="ee_prefix" value="${'' if no_prefix else arm_prefix + robot_type + '_'}" />
     </xacro:unless>
     <xacro:unless value="${connected_to == ''}">
@@ -14,5 +14,5 @@
       </joint>
     </xacro:unless>
-    <xacro:ee_link_with_sc name="${ee_id}" gazebo="${gazebo}" with_sc="${with_sc}">
+    <xacro:ee_link_with_sc name="${ee_id}" include_self_collision_geometry="${include_self_collision_geometry}" with_sc="${with_sc}">
       <self_collision_geometries>
         <xacro:collision_capsule xyz="0 0 0.04" direction="y" radius="${0.04+safety_distance}" length="0.1" />

File: src/external_dependencies/franka_config/franka_description/end_effectors/common/franka_hand.xacro (robot description, xacro)
@@ -11,5 +11,5 @@
                        tcp_rpy:='0 0 0'
                        safety_distance:=0
-                       gazebo:=false
+                       include_self_collision_geometry:=true
                        description_pkg:=franka_description
                        with_sc:=false
@@ -17,5 +17,5 @@
     <xacro:property name="ee_prefix" default="robot_"/>
     <xacro:unless value="${robot_type == ''}">
-      <xacro:property name="ee_prefix" value="${arm_prefix}${robot_type}_" />
+      <xacro:property name="ee_prefix" value="${'' if no_prefix else arm_prefix + robot_type + '_'}" />
     </xacro:unless>
     <xacro:unless value="${connected_to == ''}">
@@ -26,5 +26,5 @@
       </joint>
     </xacro:unless>
-    <xacro:ee_link_with_sc name="hand" gazebo="${gazebo}" with_sc="${with_sc}">
+    <xacro:ee_link_with_sc name="hand" include_self_collision_geometry="${include_self_collision_geometry}" with_sc="${with_sc}">
       <self_collision_geometries>
         <xacro:collision_capsule xyz="0 0 0.04" direction="y" radius="${0.04+safety_distance}" length="0.1" />

File: src/external_dependencies/franka_config/franka_description/end_effectors/common/utils.xacro (robot description, xacro)
@@ -26,11 +26,13 @@
   <!--  * detailed meshes for environmental collision checking    -->
   <!--  * and coarse geometry models for self-collision checking  -->
-  <!--    (only if 'gazebo' param is set)                         -->
+  <!--    (only if 'include_self_collision_geometry' is true)     -->
   <!--                                                            -->
   <!-- name:  Name of the end-effector (without prefix)             -->
   <!-- rpy:   Rotation of the *_sc link relative to parent [rad]  -->
   <!-- self_collision_geometries:  self <collision> models        -->
+  <!-- include_self_collision_geometry: emit the coarse capsules  -->
+  <!--   inside the *_sc sub-link (true) or leave it empty (false) -->
   <!-- ========================================================== -->
-  <xacro:macro name="ee_link_with_sc" params="name prefix=${ee_prefix} rpy:='0 0 0' **self_collision_geometries gazebo:=false with_sc:=false">
+  <xacro:macro name="ee_link_with_sc" params="name prefix=${ee_prefix} rpy:='0 0 0' **self_collision_geometries include_self_collision_geometry:=true with_sc:=false">
     <!-- sub-link defining detailed meshes for collision with environment -->
     <link name="${prefix}${name}">
@@ -50,7 +52,7 @@
     <xacro:if value="${with_sc}">
       <link name="${prefix}${name}_sc">
-        <xacro:unless value="${gazebo}">
+        <xacro:if value="${include_self_collision_geometry}">
           <xacro:insert_block name="self_collision_geometries" />
-        </xacro:unless>
+        </xacro:if>
       </link>
       <!-- fixed joint between both sub-links -->

File: src/external_dependencies/franka_config/franka_description/robots/common/franka_arm.xacro (robot description, xacro)
@@ -3,16 +3,18 @@
   <xacro:include filename="$(find franka_description)/robots/common/utils.xacro" />
   <!-- safety_distance: Minimum safety distance in [m] by which the collision volumes are expanded and which is enforced during robot motions -->
-  <!-- robot_type: Namespace of the robot arm. Serves to differentiate between arms in case of multiple instances. -->
+  <!-- robot_type: the franka robot arm type -->
   <!-- joint_limits: description of the joint limits that comes from a YAML file. Example definition: ${xacro.load_yaml('$(find franka_description)/robots/fr3/joint_limits.yaml')} -->
   <!-- kinematics: description of the kinematics that comes from a YAML file. Example definition: ${xacro.load_yaml('$(find franka_description)/robots/fr3/kinematics.yaml')} -->
   <!-- inertials: description of the inertials that comes from a YAML file. Example definition: ${xacro.load_yaml('$(find franka_description)/robots/fr3/inertials.yaml')} -->
   <!-- dynamics: description of the dynamics that comes from a YAML file. Example definition: ${xacro.load_yaml('$(find franka_description)/robots/fr3/dynamics.yaml')} -->
-  <xacro:macro name="franka_arm" params="robot_type arm_prefix:='' no_prefix:=false description_pkg:='franka_description' connected_to:='base' xyz:='0 0 0' rpy:='0 0 0' gazebo:='false' safety_distance:=0 joint_limits inertials kinematics accelerometer_config dynamics with_sc:=false" >
+  <xacro:macro name="franka_arm" params="robot_type arm_prefix:='' no_prefix:=false description_pkg:='franka_description' connected_to:='base' xyz:='0 0 0' rpy:='0 0 0' include_self_collision_geometry:='true' safety_distance:=0 with_sc:=false" >
+    <xacro:property name="joint_limits" value="${xacro.load_yaml('$(find franka_description)/robots/' + robot_type + '/joint_limits.yaml')}"/>
+    <xacro:property name="inertials" value="${xacro.load_yaml('$(find franka_description)/robots/' + robot_type  + '/inertials.yaml')}"/>
+    <xacro:property name="kinematics" value="${xacro.load_yaml('$(find franka_description)/robots/' + robot_type + '/kinematics.yaml')}"/>
+    <xacro:property name="accelerometer_config" value="${xacro.load_yaml('$(find franka_description)/robots/' + robot_type + '/accelerometers.yaml')}"/>
+    <xacro:property name="dynamics" value="${xacro.load_yaml('$(find franka_description)/robots/' + robot_type + '/dynamics.yaml')}"/>
     <!-- Define a property that defaults to 'arm_prefix_robot_type' concatenated with an underscore if 'no_prefix' is not set -->
     <xacro:property name="prefix" value="${'' if no_prefix else arm_prefix + robot_type + '_'}" />
     <xacro:property name="with_accelerometers" value="${'false' if accelerometer_config == 'none' else 'true'}" />
-    <xacro:if value="${gazebo}">
-      <xacro:property name="connected_to" value="" />
-    </xacro:if>
     <xacro:unless value="${not connected_to}">
       <link name="${connected_to}">
@@ -24,10 +26,10 @@
       </joint>
     </xacro:unless>
-    <xacro:link_with_sc no_prefix="${no_prefix}" name="link0" gazebo="${gazebo}" with_sc="${with_sc}" with_accelerometers="${with_accelerometers}">
+    <xacro:link_with_sc no_prefix="${no_prefix}" name="link0" include_self_collision_geometry="${include_self_collision_geometry}" with_sc="${with_sc}" with_accelerometers="${with_accelerometers}">
       <self_collision_geometries>
         <xacro:collision_capsule xyz="-0.075 0 0.06" direction="x" radius="${0.06+safety_distance}" length="0.03" />
       </self_collision_geometries>
     </xacro:link_with_sc>
-    <xacro:link_with_sc no_prefix="${no_prefix}" name="link1" gazebo="${gazebo}" with_sc="${with_sc}" with_accelerometers="${with_accelerometers}">
+    <xacro:link_with_sc no_prefix="${no_prefix}" name="link1" include_self_collision_geometry="${include_self_collision_geometry}" with_sc="${with_sc}" with_accelerometers="${with_accelerometers}">
       <self_collision_geometries>
         <xacro:collision_capsule xyz="0 0 -191.5e-3" radius="${0.06+safety_distance}" length="0.283" />
@@ -42,5 +44,5 @@
       <xacro:franka-dynamics name="joint1" config="${dynamics}" />
     </joint>
-    <xacro:link_with_sc no_prefix="${no_prefix}" name="link2" gazebo="${gazebo}" with_sc="${with_sc}" with_accelerometers="${with_accelerometers}">
+    <xacro:link_with_sc no_prefix="${no_prefix}" name="link2" include_self_collision_geometry="${include_self_collision_geometry}" with_sc="${with_sc}" with_accelerometers="${with_accelerometers}">
       <self_collision_geometries>
         <xacro:collision_capsule xyz="0 0 0" radius="${0.06+safety_distance}" length="0.12" />
@@ -55,5 +57,5 @@
       <xacro:franka-dynamics name="joint2" config="${dynamics}" />
     </joint>
-    <xacro:link_with_sc no_prefix="${no_prefix}" name="link3" gazebo="${gazebo}" with_sc="${with_sc}" with_accelerometers="${with_accelerometers}">
+    <xacro:link_with_sc no_prefix="${no_prefix}" name="link3" include_self_collision_geometry="${include_self_collision_geometry}" with_sc="${with_sc}" with_accelerometers="${with_accelerometers}">
       <self_collision_geometries>
         <xacro:collision_capsule xyz="0 0 -0.145" radius="${0.06+safety_distance}" length="0.15" />
@@ -68,5 +70,5 @@
       <xacro:franka-dynamics name="joint3" config="${dynamics}" />
     </joint>
-    <xacro:link_with_sc no_prefix="${no_prefix}" name="link4" gazebo="${gazebo}" with_sc="${with_sc}" with_accelerometers="${with_accelerometers}">
+    <xacro:link_with_sc no_prefix="${no_prefix}" name="link4" include_self_collision_geometry="${include_self_collision_geometry}" with_sc="${with_sc}" with_accelerometers="${with_accelerometers}">
       <self_collision_geometries>
         <xacro:collision_capsule xyz="0 0 0" radius="${0.06+safety_distance}" length="0.12" />
@@ -81,5 +83,5 @@
       <xacro:franka-dynamics name="joint4" config="${dynamics}" />
     </joint>
-    <xacro:link_with_sc no_prefix="${no_prefix}" name="link5" gazebo="${gazebo}" with_sc="${with_sc}" with_accelerometers="${with_accelerometers}">
+    <xacro:link_with_sc no_prefix="${no_prefix}" name="link5" include_self_collision_geometry="${include_self_collision_geometry}" with_sc="${with_sc}" with_accelerometers="${with_accelerometers}">
       <self_collision_geometries>
         <xacro:collision_capsule xyz="0 0 -0.26"    radius="${0.060+safety_distance}" length="0.10" />
@@ -95,5 +97,5 @@
       <xacro:franka-dynamics name="joint5" config="${dynamics}" />
     </joint>
-    <xacro:link_with_sc no_prefix="${no_prefix}" name="link6" gazebo="${gazebo}" with_sc="${with_sc}" with_accelerometers="false">
+    <xacro:link_with_sc no_prefix="${no_prefix}" name="link6" include_self_collision_geometry="${include_self_collision_geometry}" with_sc="${with_sc}" with_accelerometers="false">
       <self_collision_geometries>
         <xacro:collision_capsule xyz="0 0 -0.03" radius="${0.05+safety_distance}" length="0.08" />
@@ -108,5 +110,5 @@
       <xacro:franka-dynamics name="joint6" config="${dynamics}" />
     </joint>
-    <xacro:link_with_sc no_prefix="${no_prefix}" name="link7" gazebo="${gazebo}" rpy="0 0 ${pi/4}" with_sc="${with_sc}" with_accelerometers="false">
+    <xacro:link_with_sc no_prefix="${no_prefix}" name="link7" include_self_collision_geometry="${include_self_collision_geometry}" rpy="0 0 ${pi/4}" with_sc="${with_sc}" with_accelerometers="false">
       <self_collision_geometries>
         <xacro:collision_capsule xyz="0 0 0.01" direction="z" radius="${0.04+safety_distance}" length="0.14" />
