Commit message: chore(deps): refresh vendored franka_config to 7aeeddc449edf8d62b594f9e36a81da53e7796f9

File: src/external_dependencies/franka_config/franka_description/robots/common/franka_robot.xacro (robot description, xacro)
@@ -1,11 +1,6 @@
-<?xml version='1.0' encoding='utf-8'?>
+<?xml version="1.0" encoding="utf-8"?>
 <robot xmlns:xacro="http://www.ros.org/wiki/xacro">
   <xacro:macro name="franka_robot"
-              params="robot_type
-                      joint_limits
-                      kinematics
-                      accelerometer_config:=none
-                      inertials
-                      dynamics
+    params="robot_type
                       parent:='world'
                       xyz:='0 0 0'
@@ -13,5 +8,5 @@
                       xyz_ee:='0 0 0'
                       rpy_ee:='0 0 0'
-                      tcp_xyz:='0 0 0'
+                      tcp_xyz:=''
                       tcp_rpy:='0 0 0'
                       safety_distance:='0.03'
@@ -19,19 +14,23 @@
                       ee_id:=none
                       special_connection:=''
-                      gazebo:='false'
+                      include_self_collision_geometry:='true'
                       with_sc:='false'
-                      ros2_control:=false
-                      robot_ip:=''
-                      use_fake_hardware:=false
-                      fake_sensor_commands:=false
-                      gazebo_effort:=false
-                      no_prefix:='false'
+                      no_prefix:=false
                       arm_prefix:=''
                       description_pkg:='franka_description'
-                      connected_to:='base'
-                      is_async:=false
-                      thread_priority:=50">
-    <xacro:include filename="$(find franka_description)/robots/common/utils.xacro" />
-    <xacro:include filename="$(find franka_description)/robots/common/franka_arm.xacro" />
+                      connected_to:='base'">
+    <xacro:include filename="$(find franka_description)/robots/common/utils.xacro"/>
+    <xacro:include filename="$(find franka_description)/robots/common/franka_arm.xacro"/>
+    <!-- The tcp offset belongs to the end effector, so an empty tcp_xyz resolves to
+         that end effector's own value rather than to zero. These must match the
+         defaults in end_effectors/<ee_id>/<ee_id>_arguments.xacro, which
+         test_tcp_offset_matches_end_effector enforces. -->
+    <xacro:property name="ee_tcp_xyz"
+      value="${'0 0 0.1034' if ee_id == 'franka_hand' else '0 0 0.105' if ee_id == 'cobot_pump' else '0 0 0'}"/>
+    <xacro:property name="tcp_xyz_resolved" value="${ee_tcp_xyz if tcp_xyz == '' else tcp_xyz}"/>
+    <!-- franka_arm derives its link names this way, so the end effector has to attach to
+         the same names and prefix itself the same way, or the two halves of the robot do
+         not reference each other. -->
+    <xacro:property name="link_prefix" value="${'' if no_prefix else arm_prefix + robot_type + '_'}"/>
     <xacro:franka_arm
       robot_type="${robot_type}"
@@ -41,35 +40,33 @@
       rpy="${rpy}"
       safety_distance="0.03"
-      gazebo="${gazebo}"
-      joint_limits="${joint_limits}"
-      kinematics="${kinematics}"
-      accelerometer_config="${accelerometer_config}"
-      inertials="${inertials}"
-      dynamics="${dynamics}"
+      include_self_collision_geometry="${include_self_collision_geometry}"
       with_sc="${with_sc}"
       connected_to="${connected_to}"
     />
-    <xacro:if value="${hand and ee_id == 'franka_hand'}">
+    <xacro:if value="${hand and ee_id== 'franka_hand'}">
       <xacro:include filename="$(find franka_description)/end_effectors/common/franka_hand.xacro"/>
-      <xacro:include filename="$(find franka_description)/end_effectors/common/utils.xacro" />
+      <xacro:include filename="$(find franka_description)/end_effectors/common/utils.xacro"/>
       <xacro:if value="${robot_type == 'fp3'}">
-        <xacro:property name="ee_color" value="black" />
+        <xacro:property name="ee_color" value="black"/>
       </xacro:if>
-      <xacro:if value="${robot_type == 'fr3' or robot_type == 'fer' or robot_type == 'fr3v2' or robot_type == 'fr3v2_1'}">
-        <xacro:property name="ee_color" value="white" />
+      <xacro:if
+        value="${robot_type == 'fr3' or robot_type == 'fer' or robot_type == 'fr3v2' or robot_type == 'fr3v2_1'}">
+        <xacro:property name="ee_color" value="white"/>
       </xacro:if>
-      <xacro:property name="connection" value="${special_connection if special_connection != '' else robot_type + '_link8'}" />
+      <xacro:property name="connection"
+        value="${arm_prefix + special_connection if special_connection != '' else link_prefix + 'link8'}"/>
       <xacro:franka_hand
-        connected_to="${arm_prefix}${connection}"
+        connected_to="${connection}"
         robot_type="${robot_type}"
         arm_prefix="${arm_prefix}"
+        no_prefix="${no_prefix}"
         ee_id="${ee_id}_${ee_color}"
         ee_inertials="${xacro.load_yaml('$(find franka_description)/end_effectors/' + ee_id + '/inertials.yaml')}"
         rpy_ee="${rpy_ee}"
         xyz_ee="${xyz_ee}"
-        tcp_xyz="${tcp_xyz}"
+        tcp_xyz="${tcp_xyz_resolved}"
         tcp_rpy="${tcp_rpy}"
         safety_distance="${safety_distance}"
-        gazebo="${gazebo}"
+        include_self_collision_geometry="${include_self_collision_geometry}"
         description_pkg="${description_pkg}"
         with_sc="${with_sc}"
@@ -78,84 +75,24 @@
     <xacro:if value="${hand and ee_id != 'none' and ee_id != 'franka_hand'}">
       <xacro:include filename="$(find franka_description)/end_effectors/common/ee_with_one_link.xacro"/>
-      <xacro:include filename="$(find franka_description)/end_effectors/common/utils.xacro" />
-      <xacro:property name="connection" value="${special_connection if special_connection != '' else robot_type + '_link8'}" />
+      <xacro:include filename="$(find franka_description)/end_effectors/common/utils.xacro"/>
+      <xacro:property name="connection"
+        value="${arm_prefix + special_connection if special_connection != '' else link_prefix + 'link8'}"/>
       <xacro:ee_with_one_link
-        connected_to="${arm_prefix}${connection}"
+        connected_to="${connection}"
         robot_type="${robot_type}"
         arm_prefix="${arm_prefix}"
+        no_prefix="${no_prefix}"
         ee_id="${ee_id}"
         ee_inertials="${xacro.load_yaml('$(find franka_description)/end_effectors/' + ee_id + '/inertials.yaml')}"
         rpy_ee="${rpy_ee}"
         xyz_ee="${xyz_ee}"
-        tcp_xyz="${tcp_xyz}"
+        tcp_xyz="${tcp_xyz_resolved}"
         tcp_rpy="${tcp_rpy}"
         safety_distance="${safety_distance}"
-        gazebo="${gazebo}"
+        include_self_collision_geometry="${include_self_collision_geometry}"
         description_pkg="${description_pkg}"
         with_sc="${with_sc}"
       />
     </xacro:if>
-    <!-- Definition of additional Gazebo tags -->
-    <xacro:if value="${gazebo}">
-      <xacro:if value="${parent != ''}">
-        <!-- Gazebo requires a joint to a link called "world" for statically mounted robots -->
-        <xacro:if value="${parent == 'world'}">
-          <link name="${parent}" />
-        </xacro:if>
-        <joint name="${parent}_joint" type="fixed">
-          <origin xyz="${xyz}" rpy="${rpy}" />
-          <parent link="${parent}" />
-          <child  link="${arm_prefix}${robot_type}_link0" />
-        </joint>
-      </xacro:if>
-      <xacro:gazebo-joint joint="${arm_prefix}${robot_type}_joint1" transmission="hardware_interface/PositionJointInterface" />
-      <xacro:gazebo-joint joint="${arm_prefix}${robot_type}_joint2" transmission="hardware_interface/PositionJointInterface" />
-      <xacro:gazebo-joint joint="${arm_prefix}${robot_type}_joint3" transmission="hardware_interface/PositionJointInterface" />
-      <xacro:gazebo-joint joint="${arm_prefix}${robot_type}_joint4" transmission="hardware_interface/PositionJointInterface" />
-      <xacro:gazebo-joint joint="${arm_prefix}${robot_type}_joint5" transmission="hardware_interface/PositionJointInterface" />
-      <xacro:gazebo-joint joint="${arm_prefix}${robot_type}_joint6" transmission="hardware_interface/PositionJointInterface" />
-      <xacro:gazebo-joint joint="${arm_prefix}${robot_type}_joint7" transmission="hardware_interface/PositionJointInterface" />
-      <xacro:gazebo-joint joint="${arm_prefix}${robot_type}_joint1" transmission="hardware_interface/VelocityJointInterface" />
-      <xacro:gazebo-joint joint="${arm_prefix}${robot_type}_joint2" transmission="hardware_interface/VelocityJointInterface" />
-      <xacro:gazebo-joint joint="${arm_prefix}${robot_type}_joint3" transmission="hardware_interface/VelocityJointInterface" />
-      <xacro:gazebo-joint joint="${arm_prefix}${robot_type}_joint4" transmission="hardware_interface/VelocityJointInterface" />
-      <xacro:gazebo-joint joint="${arm_prefix}${robot_type}_joint5" transmission="hardware_interface/VelocityJointInterface" />
-      <xacro:gazebo-joint joint="${arm_prefix}${robot_type}_joint6" transmission="hardware_interface/VelocityJointInterface" />
-      <xacro:gazebo-joint joint="${arm_prefix}${robot_type}_joint7" transmission="hardware_interface/VelocityJointInterface" />
-      <xacro:gazebo-joint joint="${arm_prefix}${robot_type}_joint1" transmission="hardware_interface/EffortJointInterface" />
-      <xacro:gazebo-joint joint="${arm_prefix}${robot_type}_joint2" transmission="hardware_interface/EffortJointInterface" />
-      <xacro:gazebo-joint joint="${arm_prefix}${robot_type}_joint3" transmission="hardware_interface/EffortJointInterface" />
-      <xacro:gazebo-joint joint="${arm_prefix}${robot_type}_joint4" transmission="hardware_interface/EffortJointInterface" />
-      <xacro:gazebo-joint joint="${arm_prefix}${robot_type}_joint5" transmission="hardware_interface/EffortJointInterface" />
-      <xacro:gazebo-joint joint="${arm_prefix}${robot_type}_joint6" transmission="hardware_interface/EffortJointInterface" />
-      <xacro:gazebo-joint joint="${arm_prefix}${robot_type}_joint7" transmission="hardware_interface/EffortJointInterface" />
-      <xacro:transmission-franka-state robot_type="${robot_type}" />
-      <xacro:transmission-franka-model robot_type="${robot_type}"
-         root="${arm_prefix}${robot_type}_joint1"
-         tip="${arm_prefix}${robot_type}_joint8"
-       />
-      <xacro:if value="${ee_id == 'franka_hand'}">
-        <xacro:gazebo-joint joint="${arm_prefix}${robot_type}_finger_joint1" transmission="hardware_interface/EffortJointInterface" />
-        <xacro:gazebo-joint joint="${arm_prefix}${robot_type}_finger_joint2" transmission="hardware_interface/EffortJointInterface" />
-        <!-- Friction specific material for Rubber/Rubber contact -->
-        <xacro:gazebo-friction link="${arm_prefix}${robot_type}_leftfinger" mu="1.13" />
-        <xacro:gazebo-friction link="${arm_prefix}${robot_type}_rightfinger" mu="1.13" />
-      </xacro:if>
-    </xacro:if>
-    <xacro:if value="${ros2_control}">
-      <xacro:include filename="$(find franka_description)/robots/common/franka_arm.ros2_control.xacro"/>
-      <xacro:franka_arm_ros2_control
-          robot_type="${robot_type}"
-          robot_ip="${robot_ip}"
-          use_fake_hardware="${use_fake_hardware}"
-          fake_sensor_commands="${fake_sensor_commands}"
-          gazebo="${gazebo}"
-          hand="${hand}"
-          gazebo_effort="${gazebo_effort}"
-          arm_prefix="${arm_prefix}"
-          is_async="${is_async}"
-          thread_priority="${thread_priority}"
-      />
-    </xacro:if>
   </xacro:macro>
 </robot>

File: src/external_dependencies/franka_config/franka_description/robots/common/utils.xacro (robot description, xacro)
@@ -26,11 +26,13 @@
   <!--  * detailed meshes for environmental collision checking    -->
   <!--  * and coarse geometry models for self-collision checking  -->
-  <!--    (only if 'gazebo' param is set)                         -->
+  <!--    (only if 'include_self_collision_geometry' is true)     -->
   <!--                                                            -->
   <!-- name:  Name of the robot link (without prefix)             -->
   <!-- rpy:   Rotation of the *_sc link relative to parent [rad]  -->
   <!-- self_collision_geometries:  self <collision> models        -->
+  <!-- include_self_collision_geometry: emit the coarse capsules  -->
+  <!--   inside the *_sc sub-link (true) or leave it empty (false) -->
   <!-- ========================================================== -->
-  <xacro:macro name="link_with_sc" params="name no_prefix:='false' rpy:='0 0 0' **self_collision_geometries gazebo:=false with_sc:=false with_accelerometers:=false">
+  <xacro:macro name="link_with_sc" params="name no_prefix:='false' rpy:='0 0 0' **self_collision_geometries include_self_collision_geometry:=true with_sc:=false with_accelerometers:=false">
     <xacro:property name="prefix" value="${'' if no_prefix else arm_prefix + robot_type + '_'}" />
     <!-- sub-link defining detailed meshes for collision with environment -->
@@ -51,7 +53,7 @@
     <xacro:if value="${with_sc}">
       <link name="${prefix}${name}_sc">
-        <xacro:unless value="${gazebo}">
+        <xacro:if value="${include_self_collision_geometry}">
           <xacro:insert_block name="self_collision_geometries" />
-        </xacro:unless>
+        </xacro:if>
       </link>
       <!-- fixed joint between both sub-links -->
@@ -107,98 +109,4 @@
     </collision>
   </xacro:macro>
-  <!-- ========================================================== -->
-  <!-- Adds the required tags to simulate one joint in gazebo     -->
-  <!--                                                            -->
-  <!-- joint - Name of the fer joint to simulate                  -->
-  <!-- transmission - type of the transmission of the joint       -->
-  <!-- ========================================================== -->
-  <xacro:macro name="gazebo-joint" params="joint transmission:=hardware_interface/EffortJointInterface">
-    <gazebo reference="${joint}">
-      <!-- Needed for ODE to output external wrenches on joints -->
-      <provideFeedback>true</provideFeedback>
-    </gazebo>
-    <transmission name="${joint}_transmission">
-      <type>transmission_interface/SimpleTransmission</type>
-      <joint name="${joint}">
-        <hardwareInterface>${transmission}</hardwareInterface>
-      </joint>
-      <actuator name="${joint}_motor">
-        <hardwareInterface>${transmission}</hardwareInterface>
-      </actuator>
-    </transmission>
-  </xacro:macro>
-  <xacro:macro name="gazebo-friction" params="link mu">
-    <gazebo reference="${link}">
-      <collision>
-        <max_contacts>10</max_contacts>
-        <surface>
-          <contact>
-            <ode>
-              <!-- These two parameter need application specific tuning. -->
-              <!-- Usually you want no "snap out" velocity and a generous -->
-              <!-- penetration depth to keep the grasping stable -->
-              <max_vel>0</max_vel>
-              <min_depth>0.001</min_depth>
-            </ode>
-          </contact>
-          <friction>
-            <ode>
-              <mu>${mu}</mu>
-              <mu2>${mu}</mu2>
-            </ode>
-          </friction>
-          <bounce/>
-        </surface>
-      </collision>
-    </gazebo>
-  </xacro:macro>
-  <!-- ========================================================== -->
-  <!-- Adds the required tags to provide a `FrankaStateInterface` -->
-  <!-- when simulating with franka_hw_sim plugin                  -->
-  <!--                                                            -->
-  <!-- robot_type - Arm ID of the fer to simulate (default 'fer')     -->
-  <!-- ========================================================== -->
-  <xacro:macro name="transmission-franka-state" params="robot_type:=fer">
-    <transmission name="${arm_prefix}${robot_type}_franka_state">
-      <type>franka_hw/FrankaStateInterface</type>
-      <joint name="${arm_prefix}${robot_type}_joint1"><hardwareInterface>franka_hw/FrankaStateInterface</hardwareInterface></joint>
-      <joint name="${arm_prefix}${robot_type}_joint2"><hardwareInterface>franka_hw/FrankaStateInterface</hardwareInterface></joint>
-      <joint name="${arm_prefix}${robot_type}_joint3"><hardwareInterface>franka_hw/FrankaStateInterface</hardwareInterface></joint>
-      <joint name="${arm_prefix}${robot_type}_joint4"><hardwareInterface>franka_hw/FrankaStateInterface</hardwareInterface></joint>
-      <joint name="${arm_prefix}${robot_type}_joint5"><hardwareInterface>franka_hw/FrankaStateInterface</hardwareInterface></joint>
-      <joint name="${arm_prefix}${robot_type}_joint6"><hardwareInterface>franka_hw/FrankaStateInterface</hardwareInterface></joint>
-      <joint name="${arm_prefix}${robot_type}_joint7"><hardwareInterface>franka_hw/FrankaStateInterface</hardwareInterface></joint>
-      <actuator name="${arm_prefix}${robot_type}_motor1"><hardwareInterface>franka_hw/FrankaStateInterface</hardwareInterface></actuator>
-      <actuator name="${arm_prefix}${robot_type}_motor2"><hardwareInterface>franka_hw/FrankaStateInterface</hardwareInterface></actuator>
-      <actuator name="${arm_prefix}${robot_type}_motor3"><hardwareInterface>franka_hw/FrankaStateInterface</hardwareInterface></actuator>
-      <actuator name="${arm_prefix}${robot_type}_motor4"><hardwareInterface>franka_hw/FrankaStateInterface</hardwareInterface></actuator>
-      <actuator name="${arm_prefix}${robot_type}_motor5"><hardwareInterface>franka_hw/FrankaStateInterface</hardwareInterface></actuator>
-      <actuator name="${arm_prefix}${robot_type}_motor6"><hardwareInterface>franka_hw/FrankaStateInterface</hardwareInterface></actuator>
-      <actuator name="${arm_prefix}${robot_type}_motor7"><hardwareInterface>franka_hw/FrankaStateInterface</hardwareInterface></actuator>
-    </transmission>
-  </xacro:macro>
-  <!-- ============================================================ -->
-  <!-- Adds the required tags to provide a `FrankaModelInterface`   -->
-  <!-- when simulating with franka_hw_sim plugin                    -->
-  <!--                                                              -->
-  <!-- robot_type - Arm ID of the fer to simulate (default 'fer')       -->
-  <!-- root   - Joint name of the base of the robot                 -->
-  <!-- tip    - Joint name of the tip of the robot (flange or hand) -->
-  <!-- ============================================================ -->
-  <xacro:macro name="transmission-franka-model" params="robot_type:=fer root:=fer_joint1 tip:=fer_joint7">
-    <transmission name="${arm_prefix}${robot_type}_franka_model">
-      <type>franka_hw/FrankaModelInterface</type>
-      <joint name="${root}">
-        <role>root</role>
-        <hardwareInterface>franka_hw/FrankaModelInterface</hardwareInterface>
-      </joint>
-      <joint name="${tip}">
-        <role>tip</role>
-        <hardwareInterface>franka_hw/FrankaModelInterface</hardwareInterface>
-      </joint>
-      <actuator name="${root}_motor_root"><hardwareInterface>franka_hw/FrankaModelInterface</hardwareInterface></actuator>
-      <actuator name="${tip}_motor_tip"  ><hardwareInterface>franka_hw/FrankaModelInterface</hardwareInterface></actuator>
-    </transmission>
-  </xacro:macro>
   <xacro:macro name="inertia-cylinder" params="mass radius h">
     <inertial>
@@ -245,5 +153,7 @@
              friction="${dynamics.friction}"
              mu_coulomb="${dynamics.mu_coulomb}"
-             mu_viscous="${dynamics.mu_viscous}" />
+             mu_viscous="${dynamics.mu_viscous}"
+             motor_inertia="${dynamics.motor_inertia}"
+             gear_ratio="${dynamics.gear_ratio}" />
   </xacro:macro>
   <!-- ========================================================================= -->
