Commit message: feat(rebot_bench_base_config): add KDL gravity compensation for impedance mode
In motion (impedance) mode the reBot driver sent no torque feedforward, so
a loaded joint settled short of its target by load torque / kp.

Add kdl_gravity_compensation_controller, a ros2_control controller that
reads joint positions, computes the chain's holding torque with KDL
ChainDynParam::JntToGravity on the robot description, and writes
gain * torque + offset to each joint's effort command interface. It claims
nothing else, so the trajectory admittance, jog and Cartesian controllers
keep position. Parameters: joints, root/tip link, gravity_vector (mount
orientation), payload mass and centre of mass in the tip frame, and
per-joint gains and offsets. Gains and offsets apply live; the rest on
configure. It publishes the positions it used and the efforts it wrote on
~/commanded_effort. Deactivating it writes 0.

Re-vendor robstride_hardware_interface at the fork's
picknik/gravity-feedforward branch. The joint's effort command is the
motion-mode torque feedforward, now clamped to a per-motor
max_feedforward_effort that defaults below rated torque (9 N*m RS06,
3.5 N*m RS00). The branch also decodes the 0x15 fault word
little-endian, which the SDK read big-endian.

rebot_bench_base_config declares effort on joint1-joint6 for the real arm
in motion mode only, and loads gravity_compensation_controller inactive
with every gain at 0. The README covers enabling it, live tuning, its
parameters, and the gains tuned on the bench arm at the Raised pose
(joint2 0.25, joint3 1.25, joint4 1.50), which cut holding sag from up to
50.7 mrad to under 3 mrad.

File: src/rebot_bench_base_config/description/rebot.urdf.xacro (robot description, xacro)
@@ -10,6 +10,7 @@
   <xacro:arg name="torque_enable" default="true" />
   <!-- Real hardware only; joint1-joint6 control mode. "motion" is impedance
-       (MIT): torque = kp * error + kd * velocity error, with no gravity
-       feedforward, so a loaded joint settles short by load torque / kp.
+       (MIT): torque = kp * error + kd * velocity error + effort. effort is 0
+       unless gravity_compensation_controller is active, and without it a
+       loaded joint settles short by load torque / kp.
        "position_csp" is the motor's own position loop, which settles on
        target and is capped by the motor's stored speed limit (0x7017). The
@@ -486,5 +487,5 @@
   -->
   <xacro:property name="arm_mode" value="${dict(motion='motion', position_csp='position_csp')['$(arg arm_control_mode)']}" />
-  <xacro:macro name="rebot_joint" params="name id model kp kd mode:=${arm_mode}">
+  <xacro:macro name="rebot_joint" params="name id model kp kd mode:=${arm_mode} feedforward:=true">
     <joint name="${name}">
       <xacro:if value="${'$(arg hardware_interface)' == 'real'}">
@@ -493,7 +494,15 @@
       <command_interface name="position" />
       <!--
-        Mock only. Every controller in config/control/rebot.ros2_control.yaml
-        commands `position`, and motion mode is driven through `position`
-        alone; the driver exports whatever is declared, so a velocity
+        Real motion mode only: the impedance law's torque feedforward, written
+        by gravity_compensation_controller and clamped by the driver to the
+        motor's max_feedforward_effort. Nothing writes it by default.
+      -->
+      <xacro:if value="${'$(arg hardware_interface)' == 'real' and mode == 'motion' and feedforward}">
+        <command_interface name="effort" />
+      </xacro:if>
+      <!--
+        Mock only. Every motion controller in config/control/rebot.ros2_control.yaml
+        commands `position`, and motion mode's target is driven through
+        `position` alone; the driver exports whatever is declared, so a velocity
         declaration here would be claimable and then never written - a joint
         that accepts commands and does not move, with no error to explain it.
@@ -564,5 +573,5 @@
     <xacro:rebot_joint name="joint5" id="5" model="RS00" kp="50.0" kd="4.0" />
     <xacro:rebot_joint name="joint6" id="6" model="RS00" kp="50.0" kd="4.0" />
-    <xacro:rebot_joint name="joint7" id="7" model="RS00" kp="12.0" kd="0.05" mode="motion" />
+    <xacro:rebot_joint name="joint7" id="7" model="RS00" kp="12.0" kd="0.05" mode="motion" feedforward="false" />
   </ros2_control>
 </robot>

Commit message: feat(rebot_bench_base_config): add the real RobStride hardware backend
Vendor robstride_hardware_interface (pinned to a fork carrying
hold_torque_on_deactivate), robstride_sdk and robstride_interfaces under
src/external_dependencies, each byte-identical to its UPSTREAM.yaml pin.

hardware_interface: real drives the seven motors over SocketCAN; mock stays
the default and rebot_bench_sim stays mock-only. joint1-joint6 run in
impedance (motion) mode by default, or in the motor's own position loop
with arm_control_mode: position_csp; impedance sends no gravity
feedforward, so a loaded joint settles short by load torque / kp. The
gripper always uses motion mode. The arm has no brakes, so a clean stop holds the pose
(hold_torque_on_deactivate with motor_can_timeout_ms 0) and losing one joint
freezes the rest. position is the only real command interface.

Drive all seven joints with MoveIt Pro's joint_trajectory_admittance_controller
in place of the ros2_controllers JointTrajectoryController, through a new
manipulator_and_gripper SRDF group. With no force/torque sensor it runs as a
plain trajectory controller, and it rejects a trajectory whose first point is
more than 0.15 rad from the measured position. Its path and goal tolerances
(0.15 and 0.1 rad) are sized for motion mode's gravity sag. The Objectives use its jtac
execution pipeline.

Add Plan reBot Joint Move, which plans to a named waypoint or
target_positions and saves the trajectory and its reverse without moving,
and Execute reBot Joint Trajectory, which validates and runs a saved one
unchanged. Add two small waypoints near home; joint3 targets sit 2 mrad
inside its 0.0 lower limit, because a target exactly on a limit fails
planning.

Raise the gripper (joint7) planning and jog limits to 3.0 rad/s and 6.0
rad/s^2, so a full stroke takes about 2 s; the arm joints stay at 0.3 rad/s.

Default the optional scene camera to 640x400 at an explicit ISP ratio of
1/2, so it keeps the full field of view at 30 fps.

Shrink the D435 visual mesh from 15.8 MB to 1.7 MB by decimation (same
origin, scale and material), under the UI's 10 MB recommendation.

The README covers selection, host CAN bring-up, non-instanced running, the
start/home/stop procedure, stopping behaviour, controllers, Objectives,
cameras, what has been run on the bench arm, and known limitations.

File: src/rebot_bench_base_config/description/rebot.urdf.xacro (robot description, xacro)
@@ -3,6 +3,19 @@
 <robot name="rebot_b601_rs" xmlns:xacro="http://www.ros.org/wiki/xacro">
   <xacro:arg name="hardware_interface" default="mock" />
-  <!-- A future real driver belongs here; unsupported selectors fail expansion. -->
-  <xacro:property name="hardware_plugins" value="${dict(mock='mock_components/GenericSystem')}" />
+  <!-- Real hardware only; ignored by mock. The bench runs one 1 Mbps bus. -->
+  <xacro:arg name="can_interface" default="can0" />
+  <!-- false brings the arm up readable but limp: state is published and the
+       joints can be moved by hand, nothing is commanded. The first session on
+       real hardware uses this. -->
+  <xacro:arg name="torque_enable" default="true" />
+  <!-- Real hardware only; joint1-joint6 control mode. "motion" is impedance
+       (MIT): torque = kp * error + kd * velocity error, with no gravity
+       feedforward, so a loaded joint settles short by load torque / kp.
+       "position_csp" is the motor's own position loop, which settles on
+       target and is capped by the motor's stored speed limit (0x7017). The
+       gripper always uses motion. Unsupported values fail expansion. -->
+  <xacro:arg name="arm_control_mode" default="motion" />
+  <!-- Unsupported selectors fail expansion. -->
+  <xacro:property name="hardware_plugins" value="${dict(mock='mock_components/GenericSystem', real='robstride_hardware_interface/RobstrideHardware')}" />
   <material name="rs_base_black">
     <color rgba="0.055 0.065 0.060 1" />
@@ -360,5 +373,5 @@
     <child link="gripper_left" />
     <axis xyz="0 0 1" />
-    <limit lower="0" upper="0.04328416544945937" effort="500" velocity="0.0024" />
+    <limit lower="0" upper="0.04328416544945937" effort="500" velocity="0.024" />
     <mimic joint="joint7" multiplier="0.008" offset="0" />
   </joint>
@@ -395,5 +408,5 @@
     <child link="gripper_right" />
     <axis xyz="0 0 1" />
-    <limit lower="0" upper="0.04328416544945937" effort="500" velocity="0.0024" />
+    <limit lower="0" upper="0.04328416544945937" effort="500" velocity="0.024" />
     <mimic joint="joint7" multiplier="0.008" offset="0" />
   </joint>
@@ -403,5 +416,5 @@
     <child link="gripper_motor_frame" />
     <axis xyz="0 0 1" />
-    <limit lower="0" upper="5.410520681182422" velocity="0.3" effort="14" />
+    <limit lower="0" upper="5.410520681182422" velocity="3.0" effort="14" />
   </joint>
   <link name="world" />
@@ -461,12 +474,32 @@
     <origin xyz="0 0 0" rpy="-1.5707963267948966 0 -1.5707963267948966" />
   </joint>
-  <ros2_control name="RebotMockSystem" type="system">
-    <hardware>
-      <plugin>${hardware_plugins['$(arg hardware_interface)']}</plugin>
-      <param name="calculate_dynamics">true</param>
-    </hardware>
-    <joint name="joint1">
+  <!--
+    One motor per joint on a single CAN bus, ids 1-7 matching joint1-joint7.
+    actuator_type selects the motor's CAN quantization ranges, so RS06 on the
+    three base joints and RS00 on the wrist and gripper is not cosmetic: the
+    wrong model silently rescales every position, velocity and effort.
+    joint1-joint6 use the arm_control_mode argument (see its comment above);
+    the gripper always uses motion mode. kp/kd act only in motion mode and
+    start from Seeed's tuned follower values for this arm.
+    The URDF is already in the motor frame with the measured limits, so no
+    `direction` override is needed anywhere - joint frame equals motor frame.
+  -->
+  <xacro:property name="arm_mode" value="${dict(motion='motion', position_csp='position_csp')['$(arg arm_control_mode)']}" />
+  <xacro:macro name="rebot_joint" params="name id model kp kd mode:=${arm_mode}">
+    <joint name="${name}">
+      <xacro:if value="${'$(arg hardware_interface)' == 'real'}">
+        <param name="id">${id}</param>
+      </xacro:if>
       <command_interface name="position" />
-      <command_interface name="velocity" />
+      <!--
+        Mock only. Every controller in config/control/rebot.ros2_control.yaml
+        commands `position`, and motion mode is driven through `position`
+        alone; the driver exports whatever is declared, so a velocity
+        declaration here would be claimable and then never written - a joint
+        that accepts commands and does not move, with no error to explain it.
+      -->
+      <xacro:if value="${'$(arg hardware_interface)' == 'mock'}">
+        <command_interface name="velocity" />
+      </xacro:if>
       <state_interface name="position">
         <param name="initial_value">0.0</param>
@@ -476,64 +509,60 @@
       </state_interface>
     </joint>
-    <joint name="joint2">
-      <command_interface name="position" />
-      <command_interface name="velocity" />
-      <state_interface name="position">
-        <param name="initial_value">0.0</param>
-      </state_interface>
-      <state_interface name="velocity">
-        <param name="initial_value">0.0</param>
-      </state_interface>
-    </joint>
-    <joint name="joint3">
-      <command_interface name="position" />
-      <command_interface name="velocity" />
-      <state_interface name="position">
-        <param name="initial_value">0.0</param>
-      </state_interface>
-      <state_interface name="velocity">
-        <param name="initial_value">0.0</param>
-      </state_interface>
-    </joint>
-    <joint name="joint4">
-      <command_interface name="position" />
-      <command_interface name="velocity" />
-      <state_interface name="position">
-        <param name="initial_value">0.0</param>
-      </state_interface>
-      <state_interface name="velocity">
-        <param name="initial_value">0.0</param>
-      </state_interface>
-    </joint>
-    <joint name="joint5">
-      <command_interface name="position" />
-      <command_interface name="velocity" />
-      <state_interface name="position">
-        <param name="initial_value">0.0</param>
-      </state_interface>
-      <state_interface name="velocity">
-        <param name="initial_value">0.0</param>
-      </state_interface>
-    </joint>
-    <joint name="joint6">
-      <command_interface name="position" />
-      <command_interface name="velocity" />
-      <state_interface name="position">
-        <param name="initial_value">0.0</param>
-      </state_interface>
-      <state_interface name="velocity">
-        <param name="initial_value">0.0</param>
-      </state_interface>
-    </joint>
-    <joint name="joint7">
-      <command_interface name="position" />
-      <command_interface name="velocity" />
-      <state_interface name="position">
-        <param name="initial_value">0.0</param>
-      </state_interface>
-      <state_interface name="velocity">
-        <param name="initial_value">0.0</param>
-      </state_interface>
-    </joint>
+    <xacro:if value="${'$(arg hardware_interface)' == 'real'}">
+      <!--
+        The motor as a device, matched to its joint by id. Motor health is
+        published on the component's own ~/robstride_state topic every read()
+        cycle, so no gpio state interface is declared: nothing would claim one.
+      -->
+      <gpio name="${name}_motor">
+        <param name="type">robstride</param>
+        <param name="ID">${id}</param>
+        <param name="actuator_type">${model}</param>
+        <param name="can_interface">$(arg can_interface)</param>
+        <param name="control_mode">${mode}</param>
+        <param name="kp">${kp}</param>
+        <param name="kd">${kd}</param>
+      </gpio>
+    </xacro:if>
+  </xacro:macro>
+  <ros2_control name="RebotSystem" type="system">
+    <hardware>
+      <!-- Indexed unconditionally so an unsupported selector fails expansion
+           rather than yielding a description with no hardware plugin. -->
+      <plugin>${hardware_plugins['$(arg hardware_interface)']}</plugin>
+      <xacro:if value="${'$(arg hardware_interface)' == 'mock'}">
+        <param name="calculate_dynamics">true</param>
+      </xacro:if>
+      <xacro:if value="${'$(arg hardware_interface)' == 'real'}">
+        <!-- Host address this arm's motors are already configured to answer. -->
+        <param name="master_id">253</param>
+        <param name="number_of_joints">7</param>
+        <!--
+          The bench arm has no brakes and may only be limped at its home pose,
+          so a clean stop must hold the pose rather than drop the arm.
+          That hold is only real while the motors' own CAN_TIMEOUT watchdog is
+          off: deactivation closes the bus, and an armed watchdog would release
+          torque that long afterwards whatever hold_torque_on_deactivate says.
+          The two settings are one decision.
+        -->
+        <param name="hold_torque_on_deactivate">true</param>
+        <param name="motor_can_timeout_ms">0</param>
+        <!--
+          Losing a joint freezes the component: the lost joint is left limp,
+          every reachable joint keeps torque and holds where it was, and
+          controller commands are ignored. The alternative cuts torque on all
+          seven, which drops the arm.
+        -->
+        <param name="freeze_on_joint_loss">true</param>
+        <param name="torque_enable">$(arg torque_enable)</param>
+      </xacro:if>
+    </hardware>
+    <xacro:rebot_joint name="joint1" id="1" model="RS06" kp="50.0" kd="3.0" />
+    <xacro:rebot_joint name="joint2" id="2" model="RS06" kp="150.0" kd="10.0" />
+    <xacro:rebot_joint name="joint3" id="3" model="RS06" kp="150.0" kd="10.0" />
+    <xacro:rebot_joint name="joint4" id="4" model="RS00" kp="50.0" kd="5.0" />
+    <xacro:rebot_joint name="joint5" id="5" model="RS00" kp="50.0" kd="4.0" />
+    <xacro:rebot_joint name="joint6" id="6" model="RS00" kp="50.0" kd="4.0" />
+    <xacro:rebot_joint name="joint7" id="7" model="RS00" kp="12.0" kd="0.05" mode="motion" />
   </ros2_control>
 </robot>

Commit message: fix(rebot_bench_base_config): anchor stack legs to the command and run them at full speed
Every Stack Blue on Red leg now starts from the controller's previous
command: AnchorTrajectoryToCommand shifts each validated
trajectory onto the last committed endpoint, holds the joints it leaves out,
and falls back to measured state for a missing command or one more than
0.10 rad away. Endpoints are committed only after successful execution, and
RecordRebotTrajectory saves each trajectory before dispatch.

Pick Blue Cube first closes the jaw with the native Close Gripper, planned
from measured state, then starts from the commanded home rather than the
measured rest: a sagged joint can measure past its limit, which the planners
refuse. Gripper legs move the jaw from its measured position while holding the
arm at its command, so a jaw command left stale by an abort cannot shift the
opening past its limit. The return home
fades its anchoring offset out so it ends exactly at the waypoint.

Gripper legs go through Move reBot Gripper with named waypoints; the survey
and the return home go through reBot Move to Arm Waypoint. Pick Blue
Cube grasps with the fingertips 35 mm above the bench, and the release pose
rests the tilted cube on red before opening. A successful stack closes the
empty jaw at home with the native Close Gripper, so all seven joints end at
home; a point-to-point trajectory ending exactly on joint7's lower bound can
undershoot it and be refused.

Arm planning limits are doubled to 0.6 rad/s and 1.2 rad/s^2; the jaw keeps
3.0 rad/s and 6.0 rad/s^2, since faster it lags past the controller's single
0.15 rad path tolerance. All legs read reBot Stack Motion, now
1.0 for every kind; the README explains how to size the bench speed guard
against it. Plan reBot Joint Move keeps its 0.045 rad/s cap. rebot_bench_sim
shadows that subtree with its own settings file so the twin stays at full
speed whatever the arm's values. The twin scene enables NoSlip to stop a
resting stack creeping. The README gains a section on running the stack on
the real arm, with its settings.

Stack Blue on Red no longer stops where a failed leg left it. Once the cubes
are located from home, and before any jaw or arm motion, reBot Check Stack
Reach solves IK for the pick hover, pick, place hover and place, and an
unreachable pose fails without moving, with a message naming the cube and its
position, worded by the new ReportUnreachableCube Behavior. Any later failure,
IK included, goes through reBot Recover Home: it returns home holding the jaw
at its command, then closes the jaw with Close Gripper unless the jaw may be
around the cube, from just before the grasp closes until the release opening
is confirmed, and the Objective still fails. The close runs even when the move
home is refused, as it is from home after the final close aborts. The planning-scene
wall now stands 5 mm proud of the real face: near it, a tilted place hover that
only grazed the wall was chosen, and tracking error at full speed put the
measured arm in collision so the place descent was refused at its start.

File: src/rebot_bench_base_config/description/rebot.urdf.xacro (robot description, xacro)
@@ -105,5 +105,5 @@
     <child link="link1" />
     <axis xyz="0 0 -1" />
-    <limit lower="-2.530727415392" upper="2.530727415392" effort="36" velocity="0.3" />
+    <limit lower="-2.530727415392" upper="2.530727415392" effort="36" velocity="0.6" />
   </joint>
   <link name="link2">
@@ -164,5 +164,5 @@
     <child link="link2" />
     <axis xyz="0 0 1" />
-    <limit lower="0.000000000000" upper="3.543018381548" effort="36" velocity="0.3" />
+    <limit lower="0.000000000000" upper="3.543018381548" effort="36" velocity="0.6" />
   </joint>
   <link name="link3">
@@ -223,5 +223,5 @@
     <child link="link3" />
     <axis xyz="0 0 -1" />
-    <limit lower="0.000000000000" upper="4.171336912266" effort="36" velocity="0.3" />
+    <limit lower="0.000000000000" upper="4.171336912266" effort="36" velocity="0.6" />
   </joint>
   <link name="link4">
@@ -257,5 +257,5 @@
     <child link="link4" />
     <axis xyz="0 0 -1" />
-    <limit lower="-1.850049007114" upper="1.500983156715" effort="14" velocity="0.3" />
+    <limit lower="-1.850049007114" upper="1.500983156715" effort="14" velocity="0.6" />
   </joint>
   <link name="link5">
@@ -297,5 +297,5 @@
     <child link="link5" />
     <axis xyz="0 0 -1" />
-    <limit lower="-1.762782544514" upper="1.884955592154" effort="14" velocity="0.3" />
+    <limit lower="-1.762782544514" upper="1.884955592154" effort="14" velocity="0.6" />
   </joint>
   <link name="link6">
@@ -324,5 +324,5 @@
     <child link="link6" />
     <axis xyz="0 0 -1" />
-    <limit lower="-3.054326190990" upper="3.054326190990" effort="14" velocity="0.3" />
+    <limit lower="-3.054326190990" upper="3.054326190990" effort="14" velocity="0.6" />
   </joint>
   <link name="gripper_end">

File: src/rebot_bench_sim/description/scene.xml.xacro (robot description, xacro)
@@ -24,5 +24,7 @@
        orientations copy straight across. -->
   <compiler angle="radian" eulerseq="XYZ" autolimits="true" />
-  <option timestep="0.003" integrator="implicitfast" />
+  <!-- Remove friction-dimension drift from soft contacts under a resting stack.
+       NoSlip postprocessing preserves the contact/friction material parameters. -->
+  <option timestep="0.003" integrator="implicitfast" noslip_iterations="10" />
   <include file="rebot_assets.xml" />
   <statistic center="0.25 0.1 0.15" extent="0.8" />
