Commit message: feat(rebot): add reusable SAM3 cube stacking objectives
Add shared cube perception, pick and stack Objectives with simulation evidence and configurable motion settings. Verify preparation jaw opening with retry and measured state. Reject single-frame and nonpositive-duration evidence recordings. Preserve the original recording error, attach later cleanup failures as exception notes, and attempt stream closure, encoder reaping, node destruction and ROS shutdown even when preceding cleanup fails.

File: src/rebot_bench_base_config/description/rebot.urdf.xacro (robot description, xacro)
@@ -17,10 +17,16 @@
   <xacro:arg name="arm_control_mode" default="motion" />
   <!-- Placement of base_link and of the scene camera mount in `world`, as
-       "x y z" and URDF "roll pitch yaw". rebot_bench_sim sets both from its
-       bench layout; unset, both coincide with world. -->
+       "x y z" and URDF "roll pitch yaw". config.yaml sets the bench's
+       calibration; unset, both coincide with world. A wrapping description
+       that defines these properties first keeps its own placement over the
+       arguments: rebot_bench_sim, from its bench layout. -->
   <xacro:arg name="world_to_base_xyz" default="0 0 0" />
   <xacro:arg name="world_to_base_rpy" default="0 0 0" />
   <xacro:arg name="scene_camera_xyz" default="0 0 0" />
   <xacro:arg name="scene_camera_rpy" default="0 0 0" />
+  <xacro:property name="world_to_base_xyz" default="$(arg world_to_base_xyz)" />
+  <xacro:property name="world_to_base_rpy" default="$(arg world_to_base_rpy)" />
+  <xacro:property name="scene_camera_xyz" default="$(arg scene_camera_xyz)" />
+  <xacro:property name="scene_camera_rpy" default="$(arg scene_camera_rpy)" />
   <!-- d435_mount_joint origin (gripper_end -> d435_mount_link). The default is
        the nominal, eye-measured mount; a hand-eye calibration overrides it. -->
@@ -440,5 +446,5 @@
     <parent link="world" />
     <child link="base_link" />
-    <origin xyz="$(arg world_to_base_xyz)" rpy="$(arg world_to_base_rpy)" />
+    <origin xyz="${world_to_base_xyz}" rpy="${world_to_base_rpy}" />
   </joint>
   <link name="d435_mount_link">
@@ -487,5 +493,5 @@
     <parent link="world" />
     <child link="scene_camera_link" />
-    <origin xyz="$(arg scene_camera_xyz)" rpy="$(arg scene_camera_rpy)" />
+    <origin xyz="${scene_camera_xyz}" rpy="${scene_camera_rpy}" />
   </joint>
   <xacro:unless value="${simulator_owns_optical_frames}">

File: src/rebot_bench_sim/description/rebot_arm.xml.xacro (robot description, xacro)
@@ -268,4 +268,11 @@
                   />
                   <joint name="gripper_joint1" class="jaw" />
+                  <!-- SIM-ONLY grasp proxy, enabled by the twin's launch hook.
+                       MuJoCo activates the named weld only on cube contact. -->
+                  <site
+                    name="suction_cup_sim_grasp_proxy"
+                    size="0.001"
+                    group="5"
+                  />
                   <geom
                     class="visual"
@@ -278,5 +285,14 @@
                     material="rs_anodized_silver"
                   />
-                  <geom class="collision" mesh="gripper_left" />
+                  <!-- Keep the finger separate from its carriage: one convex hull
+                       across both fills the open grasping aperture. -->
+                  <!-- Pad friction is a simulation parameter, not a measured
+                       hardware coefficient. The actuator supplies the squeeze. -->
+                  <geom
+                    class="collision"
+                    mesh="pla_left"
+                    friction="2 0.005 0.0001"
+                  />
+                  <geom class="collision" mesh="cnc_left" />
                 </body>
                 <body
@@ -302,5 +318,14 @@
                     material="rs_anodized_silver"
                   />
-                  <geom class="collision" mesh="gripper_right" />
+                  <!-- Keep the finger separate from its carriage: one convex hull
+                       across both fills the open grasping aperture. -->
+                  <!-- Pad friction is a simulation parameter, not a measured
+                       hardware coefficient. The actuator supplies the squeeze. -->
+                  <geom
+                    class="collision"
+                    mesh="pla_right"
+                    friction="2 0.005 0.0001"
+                  />
+                  <geom class="collision" mesh="cnc_right" />
                 </body>
                 <body

File: src/rebot_bench_sim/description/rebot_bench_sim.urdf.xacro (robot description, xacro)
@@ -12,12 +12,15 @@
   <xacro:property name="layout" value="${xacro.load_yaml('$(arg layout)')}" />
   <!-- An xacro:arg keeps its first declaration, so these defaults win over
-       the base file's identity placements. -->
+       the base file's. -->
   <xacro:arg name="hardware_interface" default="mujoco" />
-  <xacro:arg name="world_to_base_xyz" default="${' '.join(map(str, layout['robot_base']['xyz']))}" />
-  <xacro:arg name="world_to_base_rpy" default="${' '.join(map(str, layout['robot_base']['rpy']))}" />
-  <xacro:arg name="scene_camera_xyz" default="${' '.join(map(str, layout['scene_camera']['xyz']))}" />
-  <xacro:arg name="scene_camera_rpy" default="${' '.join(map(str, layout['scene_camera']['rpy']))}" />
   <xacro:arg name="wrist_camera_mount_xyz" default="${' '.join(map(str, layout['wrist_camera_mount']['xyz']))}" />
   <xacro:arg name="wrist_camera_mount_rpy" default="${' '.join(map(str, layout['wrist_camera_mount']['rpy']))}" />
+  <!-- The base file keeps these properties over its placement arguments, so
+       the layout places the twin even though the base config's bench
+       calibration is inherited through urdf_params. -->
+  <xacro:property name="world_to_base_xyz" value="${' '.join(map(str, layout['robot_base']['xyz']))}" />
+  <xacro:property name="world_to_base_rpy" value="${' '.join(map(str, layout['robot_base']['rpy']))}" />
+  <xacro:property name="scene_camera_xyz" value="${' '.join(map(str, layout['scene_camera']['xyz']))}" />
+  <xacro:property name="scene_camera_rpy" value="${' '.join(map(str, layout['scene_camera']['rpy']))}" />
   <xacro:include filename="$(find rebot_bench_base_config)/description/rebot.urdf.xacro" />
   <!-- Any other selector would add a second hardware block for the same joints. -->
@@ -34,5 +37,5 @@
       <param name="mujoco_keyframe">$(arg mujoco_keyframe)</param>
       <param name="mujoco_viewer">$(arg mujoco_viewer)</param>
-      <param name="render_publish_rate">10</param>
+      <param name="render_publish_rate">30</param>
       <!-- Colour and depth images only, as on the bench: no point clouds. -->
       <param name="point_cloud_publish_rate">0</param>

Commit message: fix(rebot): allow conservative lower home margins

File: src/rebot_bench_base_config/description/rebot.urdf.xacro (robot description, xacro)
@@ -1,4 +1,4 @@
 <?xml version='1.0' encoding='UTF-8'?>
-<!-- Derived from Seeed reBot-DevArm; CERN-OHL-W-2.0. Modified by PickNik Inc., 2026-10-09 to 2026-10-12: visual replacements, hardware selectors, world placement and wrist-camera mount arguments. See NOTICE.md. Original SolidWorks exporter: Stephen Brawner (brawner@gmail.com), 1.6.0-4-g7f85cfe, build 1.6.7995.38578; http://wiki.ros.org/sw_urdf_exporter. -->
+<!-- Derived from Seeed reBot-DevArm; CERN-OHL-W-2.0. Modified by PickNik Inc., 2026-10-09 to 2026-10-14: visual replacements, hardware selectors, world placement, wrist-camera mount arguments and conservative home margins. See NOTICE.md. Original SolidWorks exporter: Stephen Brawner (brawner@gmail.com), 1.6.0-4-g7f85cfe, build 1.6.7995.38578; http://wiki.ros.org/sw_urdf_exporter. -->
 <robot name="rebot_b601_rs" xmlns:xacro="http://www.ros.org/wiki/xacro">
   <xacro:arg name="hardware_interface" default="mock" />
@@ -164,5 +164,5 @@
     <child link="link2" />
     <axis xyz="0 0 1" />
-    <limit lower="0.000000000000" upper="3.543018381548" effort="36" velocity="0.6" />
+    <limit lower="-0.020000000000" upper="3.543018381548" effort="36" velocity="0.6" />
   </joint>
   <link name="link3">
@@ -223,5 +223,5 @@
     <child link="link3" />
     <axis xyz="0 0 -1" />
-    <limit lower="0.000000000000" upper="4.171336912266" effort="36" velocity="0.6" />
+    <limit lower="-0.010000000000" upper="4.171336912266" effort="36" velocity="0.6" />
   </joint>
   <link name="link4">

File: src/rebot_bench_sim/description/rebot_arm.xml.xacro (robot description, xacro)
@@ -48,5 +48,5 @@
         fullinertia="0.00073374 0.01255987 0.01281387 -0.00000043 0.00000851 0.00000128"
       />
-      <joint name="joint2" class="rs06" axis="0 0 1" range="0 3.543018381548" />
+      <joint name="joint2" class="rs06" axis="0 0 1" range="-0.02 3.543018381548" />
       <geom class="visual" mesh="motor_2_3" material="rs_motor_black" />
       <geom class="visual" mesh="cnc2" material="rs_anodized_silver" />
@@ -105,5 +105,5 @@
           class="rs06"
           axis="0 0 -1"
-          range="0 4.171336912266"
+          range="-0.01 4.171336912266"
         />
         <geom class="visual" mesh="cnc3" material="rs_anodized_silver" />
