Commit message: fix(lunar_sim): Pin the duplicated A300 yellow material to a lower albedo
The vendored A300 declares the material name "yellow" twice with different
colours: rgba 1 0.6038269 0 for the enclosure access panels and rgba
0.8 0.8 0 for the sensor arch. The web viewer keeps one entry per material
name and the last one parsed wins, so the arch value currently paints both
parts and the enclosure colour never renders.

Declare it last so the result is pinned rather than left to file order, at
the enclosure hue scaled to 0.55 peak. At albedo 1.0 the red channel
saturates under the viewer lights and tone maps toward white against the
low-albedo regolith.

urdfdom keeps the first occurrence of a duplicated material name rather
than the last, so this pins the web viewer only. MoveIt Pro renders URDF
material colours through that viewer alone, so no other surface changes.

Co-Authored-By: Claude Opus 5 (1M context) <noreply@anthropic.com>

File: src/lunar_sim/description/husky_a300_mujoco.xacro (robot description, xacro)
@@ -55,4 +55,13 @@
   <xacro:lunar_lidar_body name="lidar_front" xyz="0.45 0 0.3208593" />
   <xacro:lunar_lidar_body name="lidar_rear" xyz="-0.2728 0 0.6500193" />
+  <!-- The vendored A300 declares the name "yellow" twice: rgba 1 0.6038269 0
+       in attachments/amp_enclosure.urdf.xacro (access panels) and rgba
+       0.8 0.8 0 in attachments/amp_sensor_arch.urdf.xacro (arch). The web
+       viewer keeps one entry per material name and the last one parsed wins, so
+       the arch value currently paints both parts. Declaring it last pins the
+       result, at the enclosure hue scaled to 0.55 peak so the red channel stays
+       under the tone mapper white point. urdfdom keeps the first occurrence
+       instead, so this pins the web viewer only. -->
+  <material name="yellow"><color rgba="0.55 0.332 0.0 1" /></material>
   <!-- MuJoCo hardware: real physics, driven by description/husky_scene.xml (see that file and
        husky_a300.xml for the body/wheel/actuator model). Wheel joint names match

Commit message: feat(lunar_sim): add lidar scans, IMU, fuse, Nav2, and dead reckoning
Co-Authored-By: Claude Opus 5.5 <noreply@anthropic.com>

File: src/lunar_sim/description/husky_a300_mujoco.xacro (robot description, xacro)
@@ -55,4 +55,10 @@
   <xacro:lunar_lidar_body name="lidar_front" xyz="0.45 0 0.3208593" />
   <xacro:lunar_lidar_body name="lidar_rear" xyz="-0.2728 0 0.6500193" />
+  <!-- Phidgets Spatial IMU; mount matches husky_a300.xml's imu_link body. -->
+  <link name="imu_link" />
+  <joint name="imu_joint" type="fixed">
+    <parent link="base_link" /><child link="imu_link" />
+    <origin xyz="0.059 0 0.161275" />
+  </joint>
   <!-- MuJoCo hardware: real physics, driven by description/husky_scene.xml (see that file and
        husky_a300.xml for the body/wheel/actuator model). Wheel joint names match
@@ -107,16 +113,6 @@
       <param name="mujoco_viewer">$(arg mujoco_viewer)</param>
       <param name="mujoco_keyframe">$(arg mujoco_keyframe)</param>
-      <!-- TF ownership: robot_state_publisher owns every link below footprint (footprint ->
-           base_link -> chassis_link -> wheels ...) and platform_velocity_controller owns
-           odom -> footprint. MuJoCo must not broadcast mj_world -> chassis_link (that 60 Hz edge
-           would beat the static base_link -> chassis_link and split the tree in two). With
-           odom_frame set, publish_mj_world_tf=true makes MujocoSystem publish mj_world -> odom as
-           identity instead (mujoco_system.cpp, publish_sites), which is what connects the
-           world-fixed scene_camera_optical_frame site (parented to mj_world, husky_scene.xml) to
-           odom so /scene_camera/points can be shown in the odom frame. base_link_name stops the
-           site TF fill-in at the chassis body instead of walking up to the MJCF worldbody. Ground
-           truth for the Dead Reckon Square calibration comes from the chassis freejoint pose read
-           from MuJoCo directly, not from TF. -->
-      <param name="publish_mj_world_tf">true</param>
+      <!-- TF ownership: robot_state_publisher owns every link below footprint, fuse owns odom -> footprint, and robot_drivers_to_persist_sim.launch.py publishes mj_world -> map -> odom. publish_mj_world_tf is off so MuJoCo does not give odom a second parent; base_link_name stops the site TF fill-in at the chassis body. -->
+      <param name="publish_mj_world_tf">false</param>
       <param name="odom_frame">odom</param>
       <param name="base_link_name">chassis_link</param>
@@ -139,9 +135,27 @@
       </xacro:if>
     </hardware>
+    <!-- The scan is the cloud's middle ring, published in the <camera>_ROS frame MujocoSystem broadcasts. -->
     <sensor name="lidar_front">
+      <param name="lidar_output">both</param>
       <param name="points_topic">/lidar_front/points</param>
+      <param name="scan_topic">/scan_front</param>
     </sensor>
     <sensor name="lidar_rear">
+      <param name="lidar_output">both</param>
       <param name="points_topic">/lidar_rear/points</param>
+      <param name="scan_topic">/scan_rear</param>
+    </sensor>
+    <!-- Named after the MJCF site carrying husky_a300.xml's framequat, gyro, and accelerometer. -->
+    <sensor name="imu_site">
+      <state_interface name="orientation.x" />
+      <state_interface name="orientation.y" />
+      <state_interface name="orientation.z" />
+      <state_interface name="orientation.w" />
+      <state_interface name="angular_velocity.x" />
+      <state_interface name="angular_velocity.y" />
+      <state_interface name="angular_velocity.z" />
+      <state_interface name="linear_acceleration.x" />
+      <state_interface name="linear_acceleration.y" />
+      <state_interface name="linear_acceleration.z" />
     </sensor>
     <joint name="front_left_wheel_joint">

Commit message: feat(lunar_sim): add lidar scans, IMU, fuse, Nav2, and dead reckoning
Co-Authored-By: Claude Opus 5.5 <noreply@anthropic.com>

File: src/lunar_sim/description/husky_a300_mujoco.xacro (robot description, xacro)
@@ -55,4 +55,10 @@
   <xacro:lunar_lidar_body name="lidar_front" xyz="0.45 0 0.3208593" />
   <xacro:lunar_lidar_body name="lidar_rear" xyz="-0.2728 0 0.6500193" />
+  <!-- Phidgets Spatial IMU; mount matches husky_a300.xml's imu_link body. -->
+  <link name="imu_link" />
+  <joint name="imu_joint" type="fixed">
+    <parent link="base_link" /><child link="imu_link" />
+    <origin xyz="0.059 0 0.161275" />
+  </joint>
   <!-- MuJoCo hardware: real physics, driven by description/husky_scene.xml (see that file and
        husky_a300.xml for the body/wheel/actuator model). Wheel joint names match
@@ -98,16 +104,6 @@
       <param name="mujoco_viewer">$(arg mujoco_viewer)</param>
       <param name="mujoco_keyframe">$(arg mujoco_keyframe)</param>
-      <!-- TF ownership: robot_state_publisher owns every link below footprint (footprint ->
-           base_link -> chassis_link -> wheels ...) and platform_velocity_controller owns
-           odom -> footprint. MuJoCo must not broadcast mj_world -> chassis_link (that 60 Hz edge
-           would beat the static base_link -> chassis_link and split the tree in two). With
-           odom_frame set, publish_mj_world_tf=true makes MujocoSystem publish mj_world -> odom as
-           identity instead (mujoco_system.cpp, publish_sites), which is what connects the
-           world-fixed scene_camera_optical_frame site (parented to mj_world, husky_scene.xml) to
-           odom so /scene_camera/points can be shown in the odom frame. base_link_name stops the
-           site TF fill-in at the chassis body instead of walking up to the MJCF worldbody. Ground
-           truth for the Dead Reckon Square calibration comes from the chassis freejoint pose read
-           from MuJoCo directly, not from TF. -->
-      <param name="publish_mj_world_tf">true</param>
+      <!-- TF ownership: robot_state_publisher owns every link below footprint, fuse owns odom -> footprint, and robot_drivers_to_persist_sim.launch.py publishes mj_world -> map -> odom. publish_mj_world_tf is off so MuJoCo does not give odom a second parent; base_link_name stops the site TF fill-in at the chassis body. -->
+      <param name="publish_mj_world_tf">false</param>
       <param name="odom_frame">odom</param>
       <param name="base_link_name">chassis_link</param>
@@ -130,9 +126,27 @@
       </xacro:if>
     </hardware>
+    <!-- The scan is the cloud's middle ring, published in the <camera>_ROS frame MujocoSystem broadcasts. -->
     <sensor name="lidar_front">
+      <param name="lidar_output">both</param>
       <param name="points_topic">/lidar_front/points</param>
+      <param name="scan_topic">/scan_front</param>
     </sensor>
     <sensor name="lidar_rear">
+      <param name="lidar_output">both</param>
       <param name="points_topic">/lidar_rear/points</param>
+      <param name="scan_topic">/scan_rear</param>
+    </sensor>
+    <!-- Named after the MJCF site carrying husky_a300.xml's framequat, gyro, and accelerometer. -->
+    <sensor name="imu_site">
+      <state_interface name="orientation.x" />
+      <state_interface name="orientation.y" />
+      <state_interface name="orientation.z" />
+      <state_interface name="orientation.w" />
+      <state_interface name="angular_velocity.x" />
+      <state_interface name="angular_velocity.y" />
+      <state_interface name="angular_velocity.z" />
+      <state_interface name="linear_acceleration.x" />
+      <state_interface name="linear_acceleration.y" />
+      <state_interface name="linear_acceleration.z" />
     </sensor>
     <joint name="front_left_wheel_joint">
